File: Power_+10V.sch (KiCad schematic (older format))
At the start: 30 parts

Commit message: Add files via upload
Parts:
- removed C?: 1u, Capacitor_SMD:C_0603_1608Metric_Pad1.08x0.95mm_HandSolder, symbol Device:C
- removed C? (x6): 10u, Capacitor_SMD:C_1206_3216Metric_Pad1.33x1.80mm_HandSolder, symbol Device:C
- removed C?: 0,1, Capacitor_SMD:C_0603_1608Metric_Pad1.08x0.95mm_HandSolder, symbol Device:C
- removed C?: 100u, symbol Device:CP
- removed D? (x3): BAT54S, Package_TO_SOT_SMD:SOT-23, symbol Diode:BAT54S
- removed D?: SMAJ5.0CA, symbol Device:D_TVS
- removed Q?: IRLML2402, Package_TO_SOT_SMD:SOT-23, symbol Transistor_FET:IRLML2060
- removed Q?: BC847, Package_TO_SOT_SMD:SOT-23, symbol Transistor_BJT:BC847
- removed Q?: IRLML6402, Package_TO_SOT_SMD:SOT-23, symbol Transistor_FET:IRLML6402
- removed R? (x2): 1,2k, Resistor_SMD:R_0603_1608Metric_Pad0.98x0.95mm_HandSolder, symbol Device:R
- removed R?: 330, Resistor_SMD:R_0603_1608Metric_Pad0.98x0.95mm_HandSolder, symbol Device:R
- removed R? (x3): 56k, Resistor_SMD:R_0603_1608Metric_Pad0.98x0.95mm_HandSolder, symbol Device:R
- removed R?: 3,3k, Resistor_SMD:R_0603_1608Metric_Pad0.98x0.95mm_HandSolder, symbol Device:R
- removed R?: 100, Resistor_SMD:R_0603_1608Metric_Pad0.98x0.95mm_HandSolder, symbol Device:R
- removed R?: 680, Resistor_SMD:R_0603_1608Metric_Pad0.98x0.95mm_HandSolder, symbol Device:R
- removed TP? (x4): TestPoint, symbol Connector:TestPoint
- removed U?: AMS1117-3.3, Package_TO_SOT_SMD:SOT-223-3_TabPin2, symbol Regulator_Linear:AMS1117-3.3
- added C? (x2): 0,1, Capacitor_SMD:C_0603_1608Metric_Pad1.08x0.95mm_HandSolder, symbol Device:C
- added C?: 100u, symbol Device:CP
- added C? (x2): 470u, symbol Device:CP
- added C?: 1000, Capacitor_SMD:C_0603_1608Metric_Pad1.08x0.95mm_HandSolder, symbol Device:C
- added D?: MBR0540, symbol Device:D_Schottky
- added FB?: Ferrite_Bead, symbol Device:Ferrite_Bead
- added L? (x2): 330u, symbol Device:L
- added R?: 0,47 2010, symbol Device:R
- added R?: 200, Resistor_SMD:R_0603_1608Metric_Pad0.98x0.95mm_HandSolder, symbol Device:R
- added R?: 2,4k 1%, Resistor_SMD:R_0603_1608Metric_Pad0.98x0.95mm_HandSolder, symbol Device:R
- added R?: 47k 1%, Resistor_SMD:R_0603_1608Metric_Pad0.98x0.95mm_HandSolder, symbol Device:R
- added TP? (x5): TestPoint, symbol Connector:TestPoint
- added U?: MC34063AD, Package_SO:SOIC-8_3.9x4.9mm_P1.27mm, symbol Regulator_Switching:MC34063AD
Connections:
- net labels added: +10V_OUT
- net labels removed: +10V, +3V3, +5V, CHARGE_PUMP_CLK, GND_IN
- wire segments 77 -> 52
- no-connect marks 2 -> 0
Other:
- note added: "Power source +10V"
- note removed: "Power sources 3V3 and 10V"

Commit message: Add files via upload
Parts:
- removed FB?: Ferrite_Bead, symbol Device:Ferrite_Bead
- C?: value 1000 -> 500
Connections:
- net +10V_OUT: now also C?.1, C?.1, L?.2
Changed lines of the file:
@@
 AR Path="/60DF07DE/60ED6B0B" Ref="C?"  Part="1"
 F 0 "C?" H 3615 4096 50  0000 L CNN
-F 1 "1000" H 3615 4005 50  0000 L CNN
+F 1 "500" H 3615 4005 50  0000 L CNN
 F 2 "Capacitor_SMD:C_0603_1608Metric_Pad1.08x0.95mm_HandSolder" H 3538 3900 50  0001 C CNN
 F 3 "~" H 3500 4050 50  0001 C CNN
@@
 	1    0    0    -1
 $EndComp
-$Comp
-L Device:Ferrite_Bead FB?
-U 1 1 60EDC632
-P 9650 3500
-F 0 "FB?" V 9376 3500 50  0000 C CNN
-F 1 "Ferrite_Bead" V 9467 3500 50  0000 C CNN
-F 2 "" V 9580 3500 50  0001 C CNN
-F 3 "~" H 9650 3500 50  0001 C CNN
-	1    9650 3500
-	0    1    1    0
-$EndComp
 Wire Wire Line
 	7500 3500 7800 3500
@@
 	8500 3500 9000 3500
 Connection ~ 9000 3500
-Wire Wire Line
-	9000 3500 9500 3500
-Wire Wire Line
-	9800 3500 10100 3500
 Wire Wire Line
 	9000 3800 9000 4500
@@
 Wire Wire Line
 	8100 4500 7500 4500
+Wire Wire Line
+	9000 3500 10100 3500
 $EndSCHEMATC
