File: Power_+10V.sch (KiCad schematic (older format))
At the start: 19 parts

Commit message: Add files via upload
Parts:
- gave numbers to parts that had none: 19
Changed lines of the file:
@@
 AR Path="/609FED99/60ED6AC7" Ref="C?"  Part="1"
 AR Path="/60DF0860/60ED6AC7" Ref="C?"  Part="1"
-AR Path="/60DF07DE/60ED6AC7" Ref="C?"  Part="1"
+AR Path="/60DF07DE/60ED6AC7" Ref="C17"  Part="1"
 AR Path="/60F1863C/60ED6AC7" Ref="C?"  Part="1"
-F 0 "C?" H 3115 3696 50  0000 L CNN
+F 0 "C17" H 3115 3696 50  0000 L CNN
 F 1 "0,1" H 3115 3605 50  0000 L CNN
 F 2 "Capacitor_SMD:C_0603_1608Metric_Pad1.08x0.95mm_HandSolder" H 3038 3500 50  0001 C CNN
@@
 AR Path="/609FED99/60ED6ACD" Ref="R?"  Part="1"
 AR Path="/60DF0860/60ED6ACD" Ref="R?"  Part="1"
-AR Path="/60DF07DE/60ED6ACD" Ref="R?"  Part="1"
+AR Path="/60DF07DE/60ED6ACD" Ref="R8"  Part="1"
 AR Path="/60F1863C/60ED6ACD" Ref="R?"  Part="1"
-F 0 "R?" V 4200 2950 50  0000 L CNN
+F 0 "R8" V 4200 2950 50  0000 L CNN
 F 1 "0,47 2010" V 4400 2800 50  0000 L CNN
 F 2 "" V 4230 3000 50  0001 C CNN
@@
 AR Path="/609FED99/60ED6AD3" Ref="R?"  Part="1"
 AR Path="/60DF0860/60ED6AD3" Ref="R?"  Part="1"
-AR Path="/60DF07DE/60ED6AD3" Ref="R?"  Part="1"
+AR Path="/60DF07DE/60ED6AD3" Ref="R9"  Part="1"
 AR Path="/60F1863C/60ED6AD3" Ref="R?"  Part="1"
-F 0 "R?" H 5320 3196 50  0000 L CNN
+F 0 "R9" H 5320 3196 50  0000 L CNN
 F 1 "200" H 5320 3105 50  0000 L CNN
 F 2 "Resistor_SMD:R_0603_1608Metric_Pad0.98x0.95mm_HandSolder" V 5180 3150 50  0001 C CNN
@@
 AR Path="/609FED99/60ED6AD9" Ref="TP?"  Part="1"
 AR Path="/60DF0860/60ED6AD9" Ref="TP?"  Part="1"
-AR Path="/60DF07DE/60ED6AD9" Ref="TP?"  Part="1"
+AR Path="/60DF07DE/60ED6AD9" Ref="TP6"  Part="1"
 AR Path="/60F1863C/60ED6AD9" Ref="TP?"  Part="1"
-F 0 "TP?" H 7308 3618 50  0000 L CNN
+F 0 "TP6" H 7308 3618 50  0000 L CNN
 F 1 "TestPoint" H 7308 3527 50  0001 L CNN
 F 2 "" H 7450 3500 50  0001 C CNN
@@
 AR Path="/609FED99/60ED6ADF" Ref="TP?"  Part="1"
 AR Path="/60DF0860/60ED6ADF" Ref="TP?"  Part="1"
-AR Path="/60DF07DE/60ED6ADF" Ref="TP?"  Part="1"
+AR Path="/60DF07DE/60ED6ADF" Ref="TP5"  Part="1"
 AR Path="/60F1863C/60ED6ADF" Ref="TP?"  Part="1"
-F 0 "TP?" H 4658 3118 50  0000 L CNN
+F 0 "TP5" H 4658 3118 50  0000 L CNN
 F 1 "TestPoint" H 4658 3027 50  0001 L CNN
 F 2 "" H 4800 3000 50  0001 C CNN
@@
 P 2500 3650
 AR Path="/60DF0860/60F18F0E" Ref="C?"  Part="1"
-AR Path="/60DF07DE/60F18F0E" Ref="C?"  Part="1"
+AR Path="/60DF07DE/60F18F0E" Ref="C16"  Part="1"
 AR Path="/60F1863C/60F18F0E" Ref="C?"  Part="1"
-F 0 "C?" H 2618 3696 50  0000 L CNN
+F 0 "C16" H 2618 3696 50  0000 L CNN
 F 1 "100u" H 2618 3605 50  0000 L CNN
 F 2 "" H 2538 3500 50  0001 C CNN
@@
 AR Path="/609FED99/60F18F0F" Ref="TP?"  Part="1"
 AR Path="/60DF0860/60F18F0F" Ref="TP?"  Part="1"
-AR Path="/60DF07DE/60F18F0F" Ref="TP?"  Part="1"
+AR Path="/60DF07DE/60F18F0F" Ref="TP4"  Part="1"
 AR Path="/60F1863C/60F18F0F" Ref="TP?"  Part="1"
-F 0 "TP?" H 4058 3118 50  0000 L CNN
+F 0 "TP4" H 4058 3118 50  0000 L CNN
 F 1 "TestPoint" H 4058 3027 50  0001 L CNN
 F 2 "" H 4200 3000 50  0001 C CNN
@@
 AR Path="/609FED99/60ED6AF3" Ref="R?"  Part="1"
 AR Path="/60DF0860/60ED6AF3" Ref="R?"  Part="1"
-AR Path="/60DF07DE/60ED6AF3" Ref="R?"  Part="1"
+AR Path="/60DF07DE/60ED6AF3" Ref="R11"  Part="1"
 AR Path="/60F1863C/60ED6AF3" Ref="R?"  Part="1"
-F 0 "R?" H 7070 4196 50  0000 L CNN
+F 0 "R11" H 7070 4196 50  0000 L CNN
 F 1 "2,4k 1%" H 7070 4105 50  0000 L CNN
 F 2 "Resistor_SMD:R_0603_1608Metric_Pad0.98x0.95mm_HandSolder" V 6930 4150 50  0001 C CNN
@@
 P 4300 3700
 AR Path="/60DF0860/60ED6AF9" Ref="U?"  Part="1"
-AR Path="/60DF07DE/60ED6AF9" Ref="U?"  Part="1"
+AR Path="/60DF07DE/60ED6AF9" Ref="U4"  Part="1"
 AR Path="/60F1863C/60ED6AF9" Ref="U?"  Part="1"
-F 0 "U?" H 4300 4167 50  0000 C CNN
+F 0 "U4" H 4300 4167 50  0000 C CNN
 F 1 "MC34063AD" H 4300 4076 50  0000 C CNN
 F 2 "Package_SO:SOIC-8_3.9x4.9mm_P1.27mm" H 4350 3250 50  0001 L CNN
@@
 P 7500 3650
 AR Path="/60DF0860/60F18F12" Ref="C?"  Part="1"
-AR Path="/60DF07DE/60F18F12" Ref="C?"  Part="1"
+AR Path="/60DF07DE/60F18F12" Ref="C19"  Part="1"
 AR Path="/60F1863C/60F18F12" Ref="C?"  Part="1"
-F 0 "C?" H 7618 3696 50  0000 L CNN
+F 0 "C19" H 7618 3696 50  0000 L CNN
 F 1 "470u" H 7618 3605 50  0000 L CNN
 F 2 "" H 7538 3500 50  0001 C CNN
@@
 AR Path="/609FED99/60F18F13" Ref="R?"  Part="1"
 AR Path="/60DF0860/60F18F13" Ref="R?"  Part="1"
-AR Path="/60DF07DE/60F18F13" Ref="R?"  Part="1"
+AR Path="/60DF07DE/60F18F13" Ref="R10"  Part="1"
 AR Path="/60F1863C/60F18F13" Ref="R?"  Part="1"
-F 0 "R?" H 7070 3696 50  0000 L CNN
+F 0 "R10" H 7070 3696 50  0000 L CNN
 F 1 "47k 1%" H 7070 3605 50  0000 L CNN
 F 2 "Resistor_SMD:R_0603_1608Metric_Pad0.98x0.95mm_HandSolder" V 6930 3650 50  0001 C CNN
@@
 AR Path="/609FED99/60ED6B0B" Ref="C?"  Part="1"
 AR Path="/60DF0860/60ED6B0B" Ref="C?"  Part="1"
-AR Path="/60DF07DE/60ED6B0B" Ref="C?"  Part="1"
+AR Path="/60DF07DE/60ED6B0B" Ref="C18"  Part="1"
 AR Path="/60F1863C/60ED6B0B" Ref="C?"  Part="1"
-F 0 "C?" H 3615 4096 50  0000 L CNN
+F 0 "C18" H 3615 4096 50  0000 L CNN
 F 1 "500" H 3615 4005 50  0000 L CNN
 F 2 "Capacitor_SMD:C_0603_1608Metric_Pad1.08x0.95mm_HandSolder" H 3538 3900 50  0001 C CNN
@@
 P 5650 3000
 AR Path="/60DF0860/60F18F15" Ref="L?"  Part="1"
-AR Path="/60DF07DE/60F18F15" Ref="L?"  Part="1"
+AR Path="/60DF07DE/60F18F15" Ref="L1"  Part="1"
 AR Path="/60F1863C/60F18F15" Ref="L?"  Part="1"
-F 0 "L?" V 5750 3000 50  0000 C CNN
+F 0 "L1" V 5750 3000 50  0000 C CNN
 F 1 "330u" V 5600 3000 50  0000 C CNN
 F 2 "" H 5650 3000 50  0001 C CNN
@@
 P 6350 3500
 AR Path="/60DF0860/60F18F16" Ref="D?"  Part="1"
-AR Path="/60DF07DE/60F18F16" Ref="D?"  Part="1"
+AR Path="/60DF07DE/60F18F16" Ref="D1"  Part="1"
 AR Path="/60F1863C/60F18F16" Ref="D?"  Part="1"
-F 0 "D?" H 6350 3400 50  0000 C CNN
+F 0 "D1" H 6350 3400 50  0000 C CNN
 F 1 "MBR0540" H 6300 3600 50  0000 C CNN
 F 2 "" H 6350 3500 50  0001 C CNN
@@
 P 7950 3500
 AR Path="/60DF0860/60F18F17" Ref="L?"  Part="1"
-AR Path="/60DF07DE/60F18F17" Ref="L?"  Part="1"
+AR Path="/60DF07DE/60F18F17" Ref="L2"  Part="1"
 AR Path="/60F1863C/60F18F17" Ref="L?"  Part="1"
-F 0 "L?" V 8050 3500 50  0000 C CNN
+F 0 "L2" V 8050 3500 50  0000 C CNN
 F 1 "330u" V 7900 3500 50  0000 C CNN
 F 2 "" H 7950 3500 50  0001 C CNN
@@
 P 9000 3650
 AR Path="/60DF0860/60F18F18" Ref="C?"  Part="1"
-AR Path="/60DF07DE/60F18F18" Ref="C?"  Part="1"
+AR Path="/60DF07DE/60F18F18" Ref="C21"  Part="1"
 AR Path="/60F1863C/60F18F18" Ref="C?"  Part="1"
-F 0 "C?" H 9118 3696 50  0000 L CNN
+F 0 "C21" H 9118 3696 50  0000 L CNN
 F 1 "470u" H 9118 3605 50  0000 L CNN
 F 2 "" H 9038 3500 50  0001 C CNN
@@
 AR Path="/609FED99/60F18F19" Ref="C?"  Part="1"
 AR Path="/60DF0860/60F18F19" Ref="C?"  Part="1"
-AR Path="/60DF07DE/60F18F19" Ref="C?"  Part="1"
+AR Path="/60DF07DE/60F18F19" Ref="C20"  Part="1"
 AR Path="/60F1863C/60F18F19" Ref="C?"  Part="1"
-F 0 "C?" H 8615 3696 50  0000 L CNN
+F 0 "C20" H 8615 3696 50  0000 L CNN
 F 1 "0,1" H 8615 3605 50  0000 L CNN
 F 2 "Capacitor_SMD:C_0603_1608Metric_Pad1.08x0.95mm_HandSolder" H 8538 3500 50  0001 C CNN
@@
 AR Path="/609FED99/60F18F1A" Ref="TP?"  Part="1"
 AR Path="/60DF0860/60F18F1A" Ref="TP?"  Part="1"
-AR Path="/60DF07DE/60F18F1A" Ref="TP?"  Part="1"
+AR Path="/60DF07DE/60F18F1A" Ref="TP8"  Part="1"
 AR Path="/60F1863C/60F18F1A" Ref="TP?"  Part="1"
-F 0 "TP?" H 10158 3618 50  0000 L CNN
+F 0 "TP8" H 10158 3618 50  0000 L CNN
 F 1 "TestPoint" H 10158 3527 50  0001 L CNN
 F 2 "" H 10300 3500 50  0001 C CNN
@@
 AR Path="/609FED99/60EE723F" Ref="TP?"  Part="1"
 AR Path="/60DF0860/60EE723F" Ref="TP?"  Part="1"
-AR Path="/60DF07DE/60EE723F" Ref="TP?"  Part="1"
+AR Path="/60DF07DE/60EE723F" Ref="TP7"  Part="1"
 AR Path="/60F1863C/60EE723F" Ref="TP?"  Part="1"
-F 0 "TP?" H 8158 4618 50  0000 L CNN
+F 0 "TP7" H 8158 4618 50  0000 L CNN
 F 1 "TestPoint" H 8158 4527 50  0001 L CNN
 F 2 "" H 8300 4500 50  0001 C CNN

Commit message: Add files via upload
Parts:
- C16, C19, C21: symbol Device:CP -> rata-rescue:CP-Device
- C17, C18, C20: symbol Device:C -> rata-rescue:C-Device
- D1: symbol Device:D_Schottky -> rata-rescue:D_Schottky-Device
- L1, L2: symbol Device:L -> rata-rescue:L-Device
- R10, R11, R8, R9: symbol Device:R -> rata-rescue:R-Device
- TP4, TP5, TP6, TP7, TP8: symbol Connector:TestPoint -> rata-rescue:TestPoint-Connector
- U4: symbol Regulator_Switching:MC34063AD -> rata-rescue:MC34063AD-Regulator_Switching
Changed lines of the file:
@@
 Boost converter +10V
 $Comp
-L Device:C C?
+L rata-rescue:C-Device C?
 U 1 1 60ED6AC7
 P 3000 3650
@@
 $EndComp
 $Comp
-L Device:R R?
+L rata-rescue:R-Device R?
 U 1 1 60ED6ACD
 P 4300 3000
@@
 $EndComp
 $Comp
-L Device:R R?
+L rata-rescue:R-Device R?
 U 1 1 60ED6AD3
 P 5250 3150
@@
 $EndComp
 $Comp
-L Connector:TestPoint TP?
+L rata-rescue:TestPoint-Connector TP?
 U 1 1 60ED6AD9
 P 7250 3500
@@
 $EndComp
 $Comp
-L Connector:TestPoint TP?
+L rata-rescue:TestPoint-Connector TP?
 U 1 1 60ED6ADF
 P 4600 3000
@@
 $EndComp
 $Comp
-L Device:CP C?
+L rata-rescue:CP-Device C?
 U 1 1 60F18F0E
 P 2500 3650
@@
 +5V_IN
 $Comp
-L Connector:TestPoint TP?
+L rata-rescue:TestPoint-Connector TP?
 U 1 1 60F18F0F
 P 4000 3000
@@
 GND
 $Comp
-L Device:R R?
+L rata-rescue:R-Device R?
 U 1 1 60ED6AF3
 P 7000 4150
@@
 $EndComp
 $Comp
-L Regulator_Switching:MC34063AD U?
+L rata-rescue:MC34063AD-Regulator_Switching U?
 U 1 1 60ED6AF9
 P 4300 3700
@@
 $EndComp
 $Comp
-L Device:CP C?
+L rata-rescue:CP-Device C?
 U 1 1 60F18F12
 P 7500 3650
@@
 $EndComp
 $Comp
-L Device:R R?
+L rata-rescue:R-Device R?
 U 1 1 60F18F13
 P 7000 3650
@@
 $EndComp
 $Comp
-L Device:C C?
+L rata-rescue:C-Device C?
 U 1 1 60ED6B0B
 P 3500 4050
@@
 $EndComp
 $Comp
-L Device:L L?
+L rata-rescue:L-Device L?
 U 1 1 60F18F15
 P 5650 3000
@@
 	7500 4500 7000 4500
 $Comp
-L Device:D_Schottky D?
+L rata-rescue:D_Schottky-Device D?
 U 1 1 60F18F16
 P 6350 3500
@@
 Connection ~ 7000 4500
 $Comp
-L Device:L L?
+L rata-rescue:L-Device L?
 U 1 1 60F18F17
 P 7950 3500
@@
 $EndComp
 $Comp
-L Device:CP C?
+L rata-rescue:CP-Device C?
 U 1 1 60F18F18
 P 9000 3650
@@
 $EndComp
 $Comp
-L Device:C C?
+L rata-rescue:C-Device C?
 U 1 1 60F18F19
 P 8500 3650
@@
 	8500 4500 8100 4500
 $Comp
-L Connector:TestPoint TP?
+L rata-rescue:TestPoint-Connector TP?
 U 1 1 60F18F1A
 P 10100 3500
@@
 	10100 3500 10500 3500
 $Comp
-L Connector:TestPoint TP?
+L rata-rescue:TestPoint-Connector TP?
 U 1 1 60EE723F
 P 8100 4500

Commit message: Add files via upload
Parts:
- C16: footprint (none) -> Capacitor_SMD:CP_Elec_6.3x7.7
- C19, C21: footprint (none) -> Capacitor_SMD:CP_Elec_10x10.5
- D1: footprint (none) -> Diode_SMD:D_SOD-123
- L1, L2: footprint (none) -> rata:L_12x12mm_H8mm
- R9: renamed from R8; footprint (none) -> Resistor_SMD:R_2010_5025Metric_Pad1.40x2.65mm_HandSolder
- TP4, TP5, TP6, TP7, TP8: footprint (none) -> rata:TP
- renumbered R9 to R10, R10 to R11, R11 to R12
Changed lines of the file:
@@
 encoding utf-8
 Sheet 6 23
-Title ""
-Date ""
-Rev ""
-Comp ""
+Title "rata"
+Date "2021-09-25"
+Rev "1.0"
+Comp "Yuriy Volkov"
 Comment1 ""
 Comment2 ""
@@
 AR Path="/609FED99/60ED6ACD" Ref="R?"  Part="1"
 AR Path="/60DF0860/60ED6ACD" Ref="R?"  Part="1"
-AR Path="/60DF07DE/60ED6ACD" Ref="R8"  Part="1"
+AR Path="/60DF07DE/60ED6ACD" Ref="R9"  Part="1"
 AR Path="/60F1863C/60ED6ACD" Ref="R?"  Part="1"
-F 0 "R8" V 4200 2950 50  0000 L CNN
+F 0 "R9" V 4200 2950 50  0000 L CNN
 F 1 "0,47 2010" V 4400 2800 50  0000 L CNN
-F 2 "" V 4230 3000 50  0001 C CNN
+F 2 "Resistor_SMD:R_2010_5025Metric_Pad1.40x2.65mm_HandSolder" V 4230 3000 50  0001 C CNN
 F 3 "~" H 4300 3000 50  0001 C CNN
 	1    4300 3000
@@
 AR Path="/609FED99/60ED6AD3" Ref="R?"  Part="1"
 AR Path="/60DF0860/60ED6AD3" Ref="R?"  Part="1"
-AR Path="/60DF07DE/60ED6AD3" Ref="R9"  Part="1"
+AR Path="/60DF07DE/60ED6AD3" Ref="R10"  Part="1"
 AR Path="/60F1863C/60ED6AD3" Ref="R?"  Part="1"
-F 0 "R9" H 5320 3196 50  0000 L CNN
+F 0 "R10" H 5320 3196 50  0000 L CNN
 F 1 "200" H 5320 3105 50  0000 L CNN
 F 2 "Resistor_SMD:R_0603_1608Metric_Pad0.98x0.95mm_HandSolder" V 5180 3150 50  0001 C CNN
@@
 F 0 "TP6" H 7308 3618 50  0000 L CNN
 F 1 "TestPoint" H 7308 3527 50  0001 L CNN
-F 2 "" H 7450 3500 50  0001 C CNN
+F 2 "rata:TP" H 7450 3500 50  0001 C CNN
 F 3 "~" H 7450 3500 50  0001 C CNN
 	1    7250 3500
@@
 F 0 "TP5" H 4658 3118 50  0000 L CNN
 F 1 "TestPoint" H 4658 3027 50  0001 L CNN
-F 2 "" H 4800 3000 50  0001 C CNN
+F 2 "rata:TP" H 4800 3000 50  0001 C CNN
 F 3 "~" H 4800 3000 50  0001 C CNN
 	1    4600 3000
@@
 F 0 "C16" H 2618 3696 50  0000 L CNN
 F 1 "100u" H 2618 3605 50  0000 L CNN
-F 2 "" H 2538 3500 50  0001 C CNN
+F 2 "Capacitor_SMD:CP_Elec_6.3x7.7" H 2538 3500 50  0001 C CNN
 F 3 "~" H 2500 3650 50  0001 C CNN
 	1    2500 3650
@@
 F 0 "TP4" H 4058 3118 50  0000 L CNN
 F 1 "TestPoint" H 4058 3027 50  0001 L CNN
-F 2 "" H 4200 3000 50  0001 C CNN
+F 2 "rata:TP" H 4200 3000 50  0001 C CNN
 F 3 "~" H 4200 3000 50  0001 C CNN
 	1    4000 3000
@@
 AR Path="/609FED99/60ED6AF3" Ref="R?"  Part="1"
 AR Path="/60DF0860/60ED6AF3" Ref="R?"  Part="1"
-AR Path="/60DF07DE/60ED6AF3" Ref="R11"  Part="1"
+AR Path="/60DF07DE/60ED6AF3" Ref="R12"  Part="1"
 AR Path="/60F1863C/60ED6AF3" Ref="R?"  Part="1"
-F 0 "R11" H 7070 4196 50  0000 L CNN
+F 0 "R12" H 7070 4196 50  0000 L CNN
 F 1 "2,4k 1%" H 7070 4105 50  0000 L CNN
 F 2 "Resistor_SMD:R_0603_1608Metric_Pad0.98x0.95mm_HandSolder" V 6930 4150 50  0001 C CNN
@@
 F 0 "C19" H 7618 3696 50  0000 L CNN
 F 1 "470u" H 7618 3605 50  0000 L CNN
-F 2 "" H 7538 3500 50  0001 C CNN
+F 2 "Capacitor_SMD:CP_Elec_10x10.5" H 7538 3500 50  0001 C CNN
 F 3 "~" H 7500 3650 50  0001 C CNN
 	1    7500 3650
@@
 AR Path="/609FED99/60F18F13" Ref="R?"  Part="1"
 AR Path="/60DF0860/60F18F13" Ref="R?"  Part="1"
-AR Path="/60DF07DE/60F18F13" Ref="R10"  Part="1"
+AR Path="/60DF07DE/60F18F13" Ref="R11"  Part="1"
 AR Path="/60F1863C/60F18F13" Ref="R?"  Part="1"
-F 0 "R10" H 7070 3696 50  0000 L CNN
+F 0 "R11" H 7070 3696 50  0000 L CNN
 F 1 "47k 1%" H 7070 3605 50  0000 L CNN
 F 2 "Resistor_SMD:R_0603_1608Metric_Pad0.98x0.95mm_HandSolder" V 6930 3650 50  0001 C CNN
@@
 F 0 "L1" V 5750 3000 50  0000 C CNN
 F 1 "330u" V 5600 3000 50  0000 C CNN
-F 2 "" H 5650 3000 50  0001 C CNN
+F 2 "rata:L_12x12mm_H8mm" H 5650 3000 50  0001 C CNN
 F 3 "~" H 5650 3000 50  0001 C CNN
 	1    5650 3000
@@
 F 0 "D1" H 6350 3400 50  0000 C CNN
 F 1 "MBR0540" H 6300 3600 50  0000 C CNN
-F 2 "" H 6350 3500 50  0001 C CNN
+F 2 "Diode_SMD:D_SOD-123" H 6350 3500 50  0001 C CNN
 F 3 "~" H 6350 3500 50  0001 C CNN
 	1    6350 3500
@@
 F 0 "L2" V 8050 3500 50  0000 C CNN
 F 1 "330u" V 7900 3500 50  0000 C CNN
-F 2 "" H 7950 3500 50  0001 C CNN
+F 2 "rata:L_12x12mm_H8mm" H 7950 3500 50  0001 C CNN
 F 3 "~" H 7950 3500 50  0001 C CNN
 	1    7950 3500
@@
 F 0 "C21" H 9118 3696 50  0000 L CNN
 F 1 "470u" H 9118 3605 50  0000 L CNN
-F 2 "" H 9038 3500 50  0001 C CNN
+F 2 "Capacitor_SMD:CP_Elec_10x10.5" H 9038 3500 50  0001 C CNN
 F 3 "~" H 9000 3650 50  0001 C CNN
 	1    9000 3650
@@
 F 0 "TP8" H 10158 3618 50  0000 L CNN
 F 1 "TestPoint" H 10158 3527 50  0001 L CNN
-F 2 "" H 10300 3500 50  0001 C CNN
+F 2 "rata:TP" H 10300 3500 50  0001 C CNN
 F 3 "~" H 10300 3500 50  0001 C CNN
 	1    10100 3500
@@
 F 0 "TP7" H 8158 4618 50  0000 L CNN
 F 1 "TestPoint" H 8158 4527 50  0001 L CNN
-F 2 "" H 8300 4500 50  0001 C CNN
+F 2 "rata:TP" H 8300 4500 50  0001 C CNN
 F 3 "~" H 8300 4500 50  0001 C CNN
 	1    8100 4500
@@
 	8100 4500 7500 4500
 Wire Wire Line
-	9000 3500 10100 3500
+	9000 3500 9500 3500
+$Comp
+L power:PWR_FLAG #FLG01
+U 1 1 615A73C8
+P 9500 3500
+F 0 "#FLG01" H 9500 3575 50  0001 C CNN
+F 1 "PWR_FLAG" H 9500 3673 50  0000 C CNN
+F 2 "" H 9500 3500 50  0001 C CNN
+F 3 "~" H 9500 3500 50  0001 C CNN
+	1    9500 3500
+	1    0    0    -1
+$EndComp
+Connection ~ 9500 3500
+Wire Wire Line
+	9500 3500 10100 3500
 $EndSCHEMATC

Commit message: Resistors values corrected to correspond actual values
Parts:
- R11: value 47k 1% -> 15k 1%
Changed lines of the file:
@@
 AR Path="/60F1863C/60F18F13" Ref="R?"  Part="1"
 F 0 "R11" H 7070 3696 50  0000 L CNN
-F 1 "47k 1%" H 7070 3605 50  0000 L CNN
+F 1 "15k 1%" H 7070 3605 50  0000 L CNN
 F 2 "Resistor_SMD:R_0603_1608Metric_Pad0.98x0.95mm_HandSolder" V 6930 3650 50  0001 C CNN
 F 3 "~" H 7000 3650 50  0001 C CNN
