File: Audio_amplifier.sch (KiCad schematic (older format))
At the start: 10 parts

Commit message: Add files via upload
Parts:
- removed C?: 0,1, Capacitor_SMD:C_0603_1608Metric_Pad1.08x0.95mm_HandSolder, symbol Device:C
- removed C?: 10u, Capacitor_SMD:C_1206_3216Metric_Pad1.33x1.80mm_HandSolder, symbol Device:C
- removed TP? (x2): TestPoint, symbol Connector:TestPoint
- added C?: 0,1, Capacitor_SMD:C_0603_1608Metric_Pad1.08x0.95mm_HandSolder, symbol Device:C
- added C?: 10u, Capacitor_SMD:C_1206_3216Metric_Pad1.33x1.80mm_HandSolder, symbol Device:C
- added TP? (x2): TestPoint, symbol Connector:TestPoint
Changed lines of the file:
@@
 $Descr A4 11693 8268
 encoding utf-8
-Sheet 5 11
+Sheet 8 15
 Title ""
 Date ""
@@
 AR Path="/60DF1072/60DF1215" Ref="U?"  Part="1"
 AR Path="/60DF1160/60DF1215" Ref="U?"  Part="1"
+AR Path="/60E72FD7/60DF1215" Ref="U?"  Part="1"
 F 0 "U?" H 6800 3742 50  0000 C CNN
 F 1 "AMS1117-3.3" H 6800 3651 50  0000 C CNN
@@
 AR Path="/60DF1072/60DF1216" Ref="C?"  Part="1"
 AR Path="/60DF1160/60DF1216" Ref="C?"  Part="1"
+AR Path="/60E72FD7/60DF1216" Ref="C?"  Part="1"
 F 0 "C?" H 7515 3696 50  0000 L CNN
 F 1 "10u" H 7515 3605 50  0000 L CNN
@@
 $Comp
 L Device:C C?
-U 1 1 60DF1217
+U 1 1 60EE8A0C
 P 6200 3650
-AR Path="/60DF1217" Ref="C?"  Part="1"
-AR Path="/609CA6A8/609D24C0/60DF1217" Ref="C?"  Part="1"
-AR Path="/609CA6A8/60A08E0B/60DF1217" Ref="C?"  Part="1"
-AR Path="/609CA6A8/60A0A46E/60DF1217" Ref="C?"  Part="1"
-AR Path="/609CA6A8/60A0A500/60DF1217" Ref="C?"  Part="1"
-AR Path="/609CA6A8/60A0A922/60DF1217" Ref="C?"  Part="1"
-AR Path="/609CA6A8/60DF1217" Ref="C?"  Part="1"
-AR Path="/609CA6A8/60AE5653/60DF1217" Ref="C?"  Part="1"
-AR Path="/609FED99/60DF1217" Ref="C?"  Part="1"
-AR Path="/60DF07DE/60DF1217" Ref="C?"  Part="1"
-AR Path="/60DF0860/60DF1217" Ref="C?"  Part="1"
-AR Path="/60DF1072/60DF1217" Ref="C?"  Part="1"
-AR Path="/60DF1160/60DF1217" Ref="C?"  Part="1"
+AR Path="/60EE8A0C" Ref="C?"  Part="1"
+AR Path="/609CA6A8/609D24C0/60EE8A0C" Ref="C?"  Part="1"
+AR Path="/609CA6A8/60A08E0B/60EE8A0C" Ref="C?"  Part="1"
+AR Path="/609CA6A8/60A0A46E/60EE8A0C" Ref="C?"  Part="1"
+AR Path="/609CA6A8/60A0A500/60EE8A0C" Ref="C?"  Part="1"
+AR Path="/609CA6A8/60A0A922/60EE8A0C" Ref="C?"  Part="1"
+AR Path="/609CA6A8/60EE8A0C" Ref="C?"  Part="1"
+AR Path="/609CA6A8/60AE5653/60EE8A0C" Ref="C?"  Part="1"
+AR Path="/609FED99/60EE8A0C" Ref="C?"  Part="1"
+AR Path="/60DF07DE/60EE8A0C" Ref="C?"  Part="1"
+AR Path="/60DF0860/60EE8A0C" Ref="C?"  Part="1"
+AR Path="/60DF1072/60EE8A0C" Ref="C?"  Part="1"
+AR Path="/60DF1160/60EE8A0C" Ref="C?"  Part="1"
+AR Path="/60E72FD7/60EE8A0C" Ref="C?"  Part="1"
 F 0 "C?" H 6315 3696 50  0000 L CNN
 F 1 "0,1" H 6315 3605 50  0000 L CNN
@@
 $Comp
 L Device:C C?
-U 1 1 60DF1218
+U 1 1 60EE8A0D
 P 7800 3650
-AR Path="/60DF1218" Ref="C?"  Part="1"
-AR Path="/609CA6A8/609D24C0/60DF1218" Ref="C?"  Part="1"
-AR Path="/609CA6A8/60A08E0B/60DF1218" Ref="C?"  Part="1"
-AR Path="/609CA6A8/60A0A46E/60DF1218" Ref="C?"  Part="1"
-AR Path="/609CA6A8/60A0A500/60DF1218" Ref="C?"  Part="1"
-AR Path="/609CA6A8/60A0A922/60DF1218" Ref="C?"  Part="1"
-AR Path="/609CA6A8/60DF1218" Ref="C?"  Part="1"
-AR Path="/609CA6A8/60AE5653/60DF1218" Ref="C?"  Part="1"
-AR Path="/609FED99/60DF1218" Ref="C?"  Part="1"
-AR Path="/60DF07DE/60DF1218" Ref="C?"  Part="1"
-AR Path="/60DF0860/60DF1218" Ref="C?"  Part="1"
-AR Path="/60DF1072/60DF1218" Ref="C?"  Part="1"
-AR Path="/60DF1160/60DF1218" Ref="C?"  Part="1"
+AR Path="/60EE8A0D" Ref="C?"  Part="1"
+AR Path="/609CA6A8/609D24C0/60EE8A0D" Ref="C?"  Part="1"
+AR Path="/609CA6A8/60A08E0B/60EE8A0D" Ref="C?"  Part="1"
+AR Path="/609CA6A8/60A0A46E/60EE8A0D" Ref="C?"  Part="1"
+AR Path="/609CA6A8/60A0A500/60EE8A0D" Ref="C?"  Part="1"
+AR Path="/609CA6A8/60A0A922/60EE8A0D" Ref="C?"  Part="1"
+AR Path="/609CA6A8/60EE8A0D" Ref="C?"  Part="1"
+AR Path="/609CA6A8/60AE5653/60EE8A0D" Ref="C?"  Part="1"
+AR Path="/609FED99/60EE8A0D" Ref="C?"  Part="1"
+AR Path="/60DF07DE/60EE8A0D" Ref="C?"  Part="1"
+AR Path="/60DF0860/60EE8A0D" Ref="C?"  Part="1"
+AR Path="/60DF1072/60EE8A0D" Ref="C?"  Part="1"
+AR Path="/60DF1160/60EE8A0D" Ref="C?"  Part="1"
+AR Path="/60E72FD7/60EE8A0D" Ref="C?"  Part="1"
 F 0 "C?" H 7915 3696 50  0000 L CNN
 F 1 "10u" H 7915 3605 50  0000 L CNN
@@
 $Comp
 L Connector:TestPoint TP?
-U 1 1 60DF1219
+U 1 1 60EE8A0E
 P 7550 3500
-AR Path="/60DF1219" Ref="TP?"  Part="1"
-AR Path="/609FED99/60DF1219" Ref="TP?"  Part="1"
-AR Path="/60DF07DE/60DF1219" Ref="TP?"  Part="1"
-AR Path="/60DF0860/60DF1219" Ref="TP?"  Part="1"
-AR Path="/60DF1072/60DF1219" Ref="TP?"  Part="1"
-AR Path="/60DF1160/60DF1219" Ref="TP?"  Part="1"
+AR Path="/60EE8A0E" Ref="TP?"  Part="1"
+AR Path="/609FED99/60EE8A0E" Ref="TP?"  Part="1"
+AR Path="/60DF07DE/60EE8A0E" Ref="TP?"  Part="1"
+AR Path="/60DF0860/60EE8A0E" Ref="TP?"  Part="1"
+AR Path="/60DF1072/60EE8A0E" Ref="TP?"  Part="1"
+AR Path="/60DF1160/60EE8A0E" Ref="TP?"  Part="1"
+AR Path="/60E72FD7/60EE8A0E" Ref="TP?"  Part="1"
 F 0 "TP?" H 7608 3618 50  0000 L CNN
 F 1 "TestPoint" H 7608 3527 50  0001 L CNN
@@
 AR Path="/60DF1072/60DF1213" Ref="TP?"  Part="1"
 AR Path="/60DF1160/60DF1213" Ref="TP?"  Part="1"
+AR Path="/60E72FD7/60DF1213" Ref="TP?"  Part="1"
 F 0 "TP?" H 5458 3618 50  0000 L CNN
 F 1 "TestPoint" H 5458 3527 50  0001 L CNN
@@
 AR Path="/60DF1072/60ACD247" Ref="C?"  Part="1"
 AR Path="/60DF1160/60ACD247" Ref="C?"  Part="1"
+AR Path="/60E72FD7/60ACD247" Ref="C?"  Part="1"
 F 0 "C?" H 4465 3696 50  0000 L CNN
 F 1 "1u" H 4465 3605 50  0000 L CNN
@@
 AR Path="/60DF1072/60DF19BB" Ref="D?"  Part="1"
 AR Path="/60DF1160/60DF19BB" Ref="D?"  Part="1"
+AR Path="/60E72FD7/60DF19BB" Ref="D?"  Part="1"
 F 0 "D?" V 4896 3570 50  0000 R CNN
 F 1 "SMAJ5.0CA" V 4805 3570 50  0000 R CNN
@@
 AR Path="/60DF1072/60DF121B" Ref="C?"  Part="1"
 AR Path="/60DF1160/60DF121B" Ref="C?"  Part="1"
+AR Path="/60E72FD7/60DF121B" Ref="C?"  Part="1"
 F 0 "C?" H 3918 3696 50  0000 L CNN
 F 1 "100u" H 3918 3605 50  0000 L CNN
@@
 $Comp
 L Connector:TestPoint TP?
-U 1 1 60DF121C
+U 1 1 60EE8A10
 P 5400 3800
-AR Path="/60DF121C" Ref="TP?"  Part="1"
-AR Path="/609FED99/60DF121C" Ref="TP?"  Part="1"
-AR Path="/60DF07DE/60DF121C" Ref="TP?"  Part="1"
-AR Path="/60DF0860/60DF121C" Ref="TP?"  Part="1"
-AR Path="/60DF1072/60DF121C" Ref="TP?"  Part="1"
-AR Path="/60DF1160/60DF121C" Ref="TP?"  Part="1"
+AR Path="/60EE8A10" Ref="TP?"  Part="1"
+AR Path="/609FED99/60EE8A10" Ref="TP?"  Part="1"
+AR Path="/60DF07DE/60EE8A10" Ref="TP?"  Part="1"
+AR Path="/60DF0860/60EE8A10" Ref="TP?"  Part="1"
+AR Path="/60DF1072/60EE8A10" Ref="TP?"  Part="1"
+AR Path="/60DF1160/60EE8A10" Ref="TP?"  Part="1"
+AR Path="/60E72FD7/60EE8A10" Ref="TP?"  Part="1"
 F 0 "TP?" H 5458 3918 50  0000 L CNN
 F 1 "TestPoint" H 5458 3827 50  0001 L CNN

Commit message: Add files via upload
Parts:
- removed C? (x2): 10u, Capacitor_SMD:C_1206_3216Metric_Pad1.33x1.80mm_HandSolder, symbol Device:C
- removed C?: 0,1, Capacitor_SMD:C_0603_1608Metric_Pad1.08x0.95mm_HandSolder, symbol Device:C
- removed D?: SMAJ5.0CA, symbol Device:D_TVS
- removed U?: AMS1117-3.3, Package_TO_SOT_SMD:SOT-223-3_TabPin2, symbol Regulator_Linear:AMS1117-3.3
- added C? (x2): 0,47, Capacitor_SMD:C_0603_1608Metric_Pad1.08x0.95mm_HandSolder, symbol Device:C
- added C? (x4): 1000, Capacitor_SMD:C_0603_1608Metric_Pad1.08x0.95mm_HandSolder, symbol Device:C
- added C? (x2): 0,1, Capacitor_SMD:C_0603_1608Metric_Pad1.08x0.95mm_HandSolder, symbol Device:C
- added C?: 100u, symbol Device:CP
- added C? (x3): 1u, Capacitor_SMD:C_0603_1608Metric_Pad1.08x0.95mm_HandSolder, symbol Device:C
- added FB? (x3): Ferrite_Bead, symbol Device:Ferrite_Bead
- added R?: 10, symbol Device:R
- added R? (x3): 100k, Resistor_SMD:R_0603_1608Metric_Pad0.98x0.95mm_HandSolder, symbol Device:R
- added R?: 20k, Resistor_SMD:R_0603_1608Metric_Pad0.98x0.95mm_HandSolder, symbol Device:R
- added R?: 1k, Resistor_SMD:R_0603_1608Metric_Pad0.98x0.95mm_HandSolder, symbol Device:R
- added U?: TPA3110D2, symbol rata:TPA3110D2
Connections:
- net labels added: +10V, AUD, SPK0, SPK1, ~DIS~
- net labels removed: +3V3_OUT, +5V_IN
- wire segments 18 -> 116
Other:
- note added: "D class audio amplifier"
- note removed: "Power source +3V3"
- moved on the sheet: C?, TP?

Commit message: Add files via upload
Parts:
- removed C?: 1u, Capacitor_SMD:C_0603_1608Metric_Pad1.08x0.95mm_HandSolder, symbol Device:C
- added C?: 1u, Capacitor_SMD:C_0603_1608Metric_Pad1.08x0.95mm_HandSolder, symbol Device:C
Connections:
- net GND: now also C?.2
- net at R?.2, U?.7 (AVCC): now also C?.1
Changed lines of the file:
@@
 $Descr A4 11693 8268
 encoding utf-8
-Sheet 8 20
+Sheet 8 24
 Title ""
 Date ""
@@
 $Comp
 L Device:C C?
-U 1 1 60ACD247
+U 1 1 60F5917C
 P 3000 3550
-AR Path="/60ACD247" Ref="C?"  Part="1"
-AR Path="/609CA6A8/609D24C0/60ACD247" Ref="C?"  Part="1"
-AR Path="/609CA6A8/60A08E0B/60ACD247" Ref="C?"  Part="1"
-AR Path="/609CA6A8/60A0A46E/60ACD247" Ref="C?"  Part="1"
-AR Path="/609CA6A8/60A0A500/60ACD247" Ref="C?"  Part="1"
-AR Path="/609CA6A8/60A0A922/60ACD247" Ref="C?"  Part="1"
-AR Path="/609CA6A8/60ACD247" Ref="C?"  Part="1"
-AR Path="/609CA6A8/60AE5653/60ACD247" Ref="C?"  Part="1"
-AR Path="/609FED99/60ACD247" Ref="C?"  Part="1"
-AR Path="/60DF07DE/60ACD247" Ref="C?"  Part="1"
-AR Path="/60DF0860/60ACD247" Ref="C?"  Part="1"
-AR Path="/60DF1072/60ACD247" Ref="C?"  Part="1"
-AR Path="/60DF1160/60ACD247" Ref="C?"  Part="1"
-AR Path="/60E72FD7/60ACD247" Ref="C?"  Part="1"
+AR Path="/60F5917C" Ref="C?"  Part="1"
+AR Path="/609CA6A8/609D24C0/60F5917C" Ref="C?"  Part="1"
+AR Path="/609CA6A8/60A08E0B/60F5917C" Ref="C?"  Part="1"
+AR Path="/609CA6A8/60A0A46E/60F5917C" Ref="C?"  Part="1"
+AR Path="/609CA6A8/60A0A500/60F5917C" Ref="C?"  Part="1"
+AR Path="/609CA6A8/60A0A922/60F5917C" Ref="C?"  Part="1"
+AR Path="/609CA6A8/60F5917C" Ref="C?"  Part="1"
+AR Path="/609CA6A8/60AE5653/60F5917C" Ref="C?"  Part="1"
+AR Path="/609FED99/60F5917C" Ref="C?"  Part="1"
+AR Path="/60DF07DE/60F5917C" Ref="C?"  Part="1"
+AR Path="/60DF0860/60F5917C" Ref="C?"  Part="1"
+AR Path="/60DF1072/60F5917C" Ref="C?"  Part="1"
+AR Path="/60DF1160/60F5917C" Ref="C?"  Part="1"
+AR Path="/60E72FD7/60F5917C" Ref="C?"  Part="1"
 F 0 "C?" H 3115 3596 50  0000 L CNN
 F 1 "1u" H 3115 3505 50  0000 L CNN

Commit message: Add files via upload
Connections:
- net GND: now also U?.3 (LINP), U?.4 (LINN)
Changed lines of the file:
@@
 	5750 4400 5900 4400
-Wire Wire Line
-	5750 4400 4500 4400
 Wire Wire Line
 	4500 4400 4500 5500
@@
 Wire Wire Line
 	7000 5500 9500 5500
+Wire Wire Line
+	5750 4400 5500 4400
+Wire Wire Line
+	5900 3900 5750 3900
+Wire Wire Line
+	5500 3900 5500 4400
+Connection ~ 5500 4400
+Wire Wire Line
+	5500 4400 4500 4400
+Wire Wire Line
+	5900 3800 5750 3800
+Wire Wire Line
+	5750 3800 5750 3900
+Connection ~ 5750 3900
+Wire Wire Line
+	5750 3900 5500 3900
 $EndSCHEMATC

Commit message: Add files via upload
Parts:
- gave numbers to parts that had none: 27
Connections:
- net +10V renamed +VCC

Commit message: Add files via upload
Parts:
- C26, C28, C29, C30, C31, C32, C34, C35, C36, C37, C38, C39: symbol Device:C -> rata-rescue:C-Device
- C27, C33: symbol Device:CP -> rata-rescue:CP-Device
- FB1, FB2, FB3: symbol Device:Ferrite_Bead -> rata-rescue:Ferrite_Bead-Device
- R16, R17, R18, R19, R20, R21: symbol Device:R -> rata-rescue:R-Device
- TP12, TP13, TP14: symbol Connector:TestPoint -> rata-rescue:TestPoint-Connector
Changed lines of the file:
@@
 $EndDescr
 $Comp
-L Connector:TestPoint TP?
+L rata-rescue:TestPoint-Connector TP?
 U 1 1 60EE8A0E
 P 10000 3000
@@
 $EndComp
 $Comp
-L Connector:TestPoint TP?
+L rata-rescue:TestPoint-Connector TP?
 U 1 1 60DF1213
 P 5500 3600
@@
 $EndComp
 $Comp
-L Device:C C?
+L rata-rescue:C-Device C?
 U 1 1 60F5917C
 P 3000 3550
@@
 $EndComp
 $Comp
-L Device:CP C?
+L rata-rescue:CP-Device C?
 U 1 1 60DF121B
 P 3500 2850
@@
 +VCC
 $Comp
-L Connector:TestPoint TP?
+L rata-rescue:TestPoint-Connector TP?
 U 1 1 60EE8A10
 P 9750 3000
@@
 $EndComp
 $Comp
-L Device:C C?
+L rata-rescue:C-Device C?
 U 1 1 60F0668E
 P 8000 4150
@@
 $EndComp
 $Comp
-L Device:C C?
+L rata-rescue:C-Device C?
 U 1 1 60F06990
 P 4500 2850
@@
 ~DIS~
 $Comp
-L Device:Ferrite_Bead FB3
+L rata-rescue:Ferrite_Bead-Device FB3
 U 1 1 60F08F65
 P 9150 4000
@@
 $EndComp
 $Comp
-L Device:Ferrite_Bead FB2
+L rata-rescue:Ferrite_Bead-Device FB2
 U 1 1 60F09757
 P 9150 3500
@@
 SPK1
 $Comp
-L Device:R R?
+L rata-rescue:R-Device R?
 U 1 1 60F0D5C7
 P 2350 3000
@@
 $EndComp
 $Comp
-L Device:R R?
+L rata-rescue:R-Device R?
 U 1 1 60F0D5D3
 P 2000 3650
@@
 $EndComp
 $Comp
-L Device:C C?
+L rata-rescue:C-Device C?
 U 1 1 60F17998
 P 4000 2850
@@
 $EndComp
 $Comp
-L Device:CP C?
+L rata-rescue:CP-Device C?
 U 1 1 60F1ACEF
 P 5500 2850
@@
 $EndComp
 $Comp
-L Device:C C?
+L rata-rescue:C-Device C?
 U 1 1 60F1ACF5
 P 6500 2850
@@
 $EndComp
 $Comp
-L Device:C C?
+L rata-rescue:C-Device C?
 U 1 1 60F1ACFB
 P 6000 2850
@@
 $EndComp
 $Comp
-L Device:Ferrite_Bead FB1
+L rata-rescue:Ferrite_Bead-Device FB1
 U 1 1 60F1C637
 P 1850 3000
@@
 $EndComp
 $Comp
-L Device:C C?
+L rata-rescue:C-Device C?
 U 1 1 60F23E88
 P 5000 4850
@@
 $EndComp
 $Comp
-L Device:C C?
+L rata-rescue:C-Device C?
 U 1 1 60F25535
 P 4500 3850
@@
 $EndComp
 $Comp
-L Device:C C?
+L rata-rescue:C-Device C?
 U 1 1 60F25FF4
 P 3850 3600
@@
 $EndComp
 $Comp
-L Device:R R?
+L rata-rescue:R-Device R?
 U 1 1 60F27980
 P 2500 3650
@@
 $EndComp
 $Comp
-L Device:C C?
+L rata-rescue:C-Device C?
 U 1 1 60F2BAB9
 P 8500 4150
@@
 $EndComp
 $Comp
-L Device:C C?
+L rata-rescue:C-Device C?
 U 1 1 60F2BCC3
 P 9500 4650
@@
 $EndComp
 $Comp
-L Device:C C?
+L rata-rescue:C-Device C?
 U 1 1 60F2BF71
 P 10000 4650
@@
 	3500 5500 4500 5500
 $Comp
-L Device:R R?
+L rata-rescue:R-Device R?
 U 1 1 60F43768
 P 5500 4850
@@
 $EndComp
 $Comp
-L Device:R R?
+L rata-rescue:R-Device R?
 U 1 1 60F43A7E
 P 5500 5250
@@
 	5750 4200 5900 4200
 $Comp
-L Device:R R?
+L rata-rescue:R-Device R?
 U 1 1 60F5E510
 P 1650 4500
