File: Audio_amplifier.sch (KiCad schematic (older format))
At the start: 27 parts, among them U6 TPA3110D2

Commit message: Add files via upload
Parts:
- C27, C33: footprint (none) -> Capacitor_SMD:CP_Elec_6.3x7.7
- FB1, FB2, FB3: footprint (none) -> Inductor_SMD:L_0805_2012Metric_Pad1.05x1.20mm_HandSolder
- R19: renamed from R18; footprint (none) -> Resistor_SMD:R_0805_2012Metric_Pad1.20x1.40mm_HandSolder
- TP12, TP13, TP14: footprint (none) -> rata:TP
- U6: footprint (none) -> Package_SO:HTSSOP-28-1EP_4.4x9.7mm_P0.65mm_EP3.4x9.5mm_ThermalVias
- renumbered R16 to R17, R17 to R18, R19 to R20, R20 to R21, R21 to R22
Changed lines of the file:
@@
 encoding utf-8
 Sheet 8 23
-Title ""
-Date ""
-Rev ""
-Comp ""
+Title "rata"
+Date "2021-09-25"
+Rev "1.0"
+Comp "Yuriy Volkov"
 Comment1 ""
 Comment2 ""
@@
 F 0 "TP14" H 10058 3118 50  0000 L CNN
 F 1 "TestPoint" H 10058 3027 50  0001 L CNN
-F 2 "" H 10200 3000 50  0001 C CNN
+F 2 "rata:TP" H 10200 3000 50  0001 C CNN
 F 3 "~" H 10200 3000 50  0001 C CNN
 	1    10000 3000
@@
 F 0 "TP12" H 5558 3718 50  0000 L CNN
 F 1 "TestPoint" H 5558 3627 50  0001 L CNN
-F 2 "" H 5700 3600 50  0001 C CNN
+F 2 "rata:TP" H 5700 3600 50  0001 C CNN
 F 3 "~" H 5700 3600 50  0001 C CNN
 	1    5500 3600
@@
 F 0 "C27" H 3618 2896 50  0000 L CNN
 F 1 "100u" H 3618 2805 50  0000 L CNN
-F 2 "" H 3538 2700 50  0001 C CNN
+F 2 "Capacitor_SMD:CP_Elec_6.3x7.7" H 3538 2700 50  0001 C CNN
 F 3 "~" H 3500 2850 50  0001 C CNN
 	1    3500 2850
@@
 F 0 "TP13" H 9808 3118 50  0000 L CNN
 F 1 "TestPoint" H 9808 3027 50  0001 L CNN
-F 2 "" H 9950 3000 50  0001 C CNN
+F 2 "rata:TP" H 9950 3000 50  0001 C CNN
 F 3 "~" H 9950 3000 50  0001 C CNN
 	1    9750 3000
@@
 F 0 "U6" H 7250 5250 50  0000 C CNN
 F 1 "TPA3110D2" H 7350 5150 50  0000 C CNN
-F 2 "" H 6900 3750 50  0001 C CNN
+F 2 "Package_SO:HTSSOP-28-1EP_4.4x9.7mm_P0.65mm_EP3.4x9.5mm_ThermalVias" H 6900 3750 50  0001 C CNN
 F 3 "" H 7200 5250 50  0001 C CNN
 	1    6800 4300
@@
 F 0 "FB3" V 8876 4000 50  0000 C CNN
 F 1 "Ferrite_Bead" V 8967 4000 50  0000 C CNN
-F 2 "" V 9080 4000 50  0001 C CNN
+F 2 "Inductor_SMD:L_0805_2012Metric_Pad1.05x1.20mm_HandSolder" V 9080 4000 50  0001 C CNN
 F 3 "~" H 9150 4000 50  0001 C CNN
 	1    9150 4000
@@
 F 0 "FB2" V 8876 3500 50  0000 C CNN
 F 1 "Ferrite_Bead" V 8967 3500 50  0000 C CNN
-F 2 "" V 9080 3500 50  0001 C CNN
+F 2 "Inductor_SMD:L_0805_2012Metric_Pad1.05x1.20mm_HandSolder" V 9080 3500 50  0001 C CNN
 F 3 "~" H 9150 3500 50  0001 C CNN
 	1    9150 3500
@@
 AR Path="/60EF6B1B/60F0D5C7" Ref="R?"  Part="1"
 AR Path="/60E72FD7/60F0D5C7" Ref="R?"  Part="1"
-AR Path="/60DF1072/60F0D5C7" Ref="R18"  Part="1"
-F 0 "R18" V 2450 2950 50  0000 L CNN
+AR Path="/60DF1072/60F0D5C7" Ref="R19"  Part="1"
+F 0 "R19" V 2450 2950 50  0000 L CNN
 F 1 "10" V 2250 2950 50  0000 L CNN
-F 2 "" V 2280 3000 50  0001 C CNN
+F 2 "Resistor_SMD:R_0805_2012Metric_Pad1.20x1.40mm_HandSolder" V 2280 3000 50  0001 C CNN
 F 3 "~" H 2350 3000 50  0001 C CNN
 	1    2350 3000
@@
 AR Path="/60EF6B1B/60F0D5D3" Ref="R?"  Part="1"
 AR Path="/60E72FD7/60F0D5D3" Ref="R?"  Part="1"
-AR Path="/60DF1072/60F0D5D3" Ref="R17"  Part="1"
-F 0 "R17" H 2070 3696 50  0000 L CNN
+AR Path="/60DF1072/60F0D5D3" Ref="R18"  Part="1"
+F 0 "R18" H 2070 3696 50  0000 L CNN
 F 1 "100k" H 2070 3605 50  0000 L CNN
 F 2 "Resistor_SMD:R_0603_1608Metric_Pad0.98x0.95mm_HandSolder" V 1930 3650 50  0001 C CNN
@@
 F 0 "C33" H 5618 2896 50  0000 L CNN
 F 1 "100u" H 5618 2805 50  0000 L CNN
-F 2 "" H 5538 2700 50  0001 C CNN
+F 2 "Capacitor_SMD:CP_Elec_6.3x7.7" H 5538 2700 50  0001 C CNN
 F 3 "~" H 5500 2850 50  0001 C CNN
 	1    5500 2850
@@
 F 0 "FB1" V 1576 3000 50  0000 C CNN
 F 1 "Ferrite_Bead" V 1667 3000 50  0000 C CNN
-F 2 "" V 1780 3000 50  0001 C CNN
+F 2 "Inductor_SMD:L_0805_2012Metric_Pad1.05x1.20mm_HandSolder" V 1780 3000 50  0001 C CNN
 F 3 "~" H 1850 3000 50  0001 C CNN
 	1    1850 3000
@@
 AR Path="/60EF6B1B/60F27980" Ref="R?"  Part="1"
 AR Path="/60E72FD7/60F27980" Ref="R?"  Part="1"
-AR Path="/60DF1072/60F27980" Ref="R19"  Part="1"
-F 0 "R19" H 2570 3696 50  0000 L CNN
+AR Path="/60DF1072/60F27980" Ref="R20"  Part="1"
+F 0 "R20" H 2570 3696 50  0000 L CNN
 F 1 "100k" H 2570 3605 50  0000 L CNN
 F 2 "Resistor_SMD:R_0603_1608Metric_Pad0.98x0.95mm_HandSolder" V 2430 3650 50  0001 C CNN
@@
 AR Path="/60EF6B1B/60F43768" Ref="R?"  Part="1"
 AR Path="/60E72FD7/60F43768" Ref="R?"  Part="1"
-AR Path="/60DF1072/60F43768" Ref="R20"  Part="1"
-F 0 "R20" H 5570 4896 50  0000 L CNN
+AR Path="/60DF1072/60F43768" Ref="R21"  Part="1"
+F 0 "R21" H 5570 4896 50  0000 L CNN
 F 1 "100k" H 5570 4805 50  0000 L CNN
 F 2 "Resistor_SMD:R_0603_1608Metric_Pad0.98x0.95mm_HandSolder" V 5430 4850 50  0001 C CNN
@@
 AR Path="/60EF6B1B/60F43A7E" Ref="R?"  Part="1"
 AR Path="/60E72FD7/60F43A7E" Ref="R?"  Part="1"
-AR Path="/60DF1072/60F43A7E" Ref="R21"  Part="1"
-F 0 "R21" H 5570 5296 50  0000 L CNN
+AR Path="/60DF1072/60F43A7E" Ref="R22"  Part="1"
+F 0 "R22" H 5570 5296 50  0000 L CNN
 F 1 "20k" H 5570 5205 50  0000 L CNN
 F 2 "Resistor_SMD:R_0603_1608Metric_Pad0.98x0.95mm_HandSolder" V 5430 5250 50  0001 C CNN
@@
 	3000 3400 3000 3000
 Wire Wire Line
-	3000 3000 2500 3000
+	3000 3000 2750 3000
 Connection ~ 3000 3400
 Wire Wire Line
@@
 AR Path="/60EF6B1B/60F5E510" Ref="R?"  Part="1"
 AR Path="/60E72FD7/60F5E510" Ref="R?"  Part="1"
-AR Path="/60DF1072/60F5E510" Ref="R16"  Part="1"
-F 0 "R16" V 1750 4450 50  0000 L CNN
+AR Path="/60DF1072/60F5E510" Ref="R17"  Part="1"
+F 0 "R17" V 1750 4450 50  0000 L CNN
 F 1 "1k" V 1550 4450 50  0000 L CNN
 F 2 "Resistor_SMD:R_0603_1608Metric_Pad0.98x0.95mm_HandSolder" V 1580 4500 50  0001 C CNN
@@
 Wire Wire Line
 	5750 3900 5500 3900
+$Comp
+L power:PWR_FLAG #FLG03
+U 1 1 615AFCE5
+P 2750 3000
+F 0 "#FLG03" H 2750 3075 50  0001 C CNN
+F 1 "PWR_FLAG" H 2750 3173 50  0000 C CNN
+F 2 "" H 2750 3000 50  0001 C CNN
+F 3 "~" H 2750 3000 50  0001 C CNN
+	1    2750 3000
+	1    0    0    -1
+$EndComp
+Connection ~ 2750 3000
+Wire Wire Line
+	2750 3000 2500 3000
 $EndSCHEMATC
