File: rata.sch (KiCad schematic (older format))
At the start: 0 parts

Commit message: Add files via upload
Other:
- note added: "Clock"
- note removed: "Controller"
Changed lines of the file:
@@
 $Descr A4 11693 8268
 encoding utf-8
-Sheet 1 11
+Sheet 1 15
 Title ""
 Date ""
@@
 $EndSheet
 $Sheet
-S 8000 6000 1000 500
+S 2500 5000 1000 750
 U 60B1951B
 F0 "MICRO_SD_CARD" 50
 F1 "Micro_SD_card.sch" 50
-F2 "~CS~" I L 8000 6100 50
-F3 "MOSI" I L 8000 6300 50
-F4 "SCK" I L 8000 6200 50
-F5 "MISO" O L 8000 6400 50
+F2 "~CS~" I L 2500 5200 50
+F3 "MOSI" I L 2500 5400 50
+F4 "SCK" I L 2500 5300 50
+F5 "MISO" O L 2500 5500 50
+F6 "+3V3" I L 2500 5050 50
+F7 "GND" I L 2500 5650 50
 $EndSheet
 $Sheet
-S 8000 5000 1000 500
+S 1000 2500 1000 500
 U 60B39FE1
 F0 "BUZZER" 50
 F1 "Buzzer.sch" 50
-F2 "EN" I L 8000 5250 50
+F2 "EN" I L 1000 2750 50
+F3 "+5V" I L 1000 2600 50
+F4 "GND" I L 1000 2900 50
 $EndSheet
 Text Notes 6750 1050 2    197  ~ 0
-Controller
+Clock
 $Sheet
-S 5500 1500 1000 500
+S 1000 3500 1000 500
 U 609FED99
-F0 "POWER_+3V3" 50
+F0 "+3V3" 50
 F1 "Power_+3V3.sch" 50
-F2 "+5V_IN" I L 5500 1600 50
-F3 "GND" I L 5500 1900 50
-F4 "+3V3_OUT" O R 6500 1600 50
+F2 "+5V_IN" I L 1000 3600 50
+F3 "GND" I L 1000 3900 50
+F4 "+3V3_OUT" O R 2000 3600 50
 $EndSheet
 $Sheet
-S 9000 1500 1000 500
+S 2500 1500 1000 500
 U 60DF07DE
-F0 "POWER_+10V" 50
+F0 "+10V" 50
 F1 "Power_+10V.sch" 50
-F2 "CHARGE_PUMP_CLK" I L 9000 1900 50
-F3 "+5V_IN" I L 9000 1600 50
-F4 "GND_IN" I L 9000 1700 50
+F2 "+5V_IN" I L 2500 1600 50
+F3 "+10V_OUT" O R 3500 1600 50
+F4 "GND" I L 2500 1900 50
 $EndSheet
 $Sheet
-S 9000 2500 1000 500
+S 1000 1500 1000 500
 U 60DF0860
-F0 "POWER_+25V" 50
+F0 "+25V" 50
 F1 "Power_+25V.sch" 50
-F2 "CHARGE_PUMP_CLK" I L 9000 2900 50
-F3 "+5V_IN" I L 9000 2600 50
-F4 "GND_IN" I L 9000 2700 50
+F2 "+5V_IN" I L 1000 1600 50
+F3 "+25V_OUT" O R 2000 1600 50
+F4 "GND" I L 1000 1900 50
 $EndSheet
 $Sheet
@@
 $EndSheet
 $Sheet
-S 2500 2000 1000 500
+S 9000 3500 1000 500
 U 60DF196E
 F0 "BUTTONS" 50
 F1 "Buttons.sch" 50
-F2 "CHARGE_PUMP_CLK" I L 2500 2400 50
-F3 "+5V_IN" I L 2500 2100 50
-F4 "GND_IN" I L 2500 2200 50
+F2 "CHARGE_PUMP_CLK" I L 9000 3900 50
+F3 "+5V_IN" I L 9000 3600 50
+F4 "GND_IN" I L 9000 3700 50
 $EndSheet
 $Sheet
-S 2500 3000 1000 500
+S 9000 4500 1000 500
 U 60DF212D
 F0 "SWITCH" 50
 F1 "Switch.sch" 50
-F2 "CHARGE_PUMP_CLK" I L 2500 3400 50
-F3 "+5V_IN" I L 2500 3100 50
-F4 "GND_IN" I L 2500 3200 50
+F2 "CHARGE_PUMP_CLK" I L 9000 4900 50
+F3 "+5V_IN" I L 9000 4600 50
+F4 "GND_IN" I L 9000 4700 50
+$EndSheet
+$Sheet
+S 1000 4500 1000 500
+U 60E6F2E9
+F0 "+3V3A" 50
+F1 "Power_+3V3.sch" 50
+F2 "+5V_IN" I L 1000 4600 50
+F3 "GND" I L 1000 4900 50
+F4 "+3V3_OUT" O R 2000 4600 50
+$EndSheet
+$Sheet
+S 7500 2000 1000 500
+U 60E72FD7
+F0 "DAC" 50
+F1 "DAC.sch" 50
+F2 "CHARGE_PUMP_CLK" I L 7500 2400 50
+F3 "+5V_IN" I L 7500 2100 50
+F4 "GND_IN" I L 7500 2200 50
+$EndSheet
+$Sheet
+S 2500 2500 1000 1000
+U 60EE89A9
+F0 "USB" 50
+F1 "USB.sch" 50
+F2 "VBUS" I L 2500 2600 50
+F3 "GND" I L 2500 3400 50
+F4 "D-" I L 2500 3100 50
+F5 "D+" I L 2500 3200 50
+F6 "USBDM" O R 3500 3100 50
+F7 "USBDP" O R 3500 3200 50
+F8 "+5V" O R 3500 2600 50
+F9 "USB_ON" I R 3500 2850 50
+F10 "+3V3_IN" I R 3500 2750 50
+$EndSheet
+$Sheet
+S 2500 4000 1000 500
+U 60EF6B1B
+F0 "RTC" 50
+F1 "RTC.sch" 50
+F2 "+3V3" I L 2500 4100 50
+F3 "GND" I L 2500 4400 50
+F4 "SDA" B L 2500 4300 50
+F5 "SCK" I L 2500 4200 50
 $EndSheet
 $EndSCHEMATC

Commit message: Add files via upload
Changed lines of the file:
@@
 $EndSheet
 $Sheet
-S 7500 3000 1000 500
+S 2500 6000 1000 500
 U 60DF1072
 F0 "AUDIO_AMPLIFIER" 50
 F1 "Audio_amplifier.sch" 50
-F2 "CHARGE_PUMP_CLK" I L 7500 3400 50
-F3 "+5V_IN" I L 7500 3100 50
-F4 "GND_IN" I L 7500 3200 50
+F2 "+10V" I L 2500 6100 50
+F3 "GND" I L 2500 6400 50
+F4 "SPK0" O R 3500 6100 50
+F5 "AUD" I L 2500 6200 50
+F6 "~DIS~" I L 2500 6300 50
+F7 "SPK1" O R 3500 6400 50
 $EndSheet
 $Sheet
@@
 $EndSheet
 $Sheet
-S 7500 2000 1000 500
+S 1000 5500 1000 500
 U 60E72FD7
 F0 "DAC" 50
 F1 "DAC.sch" 50
-F2 "CHARGE_PUMP_CLK" I L 7500 2400 50
-F3 "+5V_IN" I L 7500 2100 50
-F4 "GND_IN" I L 7500 2200 50
+F2 "AUD" O R 2000 5750 50
+F3 "+3V3" I L 1000 5600 50
+F4 "GND" I L 1000 5900 50
+F5 "SDA" B L 1000 5800 50
+F6 "SCK" I L 1000 5700 50
 $EndSheet
 $Sheet

Commit message: Add files via upload
Changed lines of the file:
@@
 $Descr A4 11693 8268
 encoding utf-8
-Sheet 1 15
+Sheet 1 20
 Title ""
 Date ""
@@
 F5 "SCK" I L 2500 4200 50
 $EndSheet
+$Sheet
+S 7500 3000 1000 500
+U 60F1863C
+F0 "+4V5" 50
+F1 "Power_+4.5V.sch" 50
+F2 "+5V_IN" I L 7500 3100 50
+F3 "+10V_OUT" O R 8500 3100 50
+F4 "GND" I L 7500 3400 50
+$EndSheet
+$Sheet
+S 7500 5000 1000 500
+U 60F18EC1
+F0 "VLD_HEATER" 50
+F1 "VLD_heater.sch" 50
+F2 "CHARGE_PUMP_CLK" I L 7500 5400 50
+F3 "+5V_IN" I L 7500 5100 50
+F4 "GND_IN" I L 7500 5200 50
+$EndSheet
+$Sheet
+S 9000 5500 1000 500
+U 60F197D4
+F0 "LIGHT_SENSOR" 50
+F1 "Light_sensor.sch" 50
+F2 "CHARGE_PUMP_CLK" I L 9000 5900 50
+F3 "+5V_IN" I L 9000 5600 50
+F4 "GND_IN" I L 9000 5700 50
+$EndSheet
+$Sheet
+S 7500 6000 1000 500
+U 60F1A0E6
+F0 "TEMP_SENSOR" 50
+F1 "Temp_sensor.sch" 50
+F2 "CHARGE_PUMP_CLK" I L 7500 6400 50
+F3 "+5V_IN" I L 7500 6100 50
+F4 "GND_IN" I L 7500 6200 50
+$EndSheet
 $EndSCHEMATC

Commit message: Add files via upload
Changed lines of the file:
@@
 $Descr A4 11693 8268
 encoding utf-8
-Sheet 1 20
+Sheet 1 24
 Title ""
 Date ""
@@
 $EndSheet
 $Sheet
-S 9000 3500 1000 500
+S 5500 1500 1000 500
 U 60DF196E
 F0 "BUTTONS" 50
 F1 "Buttons.sch" 50
-F2 "CHARGE_PUMP_CLK" I L 9000 3900 50
-F3 "+5V_IN" I L 9000 3600 50
-F4 "GND_IN" I L 9000 3700 50
+F2 "+3V3" I L 5500 1600 50
+F3 "COL0" O R 6500 1700 50
+F4 "ROW0" I L 5500 1700 50
+F5 "ROW1" I L 5500 1800 50
+F6 "ROW2" I L 5500 1900 50
+F7 "COL1" O R 6500 1800 50
+F8 "COL2" O R 6500 1900 50
 $EndSheet
 $Sheet
@@
 $EndSheet
 $Sheet
-S 7500 3000 1000 500
+S 4000 1500 1000 500
 U 60F1863C
 F0 "+4V5" 50
 F1 "Power_+4.5V.sch" 50
-F2 "+5V_IN" I L 7500 3100 50
-F3 "+10V_OUT" O R 8500 3100 50
-F4 "GND" I L 7500 3400 50
-$EndSheet
-$Sheet
-S 7500 5000 1000 500
+F2 "+5V_IN" I L 4000 1600 50
+F3 "GND" I L 4000 1900 50
+F4 "+4V5_OUT" O R 5000 1600 50
+F5 "SD" I L 4000 1750 50
+F6 "VOLT" O R 5000 1750 50
+$EndSheet
+$Sheet
+S 4000 5500 1000 1000
 U 60F18EC1
 F0 "VLD_HEATER" 50
 F1 "VLD_heater.sch" 50
-F2 "CHARGE_PUMP_CLK" I L 7500 5400 50
-F3 "+5V_IN" I L 7500 5100 50
-F4 "GND_IN" I L 7500 5200 50
-$EndSheet
-$Sheet
-S 9000 5500 1000 500
+F2 "+VDD" I L 4000 5600 50
+F3 "GND" I L 4000 6400 50
+F4 "OUT0" O R 5000 5750 50
+F5 "OUT1" O R 5000 6200 50
+F6 "IN0N" I L 4000 5900 50
+F7 "IN0P" I L 4000 5800 50
+F8 "IN1N" I L 4000 6200 50
+F9 "IN1P" I L 4000 6100 50
+$EndSheet
+$Sheet
+S 5500 6500 1000 500
 U 60F197D4
 F0 "LIGHT_SENSOR" 50
 F1 "Light_sensor.sch" 50
-F2 "CHARGE_PUMP_CLK" I L 9000 5900 50
-F3 "+5V_IN" I L 9000 5600 50
-F4 "GND_IN" I L 9000 5700 50
-$EndSheet
-$Sheet
-S 7500 6000 1000 500
+F2 "+3V3" I L 5500 6600 50
+F3 "GND" I L 5500 6900 50
+F4 "VOLT" O R 6500 6600 50
+$EndSheet
+$Sheet
+S 2500 7000 1000 500
 U 60F1A0E6
 F0 "TEMP_SENSOR" 50
 F1 "Temp_sensor.sch" 50
-F2 "CHARGE_PUMP_CLK" I L 7500 6400 50
-F3 "+5V_IN" I L 7500 6100 50
-F4 "GND_IN" I L 7500 6200 50
+F2 "+3V3" I L 2500 7100 50
+F3 "GND" I L 2500 7400 50
+F4 "+3V3A" I L 2500 7200 50
+F5 "SDA" B R 3500 7300 50
+F6 "SCK" I R 3500 7200 50
 $EndSheet
 $EndSCHEMATC

Commit message: Add files via upload
Changed lines of the file:
@@
 $Descr A4 11693 8268
 encoding utf-8
-Sheet 1 24
+Sheet 1 23
 Title ""
 Date ""
@@
 $EndDescr
 $Sheet
-S 5000 3000 1500 2000
+S 8000 1500 1500 2000
 U 609C9D41
 F0 "MCU" 50
 F1 "MCU.sch" 50
-F2 "DPY_PWR_EN" O R 6500 3500 50
-F3 "~DPY_RST" O R 6500 3600 50
-F4 "DPY_I2C_SDA" B R 6500 3800 50
-F5 "DPY_I2C_SCK" O R 6500 3700 50
-F6 "CHARGE_PUMP_CLK" O R 6500 3300 50
-F7 "KYBD" B R 6500 4000 50
-F8 "TEMP_SPI_MISO" I L 5000 3500 50
-F9 "TEMP_SPI_SCK" O L 5000 3400 50
-F10 "~TEMP_SPI_CS" O L 5000 3300 50
-F11 "BZ_EN" O R 6500 4200 50
-F12 "~SD_SPI_CS" O R 6500 4400 50
-F13 "SD_SPI_MOSI" O R 6500 4600 50
-F14 "SD_SPI_SCK" O R 6500 4500 50
-F15 "SD_SPI_MISO" I R 6500 4700 50
-F16 "EXT_UART_RX" I L 5000 3100 50
-F17 "HEATER_CTRL" O R 6500 3100 50
+F2 "DPY_PWR_EN" O R 9500 2000 50
+F3 "~DPY_RST" O R 9500 2100 50
+F4 "DPY_I2C_SDA" B R 9500 2300 50
+F5 "DPY_I2C_SCK" O R 9500 2200 50
+F6 "CHARGE_PUMP_CLK" O R 9500 1800 50
+F7 "KYBD" B R 9500 2500 50
+F8 "TEMP_SPI_MISO" I L 8000 2000 50
+F9 "TEMP_SPI_SCK" O L 8000 1900 50
+F10 "~TEMP_SPI_CS" O L 8000 1800 50
+F11 "BZ_EN" O R 9500 2700 50
+F12 "~SD_SPI_CS" O R 9500 2900 50
+F13 "SD_SPI_MOSI" O R 9500 3100 50
+F14 "SD_SPI_SCK" O R 9500 3000 50
+F15 "SD_SPI_MISO" I R 9500 3200 50
+F16 "EXT_UART_RX" I L 8000 1600 50
+F17 "HEATER_CTRL" O R 9500 1600 50
 $EndSheet
 $Sheet
@@
 $EndSheet
 $Sheet
-S 9000 4500 1000 500
+S 5500 5500 1000 500
 U 60DF212D
-F0 "SWITCH" 50
+F0 "ALARM_SW" 50
 F1 "Switch.sch" 50
-F2 "CHARGE_PUMP_CLK" I L 9000 4900 50
-F3 "+5V_IN" I L 9000 4600 50
-F4 "GND_IN" I L 9000 4700 50
+F2 "+3V3" I L 5500 5600 50
+F3 "GND" I L 5500 5900 50
+F4 "ALARM" O R 6500 5600 50
 $EndSheet
 $Sheet

Commit message: Add files via upload
Parts:
- added J?: USB_B, symbol Connector:USB_B
- added U?: ILC4-5_7L, symbol rata:ILC4-5_7L

Commit message: Add files via upload
Parts:
- added F1: Fuse, symbol Device:Fuse
- added J2: Soldering points, symbol Connector:Screw_Terminal_01x02
- gave numbers to parts that had none: 2
Connections:
- net AUDIO_AMPLIFIER/SPK0: now also J2.1 (Pin_1)
- net AUDIO_AMPLIFIER/SPK1: now also J2.2 (Pin_2)
- net USB/D+: now also J1.3 (D+)
- net USB/D-: now also J1.2 (D-)
- net USB/VBUS: now also F1.1
- net VFD_HEATER/OUT0: now also U1.1
- net VFD_HEATER/OUT1: now also U1.16
- net VFD8: now reaches U1.10 (DP)
- net VFD9: now reaches U1.11 (G1)
- net VFD10: now reaches U1.12 (B)
- net VFD11: now reaches U1.13 (F)
- net VFD12: now reaches U1.14 (G0)
- net VFD13: now reaches U1.15 (A)
- net VFD0: now reaches U1.2 (BL)
- net VFD1: now reaches U1.3 (G4)
- net VFD2: now reaches U1.4 (G)
- net VFD3: now reaches U1.5 (E)
- net VFD4: now reaches U1.6 (G3)
- net VFD5: now reaches U1.7 (C)
- net VFD6: now reaches U1.8 (D)
- net VFD7: now reaches U1.9 (G2)
- net at J1.1 (VBUS): now also F1.2
- net GND: now reaches J1.4 (GND)
- net GND: now also J1.5 (Shield)
Other:
- note added: "Speaker connection"
- moved on the sheet: J1, U1

Commit message: Add files via upload
Parts:
- F1: symbol Device:Fuse -> rata-rescue:Fuse-Device
- J1: symbol Connector:USB_B -> rata-rescue:USB_B-Connector
- J2: symbol Connector:Screw_Terminal_01x02 -> rata-rescue:Screw_Terminal_01x02-Connector
Changed lines of the file:
@@
 $EndSheet
 $Sheet
-S 4000 6500 1000 500
+S 1000 7000 1000 500
 U 60F1863C
 F0 "+4V5" 50
 F1 "Power_+4.5V.sch" 50
-F2 "+5V_IN" I L 4000 6600 50
-F3 "GND" I L 4000 6900 50
-F4 "+4V5_OUT" O R 5000 6600 50
-F5 "SD" I L 4000 6750 50
-F6 "VOLT" O R 5000 6750 50
+F2 "+5V_IN" I L 1000 7100 50
+F3 "GND" I L 1000 7400 50
+F4 "+4V5_OUT" O R 2000 7100 50
+F5 "SD" I L 1000 7250 50
+F6 "VOLT" O R 2000 7250 50
 $EndSheet
 $Sheet
@@
 $EndSheet
 $Comp
-L rata:ILC4-5_7L U1
-U 1 1 60FA6693
-P 8700 2300
-F 0 "U1" H 10200 2850 50  0000 L CNN
-F 1 "ILC4-5_7L" H 10100 2750 50  0000 L CNN
-F 2 "" H 8700 1750 50  0001 C CNN
-F 3 "" V 8850 2900 50  0001 C CNN
-	1    8700 2300
-	1    0    0    -1
-$EndComp
-$Comp
-L Connector:USB_B J1
+L rata-rescue:USB_B-Connector J1
 U 1 1 60FC5AE8
 P 1200 1500
@@
 $EndComp
 $Comp
-L Connector:Screw_Terminal_01x02 J2
+L rata-rescue:Screw_Terminal_01x02-Connector J2
 U 1 1 60FB3338
 P 10200 4600
@@
 $EndComp
 $Comp
-L power:+3V3 #PWR010
+L rata-rescue:+3V3-power #PWR010
 U 1 1 60FC0590
 P 2100 3100
@@
 $EndComp
 $Comp
-L power:+10V #PWR012
+L rata-rescue:+10V-power #PWR012
 U 1 1 60FC0B0A
 P 2100 5100
@@
 $EndComp
 $Comp
-L power:GND #PWR09
+L rata-rescue:GND-power #PWR09
 U 1 1 60FC1D65
 P 1500 2100
@@
 	1200 2100 1100 2100
 $Comp
-L power:+5V #PWR021
+L rata-rescue:+5V-power #PWR021
 U 1 1 60FC4261
 P 3100 1300
@@
 L rata:+4V5 #PWR028
 U 1 1 60FC6F1D
-P 5100 6600
-F 0 "#PWR028" H 5100 6450 50  0001 C CNN
-F 1 "+4V5" H 5050 6800 50  0000 C CNN
-F 2 "" H 5100 6600 50  0001 C CNN
-F 3 "" H 5100 6600 50  0001 C CNN
-	1    5100 6600
+P 2100 7100
+F 0 "#PWR028" H 2100 6950 50  0001 C CNN
+F 1 "+4V5" H 2050 7300 50  0000 C CNN
+F 2 "" H 2100 7100 50  0001 C CNN
+F 3 "" H 2100 7100 50  0001 C CNN
+	1    2100 7100
 	1    0    0    -1
 $EndComp
@@
 $EndComp
 $Comp
-L power:+5V #PWR01
+L rata-rescue:+5V-power #PWR01
 U 1 1 60FC86FF
 P 900 3100
@@
 $EndComp
 $Comp
-L power:+5V #PWR03
+L rata-rescue:+5V-power #PWR03
 U 1 1 60FC8CAF
 P 900 4100
@@
 $EndComp
 $Comp
-L power:+5V #PWR023
+L rata-rescue:+5V-power #PWR023
 U 1 1 60FC9068
-P 3900 6600
-F 0 "#PWR023" H 3900 6450 50  0001 C CNN
-F 1 "+5V" H 3915 6773 50  0000 C CNN
-F 2 "" H 3900 6600 50  0001 C CNN
-F 3 "" H 3900 6600 50  0001 C CNN
-	1    3900 6600
-	1    0    0    -1
-$EndComp
-$Comp
-L power:+5V #PWR05
+P 900 7100
+F 0 "#PWR023" H 900 6950 50  0001 C CNN
+F 1 "+5V" H 915 7273 50  0000 C CNN
+F 2 "" H 900 7100 50  0001 C CNN
+F 3 "" H 900 7100 50  0001 C CNN
+	1    900  7100
+	1    0    0    -1
+$EndComp
+$Comp
+L rata-rescue:+5V-power #PWR05
 U 1 1 60FC94EE
 P 900 5100
@@
 $EndComp
 $Comp
-L power:+5V #PWR07
+L rata-rescue:+5V-power #PWR07
 U 1 1 60FC9834
 P 900 6100
@@
 $EndComp
 $Comp
-L power:GND #PWR02
+L rata-rescue:GND-power #PWR02
 U 1 1 60FCCF66
 P 900 3400
@@
 $EndComp
 $Comp
-L power:GND #PWR04
+L rata-rescue:GND-power #PWR04
 U 1 1 60FCD057
 P 900 4400
@@
 $EndComp
 $Comp
-L power:GND #PWR024
+L rata-rescue:GND-power #PWR024
 U 1 1 60FCD246
-P 3900 6900
-F 0 "#PWR024" H 3900 6650 50  0001 C CNN
-F 1 "GND" H 3905 6727 50  0000 C CNN
-F 2 "" H 3900 6900 50  0001 C CNN
-F 3 "" H 3900 6900 50  0001 C CNN
-	1    3900 6900
-	1    0    0    -1
-$EndComp
-$Comp
-L power:GND #PWR06
+P 900 7400
+F 0 "#PWR024" H 900 7150 50  0001 C CNN
+F 1 "GND" H 905 7227 50  0000 C CNN
+F 2 "" H 900 7400 50  0001 C CNN
+F 3 "" H 900 7400 50  0001 C CNN
+	1    900  7400
+	1    0    0    -1
+$EndComp
+$Comp
+L rata-rescue:GND-power #PWR06
 U 1 1 60FCD683
 P 900 5400
@@
 $EndComp
 $Comp
-L power:GND #PWR08
+L rata-rescue:GND-power #PWR08
 U 1 1 60FCD9BB
 P 900 6400
@@
 $EndComp
 $Comp
-L power:GND #PWR015
+L rata-rescue:GND-power #PWR015
 U 1 1 61052AAE
 P 2400 3400
@@
 $EndComp
 $Comp
-L power:GND #PWR017
+L rata-rescue:GND-power #PWR017
 U 1 1 61052DED
 P 2400 5400
@@
 $EndComp
 $Comp
-L power:GND #PWR019
+L rata-rescue:GND-power #PWR019
 U 1 1 61052FE5
 P 2400 6400
@@
 $EndComp
 $Comp
-L power:GND #PWR027
+L rata-rescue:GND-power #PWR027
 U 1 1 610534BB
 P 4400 5400
@@
 $EndComp
 $Comp
-L power:GND #PWR031
+L rata-rescue:GND-power #PWR031
 U 1 1 61053A07
 P 5400 6400
@@
 $EndComp
 $Comp
-L power:GND #PWR033
+L rata-rescue:GND-power #PWR033
 U 1 1 61053E27
 P 5400 7400
@@
 $EndComp
 $Comp
-L power:GND #PWR043
+L rata-rescue:GND-power #PWR043
 U 1 1 61054204
 P 6900 5400
@@
 $EndComp
 $Comp
-L power:GND #PWR045
+L rata-rescue:GND-power #PWR045
 U 1 1 6105454E
 P 8400 4900
@@
 $EndComp
 $Comp
-L power:GND #PWR040
+L rata-rescue:GND-power #PWR040
 U 1 1 61054A0F
 P 6900 3900
@@
 $EndComp
 $Comp
-L power:GND #PWR038
+L rata-rescue:GND-power #PWR038
 U 1 1 61054E40
 P 6900 3150
@@
 $EndComp
 $Comp
-L power:GND #PWR036
+L rata-rescue:GND-power #PWR036
 U 1 1 61055251
 P 6900 2000
@@
 $EndComp
 $Comp
-L power:+10V #PWR044
+L rata-rescue:+10V-power #PWR044
 U 1 1 610557C9
 P 8400 4600
@@
 $EndComp
 $Comp
-L power:+5V #PWR039
+L rata-rescue:+5V-power #PWR039
 U 1 1 610610A2
 P 6900 3600
@@
 $EndComp
 $Comp
-L power:+3V3 #PWR026
+L rata-rescue:+3V3-power #PWR026
 U 1 1 61062B54
 P 4400 1600
@@
 $EndComp
 $Comp
-L power:+3V3 #PWR014
+L rata-rescue:+3V3-power #PWR014
 U 1 1 61062D2B
 P 2400 2800
@@
 $EndComp
 $Comp
-L power:+3V3 #PWR020
+L rata-rescue:+3V3-power #PWR020
 U 1 1 610632EB
 P 2900 4100
@@
 $EndComp
 $Comp
-L power:+3V3 #PWR016
+L rata-rescue:+3V3-power #PWR016
 U 1 1 610636A7
 P 2400 5100
@@
 $EndComp
 $Comp
-L power:+3V3 #PWR032
+L rata-rescue:+3V3-power #PWR032
 U 1 1 6106424C
 P 5400 7100
@@
 $EndComp
 $Comp
-L power:+3V3 #PWR030
+L rata-rescue:+3V3-power #PWR030
 U 1 1 610647C1
 P 5400 6100
@@
 $EndComp
 $Comp
-L power:+3V3 #PWR041
+L rata-rescue:+3V3-power #PWR041
 U 1 1 61064F08
 P 6900 4600
@@
 $EndComp
 $Comp
-L power:+3V3 #PWR022
+L rata-rescue:+3V3-power #PWR022
 U 1 1 61066C2D
 P 3200 1450
@@
 	2400 6400 2500 6400
 Wire Wire Line
-	3500 6100 3600 6100
-Wire Wire Line
-	3600 6100 3600 5500
-Wire Wire Line
-	3600 5500 4000 5500
-Wire Wire Line
-	4000 5500 4000 5100
-Wire Wire Line
-	4000 5100 4500 5100
-Wire Wire Line
-	3900 6600 4000 6600
-Wire Wire Line
-	3900 6900 4000 6900
-Wire Wire Line
-	5000 6600 5100 6600
-Wire Wire Line
-	4000 6750 3800 6750
-Wire Wire Line
-	3800 6750 3800 5600
-Wire Wire Line
-	3800 5600 4100 5600
-Wire Wire Line
-	4100 5600 4100 5200
+	3500 6100 3900 6100
+Wire Wire Line
+	3900 5100 4500 5100
+Wire Wire Line
+	900  7100 1000 7100
+Wire Wire Line
+	900  7400 1000 7400
+Wire Wire Line
+	2000 7100 2100 7100
+Wire Wire Line
+	800  7250 800  6850
+Wire Wire Line
+	4100 6850 4100 5200
 Wire Wire Line
 	4100 5200 4500 5200
@@
 	6250 5200 6250 5750
 Wire Wire Line
-	6250 5750 5200 5750
-Wire Wire Line
-	5200 5750 5200 6750
-Wire Wire Line
-	5200 6750 5000 6750
+	6250 5750 4200 5750
+Wire Wire Line
+	4200 5750 4200 7250
+Wire Wire Line
+	4200 7250 2000 7250
 Wire Wire Line
 	6500 6200 6600 6200
@@
 	6900 3150 7000 3150
 $Comp
-L power:+3V3 #PWR034
+L rata-rescue:+3V3-power #PWR034
 U 1 1 61120F65
 P 6800 2700
@@
 VFD13
 $Comp
-L Device:Fuse F?
+L rata-rescue:Fuse-Device F?
 U 1 1 611F8C83
 P 1750 1300
@@
 Wire Wire Line
 	1600 1300 1500 1300
+Wire Wire Line
+	800  6850 4100 6850
+Wire Wire Line
+	3900 5100 3900 6100
+Wire Wire Line
+	800  7250 1000 7250
 Wire Bus Line
 	8000 3000 10500 3000
 Wire Bus Line
 	8350 1300 10000 1300
+$Comp
+L rata:ILC4-5_7L U1
+U 1 1 60FA6693
+P 8700 2300
+F 0 "U1" H 10200 2850 50  0000 L CNN
+F 1 "ILC4-5_7L" H 10100 2750 50  0000 L CNN
+F 2 "" H 8700 1750 50  0001 C CNN
+F 3 "" V 8850 2900 50  0001 C CNN
+	1    8700 2300
+	1    0    0    -1
+$EndComp
 $EndSCHEMATC
