File: Buttons.sch (KiCad schematic (older format))
At the start: 10 parts

Commit message: Add files via upload
Parts:
- removed D?: SMAJ5.0CA, symbol Device:D_TVS
- added D?: SMAJ5.0CA, symbol Device:D_TVS
Changed lines of the file:
@@
 $Descr A4 11693 8268
 encoding utf-8
-Sheet 5 11
+Sheet 10 15
 Title ""
 Date ""
@@
 AR Path="/60DF1160/60DF0A5B" Ref="U?"  Part="1"
 AR Path="/60DF196E/60DF0A5B" Ref="U?"  Part="1"
+AR Path="/60EE89A9/60DF0A5B" Ref="U?"  Part="1"
 F 0 "U?" H 6800 3742 50  0000 C CNN
 F 1 "AMS1117-3.3" H 6800 3651 50  0000 C CNN
@@
 AR Path="/60DF1160/60DF2176" Ref="C?"  Part="1"
 AR Path="/60DF196E/60DF2176" Ref="C?"  Part="1"
+AR Path="/60EE89A9/60DF2176" Ref="C?"  Part="1"
 F 0 "C?" H 7515 3696 50  0000 L CNN
 F 1 "10u" H 7515 3605 50  0000 L CNN
@@
 AR Path="/60DF1160/60DF2177" Ref="C?"  Part="1"
 AR Path="/60DF196E/60DF2177" Ref="C?"  Part="1"
+AR Path="/60EE89A9/60DF2177" Ref="C?"  Part="1"
 F 0 "C?" H 6315 3696 50  0000 L CNN
 F 1 "0,1" H 6315 3605 50  0000 L CNN
@@
 AR Path="/60DF1160/60DF2178" Ref="C?"  Part="1"
 AR Path="/60DF196E/60DF2178" Ref="C?"  Part="1"
+AR Path="/60EE89A9/60DF2178" Ref="C?"  Part="1"
 F 0 "C?" H 7915 3696 50  0000 L CNN
 F 1 "10u" H 7915 3605 50  0000 L CNN
@@
 AR Path="/60DF1160/60DF2179" Ref="TP?"  Part="1"
 AR Path="/60DF196E/60DF2179" Ref="TP?"  Part="1"
+AR Path="/60EE89A9/60DF2179" Ref="TP?"  Part="1"
 F 0 "TP?" H 7608 3618 50  0000 L CNN
 F 1 "TestPoint" H 7608 3527 50  0001 L CNN
@@
 AR Path="/60DF1160/60DF217C" Ref="TP?"  Part="1"
 AR Path="/60DF196E/60DF217C" Ref="TP?"  Part="1"
+AR Path="/60EE89A9/60DF217C" Ref="TP?"  Part="1"
 F 0 "TP?" H 5458 3618 50  0000 L CNN
 F 1 "TestPoint" H 5458 3527 50  0001 L CNN
@@
 AR Path="/60DF1160/60DF217D" Ref="C?"  Part="1"
 AR Path="/60DF196E/60DF217D" Ref="C?"  Part="1"
+AR Path="/60EE89A9/60DF217D" Ref="C?"  Part="1"
 F 0 "C?" H 4465 3696 50  0000 L CNN
 F 1 "1u" H 4465 3605 50  0000 L CNN
@@
 $Comp
 L Device:D_TVS D?
-U 1 1 60DF121A
+U 1 1 60E73022
 P 4850 3650
-AR Path="/60DF121A" Ref="D?"  Part="1"
-AR Path="/609FED99/60DF121A" Ref="D?"  Part="1"
-AR Path="/60DF07DE/60DF121A" Ref="D?"  Part="1"
-AR Path="/60DF0860/60DF121A" Ref="D?"  Part="1"
-AR Path="/60DF1072/60DF121A" Ref="D?"  Part="1"
-AR Path="/60DF1160/60DF121A" Ref="D?"  Part="1"
-AR Path="/60DF196E/60DF121A" Ref="D?"  Part="1"
+AR Path="/60E73022" Ref="D?"  Part="1"
+AR Path="/609FED99/60E73022" Ref="D?"  Part="1"
+AR Path="/60DF07DE/60E73022" Ref="D?"  Part="1"
+AR Path="/60DF0860/60E73022" Ref="D?"  Part="1"
+AR Path="/60DF1072/60E73022" Ref="D?"  Part="1"
+AR Path="/60DF1160/60E73022" Ref="D?"  Part="1"
+AR Path="/60DF196E/60E73022" Ref="D?"  Part="1"
+AR Path="/60EE89A9/60E73022" Ref="D?"  Part="1"
 F 0 "D?" V 4896 3570 50  0000 R CNN
 F 1 "SMAJ5.0CA" V 4805 3570 50  0000 R CNN
@@
 AR Path="/60DF1160/60DF0A63" Ref="C?"  Part="1"
 AR Path="/60DF196E/60DF0A63" Ref="C?"  Part="1"
+AR Path="/60EE89A9/60DF0A63" Ref="C?"  Part="1"
 F 0 "C?" H 3918 3696 50  0000 L CNN
 F 1 "100u" H 3918 3605 50  0000 L CNN
@@
 AR Path="/60DF1160/60DF217B" Ref="TP?"  Part="1"
 AR Path="/60DF196E/60DF217B" Ref="TP?"  Part="1"
+AR Path="/60EE89A9/60DF217B" Ref="TP?"  Part="1"
 F 0 "TP?" H 5458 3918 50  0000 L CNN
 F 1 "TestPoint" H 5458 3827 50  0001 L CNN

Commit message: Add files via upload
Parts:
- removed C?: 100u, symbol Device:CP
- removed C? (x2): 10u, Capacitor_SMD:C_1206_3216Metric_Pad1.33x1.80mm_HandSolder, symbol Device:C
- removed C?: 0,1, Capacitor_SMD:C_0603_1608Metric_Pad1.08x0.95mm_HandSolder, symbol Device:C
- removed C?: 1u, Capacitor_SMD:C_0603_1608Metric_Pad1.08x0.95mm_HandSolder, symbol Device:C
- removed D?: SMAJ5.0CA, symbol Device:D_TVS
- removed TP? (x3): TestPoint, symbol Connector:TestPoint
- removed U?: AMS1117-3.3, Package_TO_SOT_SMD:SOT-223-3_TabPin2, symbol Regulator_Linear:AMS1117-3.3
- added R? (x3): 4,7k, Resistor_SMD:R_0603_1608Metric_Pad0.98x0.95mm_HandSolder, symbol Device:R
- added SW? (x9): SW_Push, symbol Switch:SW_Push
Connections:
- net labels added: +3V3, COL0, COL1, COL2, ROW0, ROW1, ROW2
- net labels removed: +3V3_OUT, +5V_IN, GND
- wire segments 18 -> 50
Other:
- note added: "Button matrix"
- note removed: "Power source +3V3"

Commit message: Add files via upload
Parts:
- gave numbers to parts that had none: 12
Changed lines of the file:
@@
 AR Path="/60EE89A9/60FAFC0E" Ref="R?"  Part="1"
 AR Path="/60EF6B1B/60FAFC0E" Ref="R?"  Part="1"
-AR Path="/60DF196E/60FAFC0E" Ref="R?"  Part="1"
-F 0 "R?" H 7570 1796 50  0000 L CNN
+AR Path="/60DF196E/60FAFC0E" Ref="R24"  Part="1"
+F 0 "R24" H 7570 1796 50  0000 L CNN
 F 1 "4,7k" H 7570 1705 50  0000 L CNN
 F 2 "Resistor_SMD:R_0603_1608Metric_Pad0.98x0.95mm_HandSolder" V 7430 1750 50  0001 C CNN
@@
 AR Path="/60EE89A9/60FC25F1" Ref="R?"  Part="1"
 AR Path="/60EF6B1B/60FC25F1" Ref="R?"  Part="1"
-AR Path="/60DF196E/60FC25F1" Ref="R?"  Part="1"
-F 0 "R?" H 6570 1796 50  0000 L CNN
+AR Path="/60DF196E/60FC25F1" Ref="R22"  Part="1"
+F 0 "R22" H 6570 1796 50  0000 L CNN
 F 1 "4,7k" H 6570 1705 50  0000 L CNN
 F 2 "Resistor_SMD:R_0603_1608Metric_Pad0.98x0.95mm_HandSolder" V 6430 1750 50  0001 C CNN
@@
 AR Path="/60EE89A9/60FC27FD" Ref="R?"  Part="1"
 AR Path="/60EF6B1B/60FC27FD" Ref="R?"  Part="1"
-AR Path="/60DF196E/60FC27FD" Ref="R?"  Part="1"
-F 0 "R?" H 7070 1796 50  0000 L CNN
+AR Path="/60DF196E/60FC27FD" Ref="R23"  Part="1"
+F 0 "R23" H 7070 1796 50  0000 L CNN
 F 1 "4,7k" H 7070 1705 50  0000 L CNN
 F 2 "Resistor_SMD:R_0603_1608Metric_Pad0.98x0.95mm_HandSolder" V 6930 1750 50  0001 C CNN
@@
 COL2
 $Comp
-L Switch:SW_Push SW?
+L Switch:SW_Push SW1
 U 1 1 60FD2C62
 P 5200 3500
-F 0 "SW?" H 5200 3785 50  0000 C CNN
+F 0 "SW1" H 5200 3785 50  0000 C CNN
 F 1 "SW_Push" H 5200 3694 50  0000 C CNN
 F 2 "" H 5200 3700 50  0001 C CNN
@@
 $EndComp
 $Comp
-L Switch:SW_Push SW?
+L Switch:SW_Push SW4
 U 1 1 60FD42DB
 P 6200 3500
-F 0 "SW?" H 6200 3785 50  0000 C CNN
+F 0 "SW4" H 6200 3785 50  0000 C CNN
 F 1 "SW_Push" H 6200 3694 50  0000 C CNN
 F 2 "" H 6200 3700 50  0001 C CNN
@@
 $EndComp
 $Comp
-L Switch:SW_Push SW?
+L Switch:SW_Push SW7
 U 1 1 60FD47DB
 P 7200 3500
-F 0 "SW?" H 7200 3785 50  0000 C CNN
+F 0 "SW7" H 7200 3785 50  0000 C CNN
 F 1 "SW_Push" H 7200 3694 50  0000 C CNN
 F 2 "" H 7200 3700 50  0001 C CNN
@@
 $EndComp
 $Comp
-L Switch:SW_Push SW?
+L Switch:SW_Push SW2
 U 1 1 60FD5B91
 P 5200 4500
-F 0 "SW?" H 5200 4785 50  0000 C CNN
+F 0 "SW2" H 5200 4785 50  0000 C CNN
 F 1 "SW_Push" H 5200 4694 50  0000 C CNN
 F 2 "" H 5200 4700 50  0001 C CNN
@@
 $EndComp
 $Comp
-L Switch:SW_Push SW?
+L Switch:SW_Push SW5
 U 1 1 60FD5B97
 P 6200 4500
-F 0 "SW?" H 6200 4785 50  0000 C CNN
+F 0 "SW5" H 6200 4785 50  0000 C CNN
 F 1 "SW_Push" H 6200 4694 50  0000 C CNN
 F 2 "" H 6200 4700 50  0001 C CNN
@@
 $EndComp
 $Comp
-L Switch:SW_Push SW?
+L Switch:SW_Push SW8
 U 1 1 60FD5B9D
 P 7200 4500
-F 0 "SW?" H 7200 4785 50  0000 C CNN
+F 0 "SW8" H 7200 4785 50  0000 C CNN
 F 1 "SW_Push" H 7200 4694 50  0000 C CNN
 F 2 "" H 7200 4700 50  0001 C CNN
@@
 $EndComp
 $Comp
-L Switch:SW_Push SW?
+L Switch:SW_Push SW3
 U 1 1 60FD6D63
 P 5200 5500
-F 0 "SW?" H 5200 5785 50  0000 C CNN
+F 0 "SW3" H 5200 5785 50  0000 C CNN
 F 1 "SW_Push" H 5200 5694 50  0000 C CNN
 F 2 "" H 5200 5700 50  0001 C CNN
@@
 $EndComp
 $Comp
-L Switch:SW_Push SW?
+L Switch:SW_Push SW6
 U 1 1 60FD6D69
 P 6200 5500
-F 0 "SW?" H 6200 5785 50  0000 C CNN
+F 0 "SW6" H 6200 5785 50  0000 C CNN
 F 1 "SW_Push" H 6200 5694 50  0000 C CNN
 F 2 "" H 6200 5700 50  0001 C CNN
@@
 $EndComp
 $Comp
-L Switch:SW_Push SW?
+L Switch:SW_Push SW9
 U 1 1 60FD6D6F
 P 7200 5500
-F 0 "SW?" H 7200 5785 50  0000 C CNN
+F 0 "SW9" H 7200 5785 50  0000 C CNN
 F 1 "SW_Push" H 7200 5694 50  0000 C CNN
 F 2 "" H 7200 5700 50  0001 C CNN

Commit message: Add files via upload
Parts:
- R22, R23, R24: symbol Device:R -> rata-rescue:R-Device
- SW1, SW2, SW3, SW4, SW5, SW6, SW7, SW8, SW9: symbol Switch:SW_Push -> rata-rescue:SW_Push-Switch
Changed lines of the file:
@@
 COL0
 $Comp
-L Device:R R?
+L rata-rescue:R-Device R?
 U 1 1 60FAFC0E
 P 7500 1750
@@
 $EndComp
 $Comp
-L Device:R R?
+L rata-rescue:R-Device R?
 U 1 1 60FC25F1
 P 6500 1750
@@
 $EndComp
 $Comp
-L Device:R R?
+L rata-rescue:R-Device R?
 U 1 1 60FC27FD
 P 7000 1750
@@
 COL2
 $Comp
-L Switch:SW_Push SW1
+L rata-rescue:SW_Push-Switch SW1
 U 1 1 60FD2C62
 P 5200 3500
@@
 $EndComp
 $Comp
-L Switch:SW_Push SW4
+L rata-rescue:SW_Push-Switch SW4
 U 1 1 60FD42DB
 P 6200 3500
@@
 $EndComp
 $Comp
-L Switch:SW_Push SW7
+L rata-rescue:SW_Push-Switch SW7
 U 1 1 60FD47DB
 P 7200 3500
@@
 $EndComp
 $Comp
-L Switch:SW_Push SW2
+L rata-rescue:SW_Push-Switch SW2
 U 1 1 60FD5B91
 P 5200 4500
@@
 $EndComp
 $Comp
-L Switch:SW_Push SW5
+L rata-rescue:SW_Push-Switch SW5
 U 1 1 60FD5B97
 P 6200 4500
@@
 $EndComp
 $Comp
-L Switch:SW_Push SW8
+L rata-rescue:SW_Push-Switch SW8
 U 1 1 60FD5B9D
 P 7200 4500
@@
 $EndComp
 $Comp
-L Switch:SW_Push SW3
+L rata-rescue:SW_Push-Switch SW3
 U 1 1 60FD6D63
 P 5200 5500
@@
 $EndComp
 $Comp
-L Switch:SW_Push SW6
+L rata-rescue:SW_Push-Switch SW6
 U 1 1 60FD6D69
 P 6200 5500
@@
 $EndComp
 $Comp
-L Switch:SW_Push SW9
+L rata-rescue:SW_Push-Switch SW9
 U 1 1 60FD6D6F
 P 7200 5500

Commit message: Add files via upload
Parts:
- SW1, SW2, SW3, SW4, SW5, SW6, SW7, SW8, SW9: footprint (none) -> Button_Switch_THT:SW_PUSH_6mm_H4.3mm
- renumbered R22 to R23, R23 to R24, R24 to R25
Changed lines of the file:
@@
 encoding utf-8
 Sheet 9 23
-Title ""
-Date ""
-Rev ""
-Comp ""
+Title "rata"
+Date "2021-09-25"
+Rev "1.0"
+Comp "Yuriy Volkov"
 Comment1 ""
 Comment2 ""
@@
 AR Path="/60EE89A9/60FAFC0E" Ref="R?"  Part="1"
 AR Path="/60EF6B1B/60FAFC0E" Ref="R?"  Part="1"
-AR Path="/60DF196E/60FAFC0E" Ref="R24"  Part="1"
-F 0 "R24" H 7570 1796 50  0000 L CNN
+AR Path="/60DF196E/60FAFC0E" Ref="R25"  Part="1"
+F 0 "R25" H 7570 1796 50  0000 L CNN
 F 1 "4,7k" H 7570 1705 50  0000 L CNN
 F 2 "Resistor_SMD:R_0603_1608Metric_Pad0.98x0.95mm_HandSolder" V 7430 1750 50  0001 C CNN
@@
 AR Path="/60EE89A9/60FC25F1" Ref="R?"  Part="1"
 AR Path="/60EF6B1B/60FC25F1" Ref="R?"  Part="1"
-AR Path="/60DF196E/60FC25F1" Ref="R22"  Part="1"
-F 0 "R22" H 6570 1796 50  0000 L CNN
+AR Path="/60DF196E/60FC25F1" Ref="R23"  Part="1"
+F 0 "R23" H 6570 1796 50  0000 L CNN
 F 1 "4,7k" H 6570 1705 50  0000 L CNN
 F 2 "Resistor_SMD:R_0603_1608Metric_Pad0.98x0.95mm_HandSolder" V 6430 1750 50  0001 C CNN
@@
 AR Path="/60EE89A9/60FC27FD" Ref="R?"  Part="1"
 AR Path="/60EF6B1B/60FC27FD" Ref="R?"  Part="1"
-AR Path="/60DF196E/60FC27FD" Ref="R23"  Part="1"
-F 0 "R23" H 7070 1796 50  0000 L CNN
+AR Path="/60DF196E/60FC27FD" Ref="R24"  Part="1"
+F 0 "R24" H 7070 1796 50  0000 L CNN
 F 1 "4,7k" H 7070 1705 50  0000 L CNN
 F 2 "Resistor_SMD:R_0603_1608Metric_Pad0.98x0.95mm_HandSolder" V 6930 1750 50  0001 C CNN
@@
 F 0 "SW1" H 5200 3785 50  0000 C CNN
 F 1 "SW_Push" H 5200 3694 50  0000 C CNN
-F 2 "" H 5200 3700 50  0001 C CNN
+F 2 "Button_Switch_THT:SW_PUSH_6mm_H4.3mm" H 5200 3700 50  0001 C CNN
 F 3 "~" H 5200 3700 50  0001 C CNN
 	1    5200 3500
@@
 F 0 "SW4" H 6200 3785 50  0000 C CNN
 F 1 "SW_Push" H 6200 3694 50  0000 C CNN
-F 2 "" H 6200 3700 50  0001 C CNN
+F 2 "Button_Switch_THT:SW_PUSH_6mm_H4.3mm" H 6200 3700 50  0001 C CNN
 F 3 "~" H 6200 3700 50  0001 C CNN
 	1    6200 3500
@@
 F 0 "SW7" H 7200 3785 50  0000 C CNN
 F 1 "SW_Push" H 7200 3694 50  0000 C CNN
-F 2 "" H 7200 3700 50  0001 C CNN
+F 2 "Button_Switch_THT:SW_PUSH_6mm_H4.3mm" H 7200 3700 50  0001 C CNN
 F 3 "~" H 7200 3700 50  0001 C CNN
 	1    7200 3500
@@
 F 0 "SW2" H 5200 4785 50  0000 C CNN
 F 1 "SW_Push" H 5200 4694 50  0000 C CNN
-F 2 "" H 5200 4700 50  0001 C CNN
+F 2 "Button_Switch_THT:SW_PUSH_6mm_H4.3mm" H 5200 4700 50  0001 C CNN
 F 3 "~" H 5200 4700 50  0001 C CNN
 	1    5200 4500
@@
 F 0 "SW5" H 6200 4785 50  0000 C CNN
 F 1 "SW_Push" H 6200 4694 50  0000 C CNN
-F 2 "" H 6200 4700 50  0001 C CNN
+F 2 "Button_Switch_THT:SW_PUSH_6mm_H4.3mm" H 6200 4700 50  0001 C CNN
 F 3 "~" H 6200 4700 50  0001 C CNN
 	1    6200 4500
@@
 F 0 "SW8" H 7200 4785 50  0000 C CNN
 F 1 "SW_Push" H 7200 4694 50  0000 C CNN
-F 2 "" H 7200 4700 50  0001 C CNN
+F 2 "Button_Switch_THT:SW_PUSH_6mm_H4.3mm" H 7200 4700 50  0001 C CNN
 F 3 "~" H 7200 4700 50  0001 C CNN
 	1    7200 4500
@@
 F 0 "SW3" H 5200 5785 50  0000 C CNN
 F 1 "SW_Push" H 5200 5694 50  0000 C CNN
-F 2 "" H 5200 5700 50  0001 C CNN
+F 2 "Button_Switch_THT:SW_PUSH_6mm_H4.3mm" H 5200 5700 50  0001 C CNN
 F 3 "~" H 5200 5700 50  0001 C CNN
 	1    5200 5500
@@
 F 0 "SW6" H 6200 5785 50  0000 C CNN
 F 1 "SW_Push" H 6200 5694 50  0000 C CNN
-F 2 "" H 6200 5700 50  0001 C CNN
+F 2 "Button_Switch_THT:SW_PUSH_6mm_H4.3mm" H 6200 5700 50  0001 C CNN
 F 3 "~" H 6200 5700 50  0001 C CNN
 	1    6200 5500
@@
 F 0 "SW9" H 7200 5785 50  0000 C CNN
 F 1 "SW_Push" H 7200 5694 50  0000 C CNN
-F 2 "" H 7200 5700 50  0001 C CNN
+F 2 "Button_Switch_THT:SW_PUSH_6mm_H4.3mm" H 7200 5700 50  0001 C CNN
 F 3 "~" H 7200 5700 50  0001 C CNN
 	1    7200 5500
