File: Buzzer.sch (KiCad schematic (older format))
At the start: 4 parts

Commit message: Add files via upload
Changed lines of the file:
@@
 $Descr A4 11693 8268
 encoding utf-8
-Sheet 4 11
+Sheet 4 15
 Title ""
 Date ""
@@
 Wire Wire Line
 	5500 4500 5000 4500
+Text HLabel 5000 3500 0    50   Input ~ 0
++5V
+Text HLabel 5000 5500 0    50   Input ~ 0
+GND
 $EndSCHEMATC

Commit message: Add files via upload
Changed lines of the file:
@@
 $Descr A4 11693 8268
 encoding utf-8
-Sheet 4 15
+Sheet 4 20
 Title ""
 Date ""
@@
 	1    0    0    -1
 $EndComp
-$Comp
-L power:GND #PWR?
-U 1 1 60B3B924
-P 6500 5000
-AR Path="/60B3B924" Ref="#PWR?"  Part="1"
-AR Path="/60B39FE1/60B3B924" Ref="#PWR?"  Part="1"
-F 0 "#PWR?" H 6500 4750 50  0001 C CNN
-F 1 "GND" H 6505 4827 50  0000 C CNN
-F 2 "" H 6500 5000 50  0001 C CNN
-F 3 "" H 6500 5000 50  0001 C CNN
-	1    6500 5000
-	1    0    0    -1
-$EndComp
 Text Notes 6150 2700 2    197  ~ 0
 Buzzer
@@
 	1    5650 4500
 	0    -1   -1   0
-$EndComp
-$Comp
-L power:+5V #PWR?
-U 1 1 60B40656
-P 6500 3500
-AR Path="/609FED99/60B40656" Ref="#PWR?"  Part="1"
-AR Path="/60B39FE1/60B40656" Ref="#PWR?"  Part="1"
-F 0 "#PWR?" H 6500 3350 50  0001 C CNN
-F 1 "+5V" H 6515 3673 50  0000 C CNN
-F 2 "" H 6500 3500 50  0001 C CNN
-F 3 "" H 6500 3500 50  0001 C CNN
-	1    6500 3500
-	1    0    0    -1
 $EndComp
 Wire Wire Line
@@
 Wire Wire Line
 	6000 5000 6500 5000
-Connection ~ 6500 5000
 Wire Wire Line
 	5500 4500 5000 4500
@@
 Text HLabel 5000 5500 0    50   Input ~ 0
 GND
+Wire Wire Line
+	5000 3500 6500 3500
+Wire Wire Line
+	6500 5000 6500 5500
+Wire Wire Line
+	6500 5500 5000 5500
+Connection ~ 6500 5000
 $EndSCHEMATC

Commit message: Add files via upload
Parts:
- R6: renamed from R?; value 3,3k -> 4.7k
- gave numbers to parts that had none: 3
Changed lines of the file:
@@
 P 6600 3900
 AR Path="/609C9D41/60B3B2EE" Ref="BZ?"  Part="1"
-AR Path="/60B39FE1/60B3B2EE" Ref="BZ?"  Part="1"
-F 0 "BZ?" H 6752 3929 50  0000 L CNN
+AR Path="/60B39FE1/60B3B2EE" Ref="BZ1"  Part="1"
+F 0 "BZ1" H 6752 3929 50  0000 L CNN
 F 1 "Buzzer" H 6752 3838 50  0000 L CNN
 F 2 "" V 6575 4000 50  0001 C CNN
@@
 P 6400 4500
 AR Path="/609C9D41/60B3B2F4" Ref="Q?"  Part="1"
-AR Path="/60B39FE1/60B3B2F4" Ref="Q?"  Part="1"
-F 0 "Q?" H 6591 4546 50  0000 L CNN
+AR Path="/60B39FE1/60B3B2F4" Ref="Q1"  Part="1"
+F 0 "Q1" H 6591 4546 50  0000 L CNN
 F 1 "BC847" H 6591 4455 50  0000 L CNN
 F 2 "Package_TO_SOT_SMD:SOT-23" H 6600 4425 50  0001 L CIN
@@
 P 6000 4750
 AR Path="/60B3B65C" Ref="R?"  Part="1"
-AR Path="/60B39FE1/60B3B65C" Ref="R?"  Part="1"
-F 0 "R?" H 6070 4796 50  0000 L CNN
+AR Path="/60B39FE1/60B3B65C" Ref="R7"  Part="1"
+F 0 "R7" H 6070 4796 50  0000 L CNN
 F 1 "56k" H 6070 4705 50  0000 L CNN
 F 2 "Resistor_SMD:R_0603_1608Metric_Pad0.98x0.95mm_HandSolder" V 5930 4750 50  0001 C CNN
@@
 P 5650 4500
 AR Path="/60B3CA8D" Ref="R?"  Part="1"
-AR Path="/60B39FE1/60B3CA8D" Ref="R?"  Part="1"
-F 0 "R?" V 5750 4450 50  0000 L CNN
-F 1 "3,3k" V 5550 4400 50  0000 L CNN
+AR Path="/60B39FE1/60B3CA8D" Ref="R6"  Part="1"
+F 0 "R6" V 5750 4450 50  0000 L CNN
+F 1 "4.7k" V 5550 4400 50  0000 L CNN
 F 2 "Resistor_SMD:R_0603_1608Metric_Pad0.98x0.95mm_HandSolder" V 5580 4500 50  0001 C CNN
 F 3 "~" H 5650 4500 50  0001 C CNN

Commit message: Add files via upload
Parts:
- BZ1: symbol Device:Buzzer -> rata-rescue:Buzzer-Device
- Q1: symbol Transistor_BJT:BC847 -> rata-rescue:BC847-Transistor_BJT
- R6, R7: symbol Device:R -> rata-rescue:R-Device
Changed lines of the file:
@@
 $EndDescr
 $Comp
-L Device:Buzzer BZ?
+L rata-rescue:Buzzer-Device BZ?
 U 1 1 60B3B2EE
 P 6600 3900
@@
 $EndComp
 $Comp
-L Transistor_BJT:BC847 Q?
+L rata-rescue:BC847-Transistor_BJT Q?
 U 1 1 60B3B2F4
 P 6400 4500
@@
 $EndComp
 $Comp
-L Device:R R?
+L rata-rescue:R-Device R?
 U 1 1 60B3B65C
 P 6000 4750
@@
 EN
 $Comp
-L Device:R R?
+L rata-rescue:R-Device R?
 U 1 1 60B3CA8D
 P 5650 4500

Commit message: Add files via upload
Parts:
- BZ1: footprint (none) -> Buzzer_Beeper:Buzzer_12x9.5RM7.6
- renumbered R6 to R7, R7 to R8
Changed lines of the file:
@@
 encoding utf-8
 Sheet 4 23
-Title ""
-Date ""
-Rev ""
-Comp ""
+Title "rata"
+Date "2021-09-25"
+Rev "1.0"
+Comp "Yuriy Volkov"
 Comment1 ""
 Comment2 ""
@@
 F 0 "BZ1" H 6752 3929 50  0000 L CNN
 F 1 "Buzzer" H 6752 3838 50  0000 L CNN
-F 2 "" V 6575 4000 50  0001 C CNN
+F 2 "Buzzer_Beeper:Buzzer_12x9.5RM7.6" V 6575 4000 50  0001 C CNN
 F 3 "~" V 6575 4000 50  0001 C CNN
 	1    6600 3900
@@
 P 6000 4750
 AR Path="/60B3B65C" Ref="R?"  Part="1"
-AR Path="/60B39FE1/60B3B65C" Ref="R7"  Part="1"
-F 0 "R7" H 6070 4796 50  0000 L CNN
+AR Path="/60B39FE1/60B3B65C" Ref="R8"  Part="1"
+F 0 "R8" H 6070 4796 50  0000 L CNN
 F 1 "56k" H 6070 4705 50  0000 L CNN
 F 2 "Resistor_SMD:R_0603_1608Metric_Pad0.98x0.95mm_HandSolder" V 5930 4750 50  0001 C CNN
@@
 P 5650 4500
 AR Path="/60B3CA8D" Ref="R?"  Part="1"
-AR Path="/60B39FE1/60B3CA8D" Ref="R6"  Part="1"
-F 0 "R6" V 5750 4450 50  0000 L CNN
+AR Path="/60B39FE1/60B3CA8D" Ref="R7"  Part="1"
+F 0 "R7" V 5750 4450 50  0000 L CNN
 F 1 "4.7k" V 5550 4400 50  0000 L CNN
 F 2 "Resistor_SMD:R_0603_1608Metric_Pad0.98x0.95mm_HandSolder" V 5580 4500 50  0001 C CNN
