File: DAC.sch (KiCad schematic (older format))
At the start: 15 parts

Commit message: Add files via upload
Parts:
- removed C?: 10u, Capacitor_SMD:C_1206_3216Metric_Pad1.33x1.80mm_HandSolder, symbol Device:C
- removed C?: 1u, Capacitor_SMD:C_0603_1608Metric_Pad1.08x0.95mm_HandSolder, symbol Device:C
- removed C?: 100u, symbol Device:CP
- removed D?: SMAJ5.0CA, symbol Device:D_TVS
- removed U?: LM321, Package_TO_SOT_SMD:SOT-23-5, symbol Amplifier_Operational:LM321
- removed U?: AMS1117-3.3, Package_TO_SOT_SMD:SOT-223-3_TabPin2, symbol Regulator_Linear:AMS1117-3.3
- added C? (x3): 0,1, Capacitor_SMD:C_0603_1608Metric_Pad1.08x0.95mm_HandSolder, symbol Device:C
- added R? (x2): 4,7k, Resistor_SMD:R_0603_1608Metric_Pad0.98x0.95mm_HandSolder, symbol Device:R
- added R? (x6): 1, Resistor_SMD:R_0603_1608Metric_Pad0.98x0.95mm_HandSolder, symbol Device:R
- added R?: 0, Resistor_SMD:R_0603_1608Metric_Pad0.98x0.95mm_HandSolder, symbol Device:R
Connections:
- net labels added: +3V3, AUD, SCK, SDA
- net labels removed: +3V3_OUT, +5V_IN
- wire segments 18 -> 72
Other:
- note added: "DAC with filter and preamplifier\n"
- note removed: "Power source +3V3"
- moved on the sheet: C?, TP?, U?, U?A, U?B, U?C

Commit message: Add files via upload
Parts:
- removed C?: 10u, Capacitor_SMD:C_1206_3216Metric_Pad1.33x1.80mm_HandSolder, symbol Device:C
- added C?: 10u, Capacitor_SMD:C_1206_3216Metric_Pad1.33x1.80mm_HandSolder, symbol Device:C
Connections:
- net +3V3: now also C?.1
- net GND: now also C?.2
Changed lines of the file:
@@
 $Descr A4 11693 8268
 encoding utf-8
-Sheet 13 15
+Sheet 14 20
 Title ""
 Date ""
@@
 $Comp
 L Device:C C?
-U 1 1 60EE8A0B
+U 1 1 60F186C4
 P 2500 3350
-AR Path="/60EE8A0B" Ref="C?"  Part="1"
-AR Path="/609CA6A8/609D24C0/60EE8A0B" Ref="C?"  Part="1"
-AR Path="/609CA6A8/60A08E0B/60EE8A0B" Ref="C?"  Part="1"
-AR Path="/609CA6A8/60A0A46E/60EE8A0B" Ref="C?"  Part="1"
-AR Path="/609CA6A8/60A0A500/60EE8A0B" Ref="C?"  Part="1"
-AR Path="/609CA6A8/60A0A922/60EE8A0B" Ref="C?"  Part="1"
-AR Path="/609CA6A8/60EE8A0B" Ref="C?"  Part="1"
-AR Path="/609CA6A8/60AE5653/60EE8A0B" Ref="C?"  Part="1"
-AR Path="/609FED99/60EE8A0B" Ref="C?"  Part="1"
-AR Path="/60DF07DE/60EE8A0B" Ref="C?"  Part="1"
-AR Path="/60DF0860/60EE8A0B" Ref="C?"  Part="1"
-AR Path="/60DF1072/60EE8A0B" Ref="C?"  Part="1"
-AR Path="/60DF1160/60EE8A0B" Ref="C?"  Part="1"
-AR Path="/60E72FD7/60EE8A0B" Ref="C?"  Part="1"
-AR Path="/60EF6B1B/60EE8A0B" Ref="C?"  Part="1"
+AR Path="/60F186C4" Ref="C?"  Part="1"
+AR Path="/609CA6A8/609D24C0/60F186C4" Ref="C?"  Part="1"
+AR Path="/609CA6A8/60A08E0B/60F186C4" Ref="C?"  Part="1"
+AR Path="/609CA6A8/60A0A46E/60F186C4" Ref="C?"  Part="1"
+AR Path="/609CA6A8/60A0A500/60F186C4" Ref="C?"  Part="1"
+AR Path="/609CA6A8/60A0A922/60F186C4" Ref="C?"  Part="1"
+AR Path="/609CA6A8/60F186C4" Ref="C?"  Part="1"
+AR Path="/609CA6A8/60AE5653/60F186C4" Ref="C?"  Part="1"
+AR Path="/609FED99/60F186C4" Ref="C?"  Part="1"
+AR Path="/60DF07DE/60F186C4" Ref="C?"  Part="1"
+AR Path="/60DF0860/60F186C4" Ref="C?"  Part="1"
+AR Path="/60DF1072/60F186C4" Ref="C?"  Part="1"
+AR Path="/60DF1160/60F186C4" Ref="C?"  Part="1"
+AR Path="/60E72FD7/60F186C4" Ref="C?"  Part="1"
+AR Path="/60EF6B1B/60F186C4" Ref="C?"  Part="1"
 F 0 "C?" H 2615 3396 50  0000 L CNN
 F 1 "10u" H 2615 3305 50  0000 L CNN

Commit message: Add files via upload
Parts:
- added J?: Conn_01x03_Male, symbol Connector:Conn_01x03_Male
Connections:
- net GND: now also J?.3 (Pin_3)
- net SCK: now also J?.1 (Pin_1)
- net SDA: now also J?.2 (Pin_2)
Changed lines of the file:
@@
 $Descr A4 11693 8268
 encoding utf-8
-Sheet 14 20
+Sheet 14 24
 Title ""
 Date ""
@@
 $EndComp
 Wire Wire Line
-	1000 5000 2500 5000
+	1000 5000 1500 5000
 Wire Wire Line
 	9250 5000 9250 4500
@@
 	2750 5000 3400 5000
 Wire Wire Line
-	1000 4500 2000 4500
+	1000 4500 1750 4500
 Wire Wire Line
 	2000 3900 2000 4100
@@
 Connection ~ 1500 4000
 Wire Wire Line
-	1500 4000 3000 4000
+	1500 4000 1850 4000
 Wire Wire Line
 	1000 3000 1500 3000
@@
 Wire Wire Line
 	9250 3800 9250 3250
+$Comp
+L Connector:Conn_01x03_Male J?
+U 1 1 60FEAD39
+P 2200 5400
+AR Path="/60EF6B1B/60FEAD39" Ref="J?"  Part="1"
+AR Path="/60E72FD7/60FEAD39" Ref="J?"  Part="1"
+F 0 "J?" H 2172 5424 50  0000 R CNN
+F 1 "Conn_01x03_Male" H 2172 5333 50  0000 R CNN
+F 2 "" H 2200 5400 50  0001 C CNN
+F 3 "~" H 2200 5400 50  0001 C CNN
+	1    2200 5400
+	-1   0    0    -1
+$EndComp
+Wire Wire Line
+	2000 5500 1500 5500
+Wire Wire Line
+	1500 5500 1500 5000
+Connection ~ 1500 5000
+Wire Wire Line
+	1500 5000 2500 5000
+Wire Wire Line
+	2000 5400 1750 5400
+Wire Wire Line
+	1750 5400 1750 4500
+Connection ~ 1750 4500
+Wire Wire Line
+	1750 4500 2000 4500
+Wire Wire Line
+	2000 5300 1850 5300
+Wire Wire Line
+	1850 5300 1850 4000
+Connection ~ 1850 4000
+Wire Wire Line
+	1850 4000 3000 4000
 $EndSCHEMATC

Commit message: Add files via upload
Connections:
- net +3V3: no longer C?.1, C?.1, C?.1, U?.3 (VDD), U?.8 (V+)
- new net +3V3A: C?.1, C?.1, C?.1, U?.3 (VDD), U?.8 (V+)
Changed lines of the file:
@@
 $Descr A4 11693 8268
 encoding utf-8
-Sheet 14 23
+Sheet 12 23
 Title ""
 Date ""
@@
 $EndComp
 Text HLabel 1000 3000 0    50   Input ~ 0
-+3V3
++3V3A
 Text HLabel 1000 5000 0    50   Input ~ 0
 GND
@@
 	1500 4000 1850 4000
 Wire Wire Line
-	1000 3000 1500 3000
-Wire Wire Line
 	4500 3200 4500 3000
 Connection ~ 4500 3000
@@
 Wire Wire Line
 	10250 3900 10500 3900
-Wire Wire Line
-	2000 3600 2000 3000
-Connection ~ 2000 3000
-Wire Wire Line
-	2000 3000 2500 3000
-Wire Wire Line
-	1500 3600 1500 3000
-Connection ~ 1500 3000
-Wire Wire Line
-	1500 3000 2000 3000
 $Comp
 L Device:R R?
@@
 Wire Wire Line
 	1850 4000 3000 4000
+Wire Wire Line
+	1000 3000 2500 3000
+Text HLabel 1000 3500 0    50   Input ~ 0
++3V3
+Wire Wire Line
+	1000 3500 1500 3500
+Wire Wire Line
+	2000 3500 2000 3600
+Wire Wire Line
+	1500 3600 1500 3500
+Connection ~ 1500 3500
+Wire Wire Line
+	1500 3500 2000 3500
 $EndSCHEMATC

Commit message: Add files via upload
Parts:
- gave numbers to parts that had none: 20
Changed lines of the file:
@@
 $Descr A4 11693 8268
 encoding utf-8
-Sheet 12 23
+Sheet 11 23
 Title ""
 Date ""
@@
 AR Path="/60DF1072/60F186C4" Ref="C?"  Part="1"
 AR Path="/60DF1160/60F186C4" Ref="C?"  Part="1"
-AR Path="/60E72FD7/60F186C4" Ref="C?"  Part="1"
+AR Path="/60E72FD7/60F186C4" Ref="C40"  Part="1"
 AR Path="/60EF6B1B/60F186C4" Ref="C?"  Part="1"
-F 0 "C?" H 2615 3396 50  0000 L CNN
+F 0 "C40" H 2615 3396 50  0000 L CNN
 F 1 "10u" H 2615 3305 50  0000 L CNN
 F 2 "Capacitor_SMD:C_1206_3216Metric_Pad1.33x1.80mm_HandSolder" H 2538 3200 50  0001 C CNN
@@
 AR Path="/60DF1072/60DF1217" Ref="C?"  Part="1"
 AR Path="/60DF1160/60DF1217" Ref="C?"  Part="1"
-AR Path="/60E72FD7/60DF1217" Ref="C?"  Part="1"
+AR Path="/60E72FD7/60DF1217" Ref="C42"  Part="1"
 AR Path="/60EF6B1B/60DF1217" Ref="C?"  Part="1"
-F 0 "C?" H 4615 3396 50  0000 L CNN
+F 0 "C42" H 4615 3396 50  0000 L CNN
 F 1 "0,1" H 4615 3305 50  0000 L CNN
 F 2 "Capacitor_SMD:C_0603_1608Metric_Pad1.08x0.95mm_HandSolder" H 4538 3200 50  0001 C CNN
@@
 AR Path="/60DF1072/60DF1219" Ref="TP?"  Part="1"
 AR Path="/60DF1160/60DF1219" Ref="TP?"  Part="1"
-AR Path="/60E72FD7/60DF1219" Ref="TP?"  Part="1"
+AR Path="/60E72FD7/60DF1219" Ref="TP15"  Part="1"
 AR Path="/60EF6B1B/60DF1219" Ref="TP?"  Part="1"
-F 0 "TP?" H 5558 4218 50  0000 L CNN
+F 0 "TP15" H 5558 4218 50  0000 L CNN
 F 1 "TestPoint" H 5558 4127 50  0001 L CNN
 F 2 "" H 5700 4100 50  0001 C CNN
@@
 AR Path="/60DF1072/60EE8A09" Ref="TP?"  Part="1"
 AR Path="/60DF1160/60EE8A09" Ref="TP?"  Part="1"
-AR Path="/60E72FD7/60EE8A09" Ref="TP?"  Part="1"
+AR Path="/60E72FD7/60EE8A09" Ref="TP17"  Part="1"
 AR Path="/60EF6B1B/60EE8A09" Ref="TP?"  Part="1"
-F 0 "TP?" H 10558 4018 50  0000 L CNN
+F 0 "TP17" H 10558 4018 50  0000 L CNN
 F 1 "TestPoint" H 10558 3927 50  0001 L CNN
 F 2 "" H 10700 3900 50  0001 C CNN
@@
 AR Path="/60DF1072/60DF121C" Ref="TP?"  Part="1"
 AR Path="/60DF1160/60DF121C" Ref="TP?"  Part="1"
-AR Path="/60E72FD7/60DF121C" Ref="TP?"  Part="1"
+AR Path="/60E72FD7/60DF121C" Ref="TP16"  Part="1"
 AR Path="/60EF6B1B/60DF121C" Ref="TP?"  Part="1"
-F 0 "TP?" H 8558 4118 50  0000 L CNN
+F 0 "TP16" H 8558 4118 50  0000 L CNN
 F 1 "TestPoint" H 8558 4027 50  0001 L CNN
 F 2 "" H 8700 4000 50  0001 C CNN
@@
 AUD
 $Comp
-L Analog_DAC:MCP4725xxx-xCH U?
+L Analog_DAC:MCP4725xxx-xCH U7
 U 1 1 60EA7615
 P 3400 4100
-F 0 "U?" H 3550 4500 50  0000 L CNN
+F 0 "U7" H 3550 4500 50  0000 L CNN
 F 1 "MCP4725xxx-xCH" H 3550 4400 50  0000 L CNN
 F 2 "Package_TO_SOT_SMD:SOT-23-6" H 3400 3850 50  0001 C CNN
@@
 $EndComp
 $Comp
-L Amplifier_Operational:MCP6022 U?
+L Amplifier_Operational:MCP6022 U8
 U 1 1 60EA87F7
 P 7600 4000
-F 0 "U?" H 7550 3600 50  0000 C CNN
+F 0 "U8" H 7550 3600 50  0000 C CNN
 F 1 "MCP6022" H 7600 3700 50  0000 C CNN
 F 2 "" H 7600 4000 50  0001 C CNN
@@
 $EndComp
 $Comp
-L Amplifier_Operational:MCP6022 U?
+L Amplifier_Operational:MCP6022 U8
 U 2 1 60EA9696
 P 9800 3900
-F 0 "U?" H 9800 3500 50  0000 C CNN
+F 0 "U8" H 9800 3500 50  0000 C CNN
 F 1 "MCP6022" H 9850 3600 50  0000 C CNN
 F 2 "" H 9800 3900 50  0001 C CNN
@@
 $EndComp
 $Comp
-L Amplifier_Operational:MCP6022 U?
+L Amplifier_Operational:MCP6022 U8
 U 3 1 60EAAD02
 P 5100 3300
-F 0 "U?" H 5058 3346 50  0000 L CNN
+F 0 "U8" H 5058 3346 50  0000 L CNN
 F 1 "MCP6022" H 5058 3255 50  0000 L CNN
 F 2 "" H 5100 3300 50  0001 C CNN
@@
 AR Path="/60DF1072/60E84E47" Ref="C?"  Part="1"
 AR Path="/60DF1160/60E84E47" Ref="C?"  Part="1"
-AR Path="/60E72FD7/60E84E47" Ref="C?"  Part="1"
+AR Path="/60E72FD7/60E84E47" Ref="C41"  Part="1"
 AR Path="/60EF6B1B/60E84E47" Ref="C?"  Part="1"
-F 0 "C?" H 3115 3396 50  0000 L CNN
+F 0 "C41" H 3115 3396 50  0000 L CNN
 F 1 "0,1" H 3115 3305 50  0000 L CNN
 F 2 "Capacitor_SMD:C_0603_1608Metric_Pad1.08x0.95mm_HandSolder" H 3038 3200 50  0001 C CNN
@@
 AR Path="/60EE89A9/60E9061F" Ref="R?"  Part="1"
 AR Path="/60EF6B1B/60E9061F" Ref="R?"  Part="1"
-AR Path="/60E72FD7/60E9061F" Ref="R?"  Part="1"
-F 0 "R?" H 2070 3796 50  0000 L CNN
+AR Path="/60E72FD7/60E9061F" Ref="R27"  Part="1"
+F 0 "R27" H 2070 3796 50  0000 L CNN
 F 1 "4,7k" H 2070 3705 50  0000 L CNN
 F 2 "Resistor_SMD:R_0603_1608Metric_Pad0.98x0.95mm_HandSolder" V 1930 3750 50  0001 C CNN
@@
 AR Path="/60EE89A9/60E90625" Ref="R?"  Part="1"
 AR Path="/60EF6B1B/60E90625" Ref="R?"  Part="1"
-AR Path="/60E72FD7/60E90625" Ref="R?"  Part="1"
-F 0 "R?" H 1570 3796 50  0000 L CNN
+AR Path="/60E72FD7/60E90625" Ref="R26"  Part="1"
+F 0 "R26" H 1570 3796 50  0000 L CNN
 F 1 "4,7k" H 1570 3705 50  0000 L CNN
 F 2 "Resistor_SMD:R_0603_1608Metric_Pad0.98x0.95mm_HandSolder" V 1430 3750 50  0001 C CNN
@@
 AR Path="/60DF1072/60E9895D" Ref="C?"  Part="1"
 AR Path="/60DF1160/60E9895D" Ref="C?"  Part="1"
-AR Path="/60E72FD7/60E9895D" Ref="C?"  Part="1"
+AR Path="/60E72FD7/60E9895D" Ref="C43"  Part="1"
 AR Path="/60EF6B1B/60E9895D" Ref="C?"  Part="1"
-F 0 "C?" H 6415 3796 50  0000 L CNN
+F 0 "C43" H 6415 3796 50  0000 L CNN
 F 1 "0,1" H 6415 3705 50  0000 L CNN
 F 2 "Capacitor_SMD:C_0603_1608Metric_Pad1.08x0.95mm_HandSolder" H 6338 3600 50  0001 C CNN
@@
 AR Path="/60DF1072/60E99198" Ref="C?"  Part="1"
 AR Path="/60DF1160/60E99198" Ref="C?"  Part="1"
-AR Path="/60E72FD7/60E99198" Ref="C?"  Part="1"
+AR Path="/60E72FD7/60E99198" Ref="C44"  Part="1"
 AR Path="/60EF6B1B/60E99198" Ref="C?"  Part="1"
-F 0 "C?" H 6915 4396 50  0000 L CNN
+F 0 "C44" H 6915 4396 50  0000 L CNN
 F 1 "0,1" H 6915 4305 50  0000 L CNN
 F 2 "Capacitor_SMD:C_0603_1608Metric_Pad1.08x0.95mm_HandSolder" H 6838 4200 50  0001 C CNN
@@
 AR Path="/60EE89A9/60EA0490" Ref="R?"  Part="1"
 AR Path="/60EF6B1B/60EA0490" Ref="R?"  Part="1"
-AR Path="/60E72FD7/60EA0490" Ref="R?"  Part="1"
-F 0 "R?" V 6250 4050 50  0000 L CNN
+AR Path="/60E72FD7/60EA0490" Ref="R28"  Part="1"
+F 0 "R28" V 6250 4050 50  0000 L CNN
 F 1 "1" V 6050 4050 50  0000 L CNN
 F 2 "Resistor_SMD:R_0603_1608Metric_Pad0.98x0.95mm_HandSolder" V 6080 4100 50  0001 C CNN
@@
 AR Path="/60EE89A9/60EA04EE" Ref="R?"  Part="1"
 AR Path="/60EF6B1B/60EA04EE" Ref="R?"  Part="1"
-AR Path="/60E72FD7/60EA04EE" Ref="R?"  Part="1"
-F 0 "R?" V 6750 4050 50  0000 L CNN
+AR Path="/60E72FD7/60EA04EE" Ref="R29"  Part="1"
+F 0 "R29" V 6750 4050 50  0000 L CNN
 F 1 "1" V 6550 4050 50  0000 L CNN
 F 2 "Resistor_SMD:R_0603_1608Metric_Pad0.98x0.95mm_HandSolder" V 6580 4100 50  0001 C CNN
@@
 AR Path="/60EE89A9/60EA070C" Ref="R?"  Part="1"
 AR Path="/60EF6B1B/60EA070C" Ref="R?"  Part="1"
-AR Path="/60E72FD7/60EA070C" Ref="R?"  Part="1"
-F 0 "R?" V 7100 2950 50  0000 L CNN
+AR Path="/60E72FD7/60EA070C" Ref="R30"  Part="1"
+F 0 "R30" V 7100 2950 50  0000 L CNN
 F 1 "0" V 6900 2950 50  0000 L CNN
 F 2 "Resistor_SMD:R_0603_1608Metric_Pad0.98x0.95mm_HandSolder" V 6930 3000 50  0001 C CNN
@@
 AR Path="/60EE89A9/60EDC724" Ref="R?"  Part="1"
 AR Path="/60EF6B1B/60EDC724" Ref="R?"  Part="1"
-AR Path="/60E72FD7/60EDC724" Ref="R?"  Part="1"
-F 0 "R?" H 9320 4396 50  0000 L CNN
+AR Path="/60E72FD7/60EDC724" Ref="R33"  Part="1"
+F 0 "R33" H 9320 4396 50  0000 L CNN
 F 1 "1" H 9320 4305 50  0000 L CNN
 F 2 "Resistor_SMD:R_0603_1608Metric_Pad0.98x0.95mm_HandSolder" V 9180 4350 50  0001 C CNN
@@
 AR Path="/60EE89A9/60EDC768" Ref="R?"  Part="1"
 AR Path="/60EF6B1B/60EDC768" Ref="R?"  Part="1"
-AR Path="/60E72FD7/60EDC768" Ref="R?"  Part="1"
-F 0 "R?" V 9850 3200 50  0000 L CNN
+AR Path="/60E72FD7/60EDC768" Ref="R34"  Part="1"
+F 0 "R34" V 9850 3200 50  0000 L CNN
 F 1 "1" V 9650 3200 50  0000 L CNN
 F 2 "Resistor_SMD:R_0603_1608Metric_Pad0.98x0.95mm_HandSolder" V 9680 3250 50  0001 C CNN
@@
 AR Path="/60EE89A9/60FAA104" Ref="R?"  Part="1"
 AR Path="/60EF6B1B/60FAA104" Ref="R?"  Part="1"
-AR Path="/60E72FD7/60FAA104" Ref="R?"  Part="1"
-F 0 "R?" H 8570 4396 50  0000 L CNN
+AR Path="/60E72FD7/60FAA104" Ref="R31"  Part="1"
+F 0 "R31" H 8570 4396 50  0000 L CNN
 F 1 "1" H 8570 4305 50  0000 L CNN
 F 2 "Resistor_SMD:R_0603_1608Metric_Pad0.98x0.95mm_HandSolder" V 8430 4350 50  0001 C CNN
@@
 AR Path="/60EE89A9/60FAA3D3" Ref="R?"  Part="1"
 AR Path="/60EF6B1B/60FAA3D3" Ref="R?"  Part="1"
-AR Path="/60E72FD7/60FAA3D3" Ref="R?"  Part="1"
-F 0 "R?" H 8570 4796 50  0000 L CNN
+AR Path="/60E72FD7/60FAA3D3" Ref="R32"  Part="1"
+F 0 "R32" H 8570 4796 50  0000 L CNN
 F 1 "1" H 8570 4705 50  0000 L CNN
 F 2 "Resistor_SMD:R_0603_1608Metric_Pad0.98x0.95mm_HandSolder" V 8430 4750 50  0001 C CNN
@@
 P 2200 5400
 AR Path="/60EF6B1B/60FEAD39" Ref="J?"  Part="1"
-AR Path="/60E72FD7/60FEAD39" Ref="J?"  Part="1"
-F 0 "J?" H 2172 5424 50  0000 R CNN
+AR Path="/60E72FD7/60FEAD39" Ref="J7"  Part="1"
+F 0 "J7" H 2172 5424 50  0000 R CNN
 F 1 "Conn_01x03_Male" H 2172 5333 50  0000 R CNN
 F 2 "" H 2200 5400 50  0001 C CNN

Commit message: Add files via upload
Parts:
- C40, C41, C42: symbol Device:C -> rata-rescue:C-Device
- C43, C44: value 0,1 -> 1u; symbol Device:C -> rata-rescue:C-Device
- J7: symbol Connector:Conn_01x03_Male -> rata-rescue:Conn_01x03_Male-Connector
- R26, R27, R30, R31, R32, R33, R34: symbol Device:R -> rata-rescue:R-Device
- R28, R29: value 1 -> 8.2k; symbol Device:R -> rata-rescue:R-Device
- TP15, TP16, TP17: symbol Connector:TestPoint -> rata-rescue:TestPoint-Connector
- U7: symbol Analog_DAC:MCP4725xxx-xCH -> rata-rescue:MCP4725xxx-xCH-Analog_DAC
- U8: symbol Amplifier_Operational:MCP6022 -> rata-rescue:MCP6022-Amplifier_Operational
Other:
- note added: "Low-pass Sallen-Key filter\nfc = 20kHz"
- moved on the sheet: R28, R29
Changed lines of the file:
@@
 $EndDescr
 $Comp
-L Device:C C?
+L rata-rescue:C-Device C?
 U 1 1 60F186C4
 P 2500 3350
@@
 $EndComp
 $Comp
-L Device:C C?
+L rata-rescue:C-Device C?
 U 1 1 60DF1217
 P 4500 3350
@@
 $EndComp
 $Comp
-L Connector:TestPoint TP?
+L rata-rescue:TestPoint-Connector TP?
 U 1 1 60DF1219
 P 5500 4100
@@
 $EndComp
 $Comp
-L Connector:TestPoint TP?
+L rata-rescue:TestPoint-Connector TP?
 U 1 1 60EE8A09
 P 10500 3900
@@
 $EndComp
 $Comp
-L Connector:TestPoint TP?
+L rata-rescue:TestPoint-Connector TP?
 U 1 1 60DF121C
 P 8500 4000
@@
 AUD
 $Comp
-L Analog_DAC:MCP4725xxx-xCH U7
+L rata-rescue:MCP4725xxx-xCH-Analog_DAC U7
 U 1 1 60EA7615
 P 3400 4100
@@
 $EndComp
 $Comp
-L Amplifier_Operational:MCP6022 U8
+L rata-rescue:MCP6022-Amplifier_Operational U8
 U 1 1 60EA87F7
 P 7600 4000
+AR Path="/60EA87F7" Ref="U8"  Part="1"
+AR Path="/60E72FD7/60EA87F7" Ref="U8"  Part="1"
 F 0 "U8" H 7550 3600 50  0000 C CNN
 F 1 "MCP6022" H 7600 3700 50  0000 C CNN
@@
 $EndComp
 $Comp
-L Amplifier_Operational:MCP6022 U8
+L rata-rescue:MCP6022-Amplifier_Operational U8
 U 2 1 60EA9696
 P 9800 3900
+AR Path="/60EA9696" Ref="U8"  Part="2"
+AR Path="/60E72FD7/60EA9696" Ref="U8"  Part="2"
 F 0 "U8" H 9800 3500 50  0000 C CNN
 F 1 "MCP6022" H 9850 3600 50  0000 C CNN
@@
 $EndComp
 $Comp
-L Amplifier_Operational:MCP6022 U8
+L rata-rescue:MCP6022-Amplifier_Operational U8
 U 3 1 60EAAD02
 P 5100 3300
+AR Path="/60EAAD02" Ref="U8"  Part="3"
+AR Path="/60E72FD7/60EAAD02" Ref="U8"  Part="3"
 F 0 "U8" H 5058 3346 50  0000 L CNN
 F 1 "MCP6022" H 5058 3255 50  0000 L CNN
@@
 SCK
 $Comp
-L Device:C C?
+L rata-rescue:C-Device C?
 U 1 1 60E84E47
 P 3000 3350
@@
 $EndComp
 $Comp
-L Device:R R?
+L rata-rescue:R-Device R?
 U 1 1 60E9061F
 P 2000 3750
@@
 $EndComp
 $Comp
-L Device:R R?
+L rata-rescue:R-Device R?
 U 1 1 60E90625
 P 1500 3750
@@
 $EndComp
 $Comp
-L Device:C C?
+L rata-rescue:C-Device C?
 U 1 1 60E9895D
 P 6300 3750
@@
 AR Path="/60EF6B1B/60E9895D" Ref="C?"  Part="1"
 F 0 "C43" H 6415 3796 50  0000 L CNN
-F 1 "0,1" H 6415 3705 50  0000 L CNN
+F 1 "1u" H 6415 3705 50  0000 L CNN
 F 2 "Capacitor_SMD:C_0603_1608Metric_Pad1.08x0.95mm_HandSolder" H 6338 3600 50  0001 C CNN
 F 3 "~" H 6300 3750 50  0001 C CNN
@@
 $EndComp
 $Comp
-L Device:C C?
+L rata-rescue:C-Device C?
 U 1 1 60E99198
 P 6800 4350
@@
 AR Path="/60EF6B1B/60E99198" Ref="C?"  Part="1"
 F 0 "C44" H 6915 4396 50  0000 L CNN
-F 1 "0,1" H 6915 4305 50  0000 L CNN
+F 1 "1u" H 6915 4305 50  0000 L CNN
 F 2 "Capacitor_SMD:C_0603_1608Metric_Pad1.08x0.95mm_HandSolder" H 6838 4200 50  0001 C CNN
 F 3 "~" H 6800 4350 50  0001 C CNN
@@
 $EndComp
 $Comp
-L Device:R R?
+L rata-rescue:R-Device R?
 U 1 1 60EA0490
-P 6150 4100
+P 6050 4100
 AR Path="/60EA0490" Ref="R?"  Part="1"
 AR Path="/60B39FE1/60EA0490" Ref="R?"  Part="1"
@@
 AR Path="/60EF6B1B/60EA0490" Ref="R?"  Part="1"
 AR Path="/60E72FD7/60EA0490" Ref="R28"  Part="1"
-F 0 "R28" V 6250 4050 50  0000 L CNN
-F 1 "1" V 6050 4050 50  0000 L CNN
-F 2 "Resistor_SMD:R_0603_1608Metric_Pad0.98x0.95mm_HandSolder" V 6080 4100 50  0001 C CNN
-F 3 "~" H 6150 4100 50  0001 C CNN
-	1    6150 4100
+F 0 "R28" V 6150 4050 50  0000 L CNN
+F 1 "8.2k" V 5950 4000 50  0000 L CNN
+F 2 "Resistor_SMD:R_0603_1608Metric_Pad0.98x0.95mm_HandSolder" V 5980 4100 50  0001 C CNN
+F 3 "~" H 6050 4100 50  0001 C CNN
+	1    6050 4100
 	0    -1   -1   0
 $EndComp
 $Comp
-L Device:R R?
+L rata-rescue:R-Device R?
 U 1 1 60EA04EE
-P 6650 4100
+P 6550 4100
 AR Path="/60EA04EE" Ref="R?"  Part="1"
 AR Path="/60B39FE1/60EA04EE" Ref="R?"  Part="1"
@@
 AR Path="/60EF6B1B/60EA04EE" Ref="R?"  Part="1"
 AR Path="/60E72FD7/60EA04EE" Ref="R29"  Part="1"
-F 0 "R29" V 6750 4050 50  0000 L CNN
-F 1 "1" V 6550 4050 50  0000 L CNN
-F 2 "Resistor_SMD:R_0603_1608Metric_Pad0.98x0.95mm_HandSolder" V 6580 4100 50  0001 C CNN
-F 3 "~" H 6650 4100 50  0001 C CNN
-	1    6650 4100
+F 0 "R29" V 6650 4050 50  0000 L CNN
+F 1 "8.2k" V 6450 4000 50  0000 L CNN
+F 2 "Resistor_SMD:R_0603_1608Metric_Pad0.98x0.95mm_HandSolder" V 6480 4100 50  0001 C CNN
+F 3 "~" H 6550 4100 50  0001 C CNN
+	1    6550 4100
 	0    -1   -1   0
 $EndComp
 $Comp
-L Device:R R?
+L rata-rescue:R-Device R?
 U 1 1 60EA070C
 P 7000 3000
@@
 $EndComp
 $Comp
-L Device:R R?
+L rata-rescue:R-Device R?
 U 1 1 60EDC724
 P 9250 4350
@@
 $EndComp
 $Comp
-L Device:R R?
+L rata-rescue:R-Device R?
 U 1 1 60EDC768
 P 9750 3250
@@
 	5500 4100 5750 4100
 Wire Wire Line
-	6300 4100 6500 4100
-Wire Wire Line
 	6800 4100 7300 4100
 Wire Wire Line
 	6800 4200 6800 4100
-Connection ~ 6800 4100
-Wire Wire Line
-	6300 3900 6300 4100
-Connection ~ 6300 4100
 Wire Wire Line
 	6300 3600 6300 3500
@@
 Connection ~ 5750 4100
 Wire Wire Line
-	5750 4100 6000 4100
+	5750 4100 5900 4100
 Wire Wire Line
 	7150 3000 8200 3000
@@
 	10250 3900 10500 3900
 $Comp
-L Device:R R?
+L rata-rescue:R-Device R?
 U 1 1 60FAA104
 P 8500 4350
@@
 $EndComp
 $Comp
-L Device:R R?
+L rata-rescue:R-Device R?
 U 1 1 60FAA3D3
 P 8500 4750
@@
 	9250 3800 9250 3250
 $Comp
-L Connector:Conn_01x03_Male J?
+L rata-rescue:Conn_01x03_Male-Connector J?
 U 1 1 60FEAD39
 P 2200 5400
@@
 Wire Wire Line
 	1500 3500 2000 3500
+Wire Wire Line
+	6200 4100 6300 4100
+Wire Wire Line
+	6700 4100 6800 4100
+Connection ~ 6800 4100
+Wire Wire Line
+	6300 3900 6300 4100
+Connection ~ 6300 4100
+Wire Wire Line
+	6300 4100 6400 4100
+Text Notes 7200 4450 0    50   ~ 0
+Low-pass Sallen-Key filter\nfc = 20kHz
 $EndSCHEMATC
