File: DAC.sch (KiCad schematic (older format))
At the start: 20 parts, among them J7 Conn_01x03_Male, U7 MCP4725xxx-xCH, U8 MCP6022

Commit message: Add files via upload
Parts:
- J7: value Conn_01x03_Male -> PLS-3; footprint (none) -> Connector_PinHeader_2.54mm:PinHeader_1x03_P2.54mm_Vertical
- R31: renamed from R30; footprint Resistor_SMD:R_0603_1608Metric_Pad0.98x0.95mm_HandSolder -> Resistor_SMD:R_0805_2012Metric_Pad1.20x1.40mm_HandSolder
- TP15, TP16, TP17: footprint (none) -> rata:TP
- U8: footprint (none) -> Package_SO:SOIC-8_3.9x4.9mm_P1.27mm
- renumbered R26 to R27, R27 to R28, R28 to R29, R29 to R30, R31 to R32, R32 to R33, R33 to R34, R34 to R35
Changed lines of the file:
@@
 encoding utf-8
 Sheet 11 23
-Title ""
-Date ""
-Rev ""
-Comp ""
+Title "rata"
+Date "2021-09-25"
+Rev "1.0"
+Comp "Yuriy Volkov"
 Comment1 ""
 Comment2 ""
@@
 F 0 "TP15" H 5558 4218 50  0000 L CNN
 F 1 "TestPoint" H 5558 4127 50  0001 L CNN
-F 2 "" H 5700 4100 50  0001 C CNN
+F 2 "rata:TP" H 5700 4100 50  0001 C CNN
 F 3 "~" H 5700 4100 50  0001 C CNN
 	1    5500 4100
@@
 F 0 "TP17" H 10558 4018 50  0000 L CNN
 F 1 "TestPoint" H 10558 3927 50  0001 L CNN
-F 2 "" H 10700 3900 50  0001 C CNN
+F 2 "rata:TP" H 10700 3900 50  0001 C CNN
 F 3 "~" H 10700 3900 50  0001 C CNN
 	1    10500 3900
@@
 F 0 "TP16" H 8558 4118 50  0000 L CNN
 F 1 "TestPoint" H 8558 4027 50  0001 L CNN
-F 2 "" H 8700 4000 50  0001 C CNN
+F 2 "rata:TP" H 8700 4000 50  0001 C CNN
 F 3 "~" H 8700 4000 50  0001 C CNN
 	1    8500 4000
@@
 $EndComp
 $Comp
-L rata-rescue:MCP6022-Amplifier_Operational U8
+L rata-rescue:MCP6022-Amplifier_Operational U?
 U 1 1 60EA87F7
 P 7600 4000
-AR Path="/60EA87F7" Ref="U8"  Part="1"
+AR Path="/60EA87F7" Ref="U?"  Part="1"
 AR Path="/60E72FD7/60EA87F7" Ref="U8"  Part="1"
 F 0 "U8" H 7550 3600 50  0000 C CNN
 F 1 "MCP6022" H 7600 3700 50  0000 C CNN
-F 2 "" H 7600 4000 50  0001 C CNN
+F 2 "Package_SO:SOIC-8_3.9x4.9mm_P1.27mm" H 7600 4000 50  0001 C CNN
 F 3 "http://ww1.microchip.com/downloads/en/devicedoc/20001685e.pdf" H 7600 4000 50  0001 C CNN
 	1    7600 4000
@@
 $EndComp
 $Comp
-L rata-rescue:MCP6022-Amplifier_Operational U8
+L rata-rescue:MCP6022-Amplifier_Operational U?
 U 2 1 60EA9696
 P 9800 3900
-AR Path="/60EA9696" Ref="U8"  Part="2"
+AR Path="/60EA9696" Ref="U?"  Part="2"
 AR Path="/60E72FD7/60EA9696" Ref="U8"  Part="2"
 F 0 "U8" H 9800 3500 50  0000 C CNN
 F 1 "MCP6022" H 9850 3600 50  0000 C CNN
-F 2 "" H 9800 3900 50  0001 C CNN
+F 2 "Package_SO:SOIC-8_3.9x4.9mm_P1.27mm" H 9800 3900 50  0001 C CNN
 F 3 "http://ww1.microchip.com/downloads/en/devicedoc/20001685e.pdf" H 9800 3900 50  0001 C CNN
 	2    9800 3900
@@
 $EndComp
 $Comp
-L rata-rescue:MCP6022-Amplifier_Operational U8
+L rata-rescue:MCP6022-Amplifier_Operational U?
 U 3 1 60EAAD02
 P 5100 3300
-AR Path="/60EAAD02" Ref="U8"  Part="3"
+AR Path="/60EAAD02" Ref="U?"  Part="3"
 AR Path="/60E72FD7/60EAAD02" Ref="U8"  Part="3"
 F 0 "U8" H 5058 3346 50  0000 L CNN
 F 1 "MCP6022" H 5058 3255 50  0000 L CNN
-F 2 "" H 5100 3300 50  0001 C CNN
+F 2 "Package_SO:SOIC-8_3.9x4.9mm_P1.27mm" H 5100 3300 50  0001 C CNN
 F 3 "http://ww1.microchip.com/downloads/en/devicedoc/20001685e.pdf" H 5100 3300 50  0001 C CNN
 	3    5100 3300
@@
 AR Path="/60EE89A9/60E9061F" Ref="R?"  Part="1"
 AR Path="/60EF6B1B/60E9061F" Ref="R?"  Part="1"
-AR Path="/60E72FD7/60E9061F" Ref="R27"  Part="1"
-F 0 "R27" H 2070 3796 50  0000 L CNN
+AR Path="/60E72FD7/60E9061F" Ref="R28"  Part="1"
+F 0 "R28" H 2070 3796 50  0000 L CNN
 F 1 "4,7k" H 2070 3705 50  0000 L CNN
 F 2 "Resistor_SMD:R_0603_1608Metric_Pad0.98x0.95mm_HandSolder" V 1930 3750 50  0001 C CNN
@@
 AR Path="/60EE89A9/60E90625" Ref="R?"  Part="1"
 AR Path="/60EF6B1B/60E90625" Ref="R?"  Part="1"
-AR Path="/60E72FD7/60E90625" Ref="R26"  Part="1"
-F 0 "R26" H 1570 3796 50  0000 L CNN
+AR Path="/60E72FD7/60E90625" Ref="R27"  Part="1"
+F 0 "R27" H 1570 3796 50  0000 L CNN
 F 1 "4,7k" H 1570 3705 50  0000 L CNN
 F 2 "Resistor_SMD:R_0603_1608Metric_Pad0.98x0.95mm_HandSolder" V 1430 3750 50  0001 C CNN
@@
 AR Path="/60EE89A9/60EA0490" Ref="R?"  Part="1"
 AR Path="/60EF6B1B/60EA0490" Ref="R?"  Part="1"
-AR Path="/60E72FD7/60EA0490" Ref="R28"  Part="1"
-F 0 "R28" V 6150 4050 50  0000 L CNN
+AR Path="/60E72FD7/60EA0490" Ref="R29"  Part="1"
+F 0 "R29" V 6150 4050 50  0000 L CNN
 F 1 "8.2k" V 5950 4000 50  0000 L CNN
 F 2 "Resistor_SMD:R_0603_1608Metric_Pad0.98x0.95mm_HandSolder" V 5980 4100 50  0001 C CNN
@@
 AR Path="/60EE89A9/60EA04EE" Ref="R?"  Part="1"
 AR Path="/60EF6B1B/60EA04EE" Ref="R?"  Part="1"
-AR Path="/60E72FD7/60EA04EE" Ref="R29"  Part="1"
-F 0 "R29" V 6650 4050 50  0000 L CNN
+AR Path="/60E72FD7/60EA04EE" Ref="R30"  Part="1"
+F 0 "R30" V 6650 4050 50  0000 L CNN
 F 1 "8.2k" V 6450 4000 50  0000 L CNN
 F 2 "Resistor_SMD:R_0603_1608Metric_Pad0.98x0.95mm_HandSolder" V 6480 4100 50  0001 C CNN
@@
 AR Path="/60EE89A9/60EA070C" Ref="R?"  Part="1"
 AR Path="/60EF6B1B/60EA070C" Ref="R?"  Part="1"
-AR Path="/60E72FD7/60EA070C" Ref="R30"  Part="1"
-F 0 "R30" V 7100 2950 50  0000 L CNN
+AR Path="/60E72FD7/60EA070C" Ref="R31"  Part="1"
+F 0 "R31" V 7100 2950 50  0000 L CNN
 F 1 "0" V 6900 2950 50  0000 L CNN
-F 2 "Resistor_SMD:R_0603_1608Metric_Pad0.98x0.95mm_HandSolder" V 6930 3000 50  0001 C CNN
+F 2 "Resistor_SMD:R_0805_2012Metric_Pad1.20x1.40mm_HandSolder" V 6930 3000 50  0001 C CNN
 F 3 "~" H 7000 3000 50  0001 C CNN
 	1    7000 3000
@@
 AR Path="/60EE89A9/60EDC724" Ref="R?"  Part="1"
 AR Path="/60EF6B1B/60EDC724" Ref="R?"  Part="1"
-AR Path="/60E72FD7/60EDC724" Ref="R33"  Part="1"
-F 0 "R33" H 9320 4396 50  0000 L CNN
+AR Path="/60E72FD7/60EDC724" Ref="R34"  Part="1"
+F 0 "R34" H 9320 4396 50  0000 L CNN
 F 1 "1" H 9320 4305 50  0000 L CNN
 F 2 "Resistor_SMD:R_0603_1608Metric_Pad0.98x0.95mm_HandSolder" V 9180 4350 50  0001 C CNN
@@
 AR Path="/60EE89A9/60EDC768" Ref="R?"  Part="1"
 AR Path="/60EF6B1B/60EDC768" Ref="R?"  Part="1"
-AR Path="/60E72FD7/60EDC768" Ref="R34"  Part="1"
-F 0 "R34" V 9850 3200 50  0000 L CNN
+AR Path="/60E72FD7/60EDC768" Ref="R35"  Part="1"
+F 0 "R35" V 9850 3200 50  0000 L CNN
 F 1 "1" V 9650 3200 50  0000 L CNN
 F 2 "Resistor_SMD:R_0603_1608Metric_Pad0.98x0.95mm_HandSolder" V 9680 3250 50  0001 C CNN
@@
 AR Path="/60EE89A9/60FAA104" Ref="R?"  Part="1"
 AR Path="/60EF6B1B/60FAA104" Ref="R?"  Part="1"
-AR Path="/60E72FD7/60FAA104" Ref="R31"  Part="1"
-F 0 "R31" H 8570 4396 50  0000 L CNN
+AR Path="/60E72FD7/60FAA104" Ref="R32"  Part="1"
+F 0 "R32" H 8570 4396 50  0000 L CNN
 F 1 "1" H 8570 4305 50  0000 L CNN
 F 2 "Resistor_SMD:R_0603_1608Metric_Pad0.98x0.95mm_HandSolder" V 8430 4350 50  0001 C CNN
@@
 AR Path="/60EE89A9/60FAA3D3" Ref="R?"  Part="1"
 AR Path="/60EF6B1B/60FAA3D3" Ref="R?"  Part="1"
-AR Path="/60E72FD7/60FAA3D3" Ref="R32"  Part="1"
-F 0 "R32" H 8570 4796 50  0000 L CNN
+AR Path="/60E72FD7/60FAA3D3" Ref="R33"  Part="1"
+F 0 "R33" H 8570 4796 50  0000 L CNN
 F 1 "1" H 8570 4705 50  0000 L CNN
 F 2 "Resistor_SMD:R_0603_1608Metric_Pad0.98x0.95mm_HandSolder" V 8430 4750 50  0001 C CNN
@@
 AR Path="/60E72FD7/60FEAD39" Ref="J7"  Part="1"
 F 0 "J7" H 2172 5424 50  0000 R CNN
-F 1 "Conn_01x03_Male" H 2172 5333 50  0000 R CNN
-F 2 "" H 2200 5400 50  0001 C CNN
+F 1 "PLS-3" H 2172 5333 50  0000 R CNN
+F 2 "Connector_PinHeader_2.54mm:PinHeader_1x03_P2.54mm_Vertical" H 2200 5400 50  0001 C CNN
 F 3 "~" H 2200 5400 50  0001 C CNN
 	1    2200 5400
