File: DAC.sch (KiCad schematic (older format))
At the start: 20 parts, among them J7 PLS-3, U7 MCP4725xxx-xCH, U8 MCP6022

Commit message: Resistors values corrected to correspond actual values
Parts:
- C43, C44: value 1u -> 1000
- R32, R35: value 1 -> 0
- R33, R34: value 1 -> -
Changed lines of the file:
@@
 AR Path="/60EF6B1B/60E9895D" Ref="C?"  Part="1"
 F 0 "C43" H 6415 3796 50  0000 L CNN
-F 1 "1u" H 6415 3705 50  0000 L CNN
+F 1 "1000" H 6415 3705 50  0000 L CNN
 F 2 "Capacitor_SMD:C_0603_1608Metric_Pad1.08x0.95mm_HandSolder" H 6338 3600 50  0001 C CNN
 F 3 "~" H 6300 3750 50  0001 C CNN
@@
 AR Path="/60EF6B1B/60E99198" Ref="C?"  Part="1"
 F 0 "C44" H 6915 4396 50  0000 L CNN
-F 1 "1u" H 6915 4305 50  0000 L CNN
+F 1 "1000" H 6915 4305 50  0000 L CNN
 F 2 "Capacitor_SMD:C_0603_1608Metric_Pad1.08x0.95mm_HandSolder" H 6838 4200 50  0001 C CNN
 F 3 "~" H 6800 4350 50  0001 C CNN
@@
 AR Path="/60E72FD7/60EDC724" Ref="R34"  Part="1"
 F 0 "R34" H 9320 4396 50  0000 L CNN
-F 1 "1" H 9320 4305 50  0000 L CNN
+F 1 "-" H 9320 4305 50  0000 L CNN
 F 2 "Resistor_SMD:R_0603_1608Metric_Pad0.98x0.95mm_HandSolder" V 9180 4350 50  0001 C CNN
 F 3 "~" H 9250 4350 50  0001 C CNN
@@
 AR Path="/60E72FD7/60EDC768" Ref="R35"  Part="1"
 F 0 "R35" V 9850 3200 50  0000 L CNN
-F 1 "1" V 9650 3200 50  0000 L CNN
+F 1 "0" V 9650 3200 50  0000 L CNN
 F 2 "Resistor_SMD:R_0603_1608Metric_Pad0.98x0.95mm_HandSolder" V 9680 3250 50  0001 C CNN
 F 3 "~" H 9750 3250 50  0001 C CNN
@@
 AR Path="/60E72FD7/60FAA104" Ref="R32"  Part="1"
 F 0 "R32" H 8570 4396 50  0000 L CNN
-F 1 "1" H 8570 4305 50  0000 L CNN
+F 1 "0" H 8570 4305 50  0000 L CNN
 F 2 "Resistor_SMD:R_0603_1608Metric_Pad0.98x0.95mm_HandSolder" V 8430 4350 50  0001 C CNN
 F 3 "~" H 8500 4350 50  0001 C CNN
@@
 AR Path="/60E72FD7/60FAA3D3" Ref="R33"  Part="1"
 F 0 "R33" H 8570 4796 50  0000 L CNN
-F 1 "1" H 8570 4705 50  0000 L CNN
+F 1 "-" H 8570 4705 50  0000 L CNN
 F 2 "Resistor_SMD:R_0603_1608Metric_Pad0.98x0.95mm_HandSolder" V 8430 4750 50  0001 C CNN
 F 3 "~" H 8500 4750 50  0001 C CNN
