File: Emitter_follower.sch (KiCad schematic (older format))
At the start: 7 parts

Commit message: Add files via upload
Parts:
- R88, R90, R91: renamed from R?; value 3.3k -> 4.7k
- gave numbers to parts that had none: 4
Changed lines of the file:
@@
 $Descr A4 11693 8268
 encoding utf-8
-Sheet 20 23
+Sheet 22 23
 Title ""
 Date ""
@@
 AR Path="/609FED99/60F64272" Ref="Q?"  Part="1"
 AR Path="/60F18EC1/60F64272" Ref="Q?"  Part="1"
-AR Path="/60F18EC1/60F620C8/60F64272" Ref="Q?"  Part="1"
-AR Path="/60F18EC1/60F77249/60F64272" Ref="Q?"  Part="1"
-AR Path="/60F18EC1/60F77470/60F64272" Ref="Q?"  Part="1"
-AR Path="/60F18EC1/60F77508/60F64272" Ref="Q?"  Part="1"
-F 0 "Q?" H 7091 3796 50  0000 L CNN
+AR Path="/60F18EC1/60F620C8/60F64272" Ref="Q9"  Part="1"
+AR Path="/60F18EC1/60F77249/60F64272" Ref="Q12"  Part="1"
+AR Path="/60F18EC1/60F77470/60F64272" Ref="Q15"  Part="1"
+AR Path="/60F18EC1/60F77508/60F64272" Ref="Q18"  Part="1"
+F 0 "Q18" H 7091 3796 50  0000 L CNN
 F 1 "BC847" H 7091 3705 50  0000 L CNN
 F 2 "Package_TO_SOT_SMD:SOT-23" H 7100 3675 50  0001 L CIN
@@
 AR Path="/609FED99/60F64278" Ref="R?"  Part="1"
 AR Path="/60F18EC1/60F64278" Ref="R?"  Part="1"
-AR Path="/60F18EC1/60F620C8/60F64278" Ref="R?"  Part="1"
-AR Path="/60F18EC1/60F77249/60F64278" Ref="R?"  Part="1"
-AR Path="/60F18EC1/60F77470/60F64278" Ref="R?"  Part="1"
-AR Path="/60F18EC1/60F77508/60F64278" Ref="R?"  Part="1"
-F 0 "R?" H 5570 4796 50  0000 L CNN
+AR Path="/60F18EC1/60F620C8/60F64278" Ref="R89"  Part="1"
+AR Path="/60F18EC1/60F77249/60F64278" Ref="R93"  Part="1"
+AR Path="/60F18EC1/60F77470/60F64278" Ref="R97"  Part="1"
+AR Path="/60F18EC1/60F77508/60F64278" Ref="R101"  Part="1"
+F 0 "R101" H 5570 4796 50  0000 L CNN
 F 1 "56k" H 5570 4705 50  0000 L CNN
 F 2 "Resistor_SMD:R_0603_1608Metric_Pad0.98x0.95mm_HandSolder" V 5430 4750 50  0001 C CNN
@@
 AR Path="/609FED99/60F6427E" Ref="R?"  Part="1"
 AR Path="/60F18EC1/60F6427E" Ref="R?"  Part="1"
-AR Path="/60F18EC1/60F620C8/60F6427E" Ref="R?"  Part="1"
-AR Path="/60F18EC1/60F77249/60F6427E" Ref="R?"  Part="1"
-AR Path="/60F18EC1/60F77470/60F6427E" Ref="R?"  Part="1"
-AR Path="/60F18EC1/60F77508/60F6427E" Ref="R?"  Part="1"
-F 0 "R?" V 5350 4450 50  0000 L CNN
-F 1 "3.3k" V 5150 4400 50  0000 L CNN
+AR Path="/60F18EC1/60F620C8/60F6427E" Ref="R88"  Part="1"
+AR Path="/60F18EC1/60F77249/60F6427E" Ref="R92"  Part="1"
+AR Path="/60F18EC1/60F77470/60F6427E" Ref="R96"  Part="1"
+AR Path="/60F18EC1/60F77508/60F6427E" Ref="R100"  Part="1"
+F 0 "R100" V 5350 4450 50  0000 L CNN
+F 1 "4.7k" V 5150 4400 50  0000 L CNN
 F 2 "Resistor_SMD:R_0603_1608Metric_Pad0.98x0.95mm_HandSolder" V 5180 4500 50  0001 C CNN
 F 3 "~" H 5250 4500 50  0001 C CNN
@@
 P 6900 4250
 AR Path="/60F18EC1/60F64284" Ref="Q?"  Part="1"
-AR Path="/60F18EC1/60F620C8/60F64284" Ref="Q?"  Part="1"
-AR Path="/60F18EC1/60F77249/60F64284" Ref="Q?"  Part="1"
-AR Path="/60F18EC1/60F77470/60F64284" Ref="Q?"  Part="1"
-AR Path="/60F18EC1/60F77508/60F64284" Ref="Q?"  Part="1"
-F 0 "Q?" H 7091 4204 50  0000 L CNN
+AR Path="/60F18EC1/60F620C8/60F64284" Ref="Q10"  Part="1"
+AR Path="/60F18EC1/60F77249/60F64284" Ref="Q13"  Part="1"
+AR Path="/60F18EC1/60F77470/60F64284" Ref="Q16"  Part="1"
+AR Path="/60F18EC1/60F77508/60F64284" Ref="Q19"  Part="1"
+F 0 "Q19" H 7091 4204 50  0000 L CNN
 F 1 "BC857" H 7091 4295 50  0000 L CNN
 F 2 "Package_TO_SOT_SMD:SOT-23" H 7100 4175 50  0001 L CIN
@@
 AR Path="/609FED99/60F64A50" Ref="Q?"  Part="1"
 AR Path="/60F18EC1/60F64A50" Ref="Q?"  Part="1"
-AR Path="/60F18EC1/60F620C8/60F64A50" Ref="Q?"  Part="1"
-AR Path="/60F18EC1/60F77249/60F64A50" Ref="Q?"  Part="1"
-AR Path="/60F18EC1/60F77470/60F64A50" Ref="Q?"  Part="1"
-AR Path="/60F18EC1/60F77508/60F64A50" Ref="Q?"  Part="1"
-F 0 "Q?" H 6091 4546 50  0000 L CNN
+AR Path="/60F18EC1/60F620C8/60F64A50" Ref="Q8"  Part="1"
+AR Path="/60F18EC1/60F77249/60F64A50" Ref="Q11"  Part="1"
+AR Path="/60F18EC1/60F77470/60F64A50" Ref="Q14"  Part="1"
+AR Path="/60F18EC1/60F77508/60F64A50" Ref="Q17"  Part="1"
+F 0 "Q17" H 6091 4546 50  0000 L CNN
 F 1 "BC847" H 6091 4455 50  0000 L CNN
 F 2 "Package_TO_SOT_SMD:SOT-23" H 6100 4425 50  0001 L CIN
@@
 AR Path="/609FED99/60F68AA3" Ref="R?"  Part="1"
 AR Path="/60F18EC1/60F68AA3" Ref="R?"  Part="1"
-AR Path="/60F18EC1/60F620C8/60F68AA3" Ref="R?"  Part="1"
-AR Path="/60F18EC1/60F77249/60F68AA3" Ref="R?"  Part="1"
-AR Path="/60F18EC1/60F77470/60F68AA3" Ref="R?"  Part="1"
-AR Path="/60F18EC1/60F77508/60F68AA3" Ref="R?"  Part="1"
-F 0 "R?" V 6450 3950 50  0000 L CNN
-F 1 "3.3k" V 6250 3900 50  0000 L CNN
+AR Path="/60F18EC1/60F620C8/60F68AA3" Ref="R91"  Part="1"
+AR Path="/60F18EC1/60F77249/60F68AA3" Ref="R95"  Part="1"
+AR Path="/60F18EC1/60F77470/60F68AA3" Ref="R99"  Part="1"
+AR Path="/60F18EC1/60F77508/60F68AA3" Ref="R103"  Part="1"
+F 0 "R103" V 6450 3950 50  0000 L CNN
+F 1 "4.7k" V 6250 3900 50  0000 L CNN
 F 2 "Resistor_SMD:R_0603_1608Metric_Pad0.98x0.95mm_HandSolder" V 6280 4000 50  0001 C CNN
 F 3 "~" H 6350 4000 50  0001 C CNN
@@
 AR Path="/609FED99/60F6906A" Ref="R?"  Part="1"
 AR Path="/60F18EC1/60F6906A" Ref="R?"  Part="1"
-AR Path="/60F18EC1/60F620C8/60F6906A" Ref="R?"  Part="1"
-AR Path="/60F18EC1/60F77249/60F6906A" Ref="R?"  Part="1"
-AR Path="/60F18EC1/60F77470/60F6906A" Ref="R?"  Part="1"
-AR Path="/60F18EC1/60F77508/60F6906A" Ref="R?"  Part="1"
-F 0 "R?" H 6070 3796 50  0000 L CNN
-F 1 "3.3k" H 6070 3705 50  0000 L CNN
+AR Path="/60F18EC1/60F620C8/60F6906A" Ref="R90"  Part="1"
+AR Path="/60F18EC1/60F77249/60F6906A" Ref="R94"  Part="1"
+AR Path="/60F18EC1/60F77470/60F6906A" Ref="R98"  Part="1"
+AR Path="/60F18EC1/60F77508/60F6906A" Ref="R102"  Part="1"
+F 0 "R102" H 6070 3796 50  0000 L CNN
+F 1 "4.7k" H 6070 3705 50  0000 L CNN
 F 2 "Resistor_SMD:R_0603_1608Metric_Pad0.98x0.95mm_HandSolder" V 5930 3750 50  0001 C CNN
 F 3 "~" H 6000 3750 50  0001 C CNN

Commit message: Add files via upload
Parts:
- Q10: symbol Transistor_BJT:BC857 -> rata-rescue:BC857-Transistor_BJT
- Q8, Q9: symbol Transistor_BJT:BC847 -> rata-rescue:BC847-Transistor_BJT
- R88, R89, R90, R91: symbol Device:R -> rata-rescue:R-Device
Changed lines of the file:
@@
 $EndDescr
 $Comp
-L Transistor_BJT:BC847 Q?
+L rata-rescue:BC847-Transistor_BJT Q?
 U 1 1 60F64272
 P 6900 3750
@@
 $EndComp
 $Comp
-L Device:R R?
+L rata-rescue:R-Device R?
 U 1 1 60F64278
 P 5500 4750
@@
 $EndComp
 $Comp
-L Device:R R?
+L rata-rescue:R-Device R?
 U 1 1 60F6427E
 P 5250 4500
@@
 $EndComp
 $Comp
-L Transistor_BJT:BC857 Q?
+L rata-rescue:BC857-Transistor_BJT Q?
 U 1 1 60F64284
 P 6900 4250
@@
 Double emitter follower
 $Comp
-L Transistor_BJT:BC847 Q?
+L rata-rescue:BC847-Transistor_BJT Q?
 U 1 1 60F64A50
 P 5900 4500
@@
 $EndComp
 $Comp
-L Device:R R?
+L rata-rescue:R-Device R?
 U 1 1 60F68AA3
 P 6350 4000
@@
 $EndComp
 $Comp
-L Device:R R?
+L rata-rescue:R-Device R?
 U 1 1 60F6906A
 P 6000 3750

Commit message: Add files via upload
Parts:
- renumbered R88 to R59, R89 to R60, R90 to R61, R91 to R62
Changed lines of the file:
@@
 $Descr A4 11693 8268
 encoding utf-8
-Sheet 22 23
-Title ""
-Date ""
-Rev ""
-Comp ""
+Sheet 18 23
+Title "rata"
+Date "2021-09-25"
+Rev "1.0"
+Comp "Yuriy Volkov"
 Comment1 ""
 Comment2 ""
@@
 AR Path="/60F18EC1/60F77470/60F64272" Ref="Q15"  Part="1"
 AR Path="/60F18EC1/60F77508/60F64272" Ref="Q18"  Part="1"
-F 0 "Q18" H 7091 3796 50  0000 L CNN
+F 0 "Q9" H 7091 3796 50  0000 L CNN
 F 1 "BC847" H 7091 3705 50  0000 L CNN
 F 2 "Package_TO_SOT_SMD:SOT-23" H 7100 3675 50  0001 L CIN
@@
 AR Path="/609FED99/60F64278" Ref="R?"  Part="1"
 AR Path="/60F18EC1/60F64278" Ref="R?"  Part="1"
-AR Path="/60F18EC1/60F620C8/60F64278" Ref="R89"  Part="1"
-AR Path="/60F18EC1/60F77249/60F64278" Ref="R93"  Part="1"
-AR Path="/60F18EC1/60F77470/60F64278" Ref="R97"  Part="1"
-AR Path="/60F18EC1/60F77508/60F64278" Ref="R101"  Part="1"
-F 0 "R101" H 5570 4796 50  0000 L CNN
+AR Path="/60F18EC1/60F620C8/60F64278" Ref="R60"  Part="1"
+AR Path="/60F18EC1/60F77249/60F64278" Ref="R64"  Part="1"
+AR Path="/60F18EC1/60F77470/60F64278" Ref="R68"  Part="1"
+AR Path="/60F18EC1/60F77508/60F64278" Ref="R72"  Part="1"
+F 0 "R60" H 5570 4796 50  0000 L CNN
 F 1 "56k" H 5570 4705 50  0000 L CNN
 F 2 "Resistor_SMD:R_0603_1608Metric_Pad0.98x0.95mm_HandSolder" V 5430 4750 50  0001 C CNN
@@
 AR Path="/609FED99/60F6427E" Ref="R?"  Part="1"
 AR Path="/60F18EC1/60F6427E" Ref="R?"  Part="1"
-AR Path="/60F18EC1/60F620C8/60F6427E" Ref="R88"  Part="1"
-AR Path="/60F18EC1/60F77249/60F6427E" Ref="R92"  Part="1"
-AR Path="/60F18EC1/60F77470/60F6427E" Ref="R96"  Part="1"
-AR Path="/60F18EC1/60F77508/60F6427E" Ref="R100"  Part="1"
-F 0 "R100" V 5350 4450 50  0000 L CNN
+AR Path="/60F18EC1/60F620C8/60F6427E" Ref="R59"  Part="1"
+AR Path="/60F18EC1/60F77249/60F6427E" Ref="R63"  Part="1"
+AR Path="/60F18EC1/60F77470/60F6427E" Ref="R67"  Part="1"
+AR Path="/60F18EC1/60F77508/60F6427E" Ref="R71"  Part="1"
+F 0 "R59" V 5350 4450 50  0000 L CNN
 F 1 "4.7k" V 5150 4400 50  0000 L CNN
 F 2 "Resistor_SMD:R_0603_1608Metric_Pad0.98x0.95mm_HandSolder" V 5180 4500 50  0001 C CNN
@@
 AR Path="/60F18EC1/60F77470/60F64284" Ref="Q16"  Part="1"
 AR Path="/60F18EC1/60F77508/60F64284" Ref="Q19"  Part="1"
-F 0 "Q19" H 7091 4204 50  0000 L CNN
+F 0 "Q10" H 7091 4204 50  0000 L CNN
 F 1 "BC857" H 7091 4295 50  0000 L CNN
 F 2 "Package_TO_SOT_SMD:SOT-23" H 7100 4175 50  0001 L CIN
@@
 AR Path="/60F18EC1/60F77470/60F64A50" Ref="Q14"  Part="1"
 AR Path="/60F18EC1/60F77508/60F64A50" Ref="Q17"  Part="1"
-F 0 "Q17" H 6091 4546 50  0000 L CNN
+F 0 "Q8" H 6091 4546 50  0000 L CNN
 F 1 "BC847" H 6091 4455 50  0000 L CNN
 F 2 "Package_TO_SOT_SMD:SOT-23" H 6100 4425 50  0001 L CIN
@@
 AR Path="/609FED99/60F68AA3" Ref="R?"  Part="1"
 AR Path="/60F18EC1/60F68AA3" Ref="R?"  Part="1"
-AR Path="/60F18EC1/60F620C8/60F68AA3" Ref="R91"  Part="1"
-AR Path="/60F18EC1/60F77249/60F68AA3" Ref="R95"  Part="1"
-AR Path="/60F18EC1/60F77470/60F68AA3" Ref="R99"  Part="1"
-AR Path="/60F18EC1/60F77508/60F68AA3" Ref="R103"  Part="1"
-F 0 "R103" V 6450 3950 50  0000 L CNN
+AR Path="/60F18EC1/60F620C8/60F68AA3" Ref="R62"  Part="1"
+AR Path="/60F18EC1/60F77249/60F68AA3" Ref="R66"  Part="1"
+AR Path="/60F18EC1/60F77470/60F68AA3" Ref="R70"  Part="1"
+AR Path="/60F18EC1/60F77508/60F68AA3" Ref="R74"  Part="1"
+F 0 "R62" V 6450 3950 50  0000 L CNN
 F 1 "4.7k" V 6250 3900 50  0000 L CNN
 F 2 "Resistor_SMD:R_0603_1608Metric_Pad0.98x0.95mm_HandSolder" V 6280 4000 50  0001 C CNN
@@
 AR Path="/609FED99/60F6906A" Ref="R?"  Part="1"
 AR Path="/60F18EC1/60F6906A" Ref="R?"  Part="1"
-AR Path="/60F18EC1/60F620C8/60F6906A" Ref="R90"  Part="1"
-AR Path="/60F18EC1/60F77249/60F6906A" Ref="R94"  Part="1"
-AR Path="/60F18EC1/60F77470/60F6906A" Ref="R98"  Part="1"
-AR Path="/60F18EC1/60F77508/60F6906A" Ref="R102"  Part="1"
-F 0 "R102" H 6070 3796 50  0000 L CNN
+AR Path="/60F18EC1/60F620C8/60F6906A" Ref="R61"  Part="1"
+AR Path="/60F18EC1/60F77249/60F6906A" Ref="R65"  Part="1"
+AR Path="/60F18EC1/60F77470/60F6906A" Ref="R69"  Part="1"
+AR Path="/60F18EC1/60F77508/60F6906A" Ref="R73"  Part="1"
+F 0 "R61" H 6070 3796 50  0000 L CNN
 F 1 "4.7k" H 6070 3705 50  0000 L CNN
 F 2 "Resistor_SMD:R_0603_1608Metric_Pad0.98x0.95mm_HandSolder" V 5930 3750 50  0001 C CNN
