File: Light_sensor.sch (KiCad schematic (older format))
At the start: 12 parts

Commit message: Add files via upload
Parts:
- removed C?: 1u, Capacitor_SMD:C_0603_1608Metric_Pad1.08x0.95mm_HandSolder, symbol Device:C
- removed C? (x2): 10u, Capacitor_SMD:C_1206_3216Metric_Pad1.33x1.80mm_HandSolder, symbol Device:C
- removed C?: 100u, symbol Device:CP
- removed D?: SMAJ5.0CA, symbol Device:D_TVS
- removed TP? (x2): TestPoint, symbol Connector:TestPoint
- removed U?: AMS1117-3.3, Package_TO_SOT_SMD:SOT-223-3_TabPin2, symbol Regulator_Linear:AMS1117-3.3
- removed U?: LM321, Package_TO_SOT_SMD:SOT-23-5, symbol Amplifier_Operational:LM321
- added R?: 1k, Resistor_SMD:R_0603_1608Metric_Pad0.98x0.95mm_HandSolder, symbol Device:R
- added R?: 10k, Resistor_SMD:R_0603_1608Metric_Pad0.98x0.95mm_HandSolder, symbol Device:R
- added TP?: TestPoint, symbol Connector:TestPoint
- C?: value 0,1 -> 1u
- Q?: value SFH300 -> SFH3310
Connections:
- net labels added: +3V3, VOLT
- net labels removed: +3V3_OUT, +5V_IN
- wire segments 18 -> 14
Other:
- note added: "Light level sensor"
- note removed: "Power source +3V3"
- moved on the sheet: C?, Q?, TP?

Commit message: Add files via upload
Parts:
- R49: renamed from R?; value 10k -> 4.7k
- gave numbers to parts that had none: 5
Changed lines of the file:
@@
 $Descr A4 11693 8268
 encoding utf-8
-Sheet 16 23
+Sheet 15 23
 Title ""
 Date ""
@@
 AR Path="/60DF196E/60F26C9D" Ref="C?"  Part="1"
 AR Path="/60DF212D/60F26C9D" Ref="C?"  Part="1"
-AR Path="/60F197D4/60F26C9D" Ref="C?"  Part="1"
+AR Path="/60F197D4/60F26C9D" Ref="C54"  Part="1"
 AR Path="/60F1A0E6/60F26C9D" Ref="C?"  Part="1"
-F 0 "C?" H 6615 4796 50  0000 L CNN
+F 0 "C54" H 6615 4796 50  0000 L CNN
 F 1 "1u" H 6615 4705 50  0000 L CNN
 F 2 "Capacitor_SMD:C_0603_1608Metric_Pad1.08x0.95mm_HandSolder" H 6538 4600 50  0001 C CNN
@@
 AR Path="/60DF196E/60F1A12F" Ref="TP?"  Part="1"
 AR Path="/60DF212D/60F1A12F" Ref="TP?"  Part="1"
-AR Path="/60F197D4/60F1A12F" Ref="TP?"  Part="1"
+AR Path="/60F197D4/60F1A12F" Ref="TP22"  Part="1"
 AR Path="/60F1A0E6/60F1A12F" Ref="TP?"  Part="1"
-F 0 "TP?" H 5558 4618 50  0000 L CNN
+F 0 "TP22" H 5558 4618 50  0000 L CNN
 F 1 "TestPoint" H 5558 4527 50  0001 L CNN
 F 2 "" H 5700 4500 50  0001 C CNN
@@
 VOLT
 $Comp
-L Sensor_Optical:SFH300 Q?
+L Sensor_Optical:SFH300 Q3
 U 1 1 60F482D9
 P 4900 4200
-F 0 "Q?" H 5090 4246 50  0000 L CNN
+F 0 "Q3" H 5090 4246 50  0000 L CNN
 F 1 "SFH3310" H 5090 4155 50  0000 L CNN
 F 2 "LED_THT:LED_D5.0mm_Clear" H 5380 4060 50  0001 C CNN
@@
 AR Path="/60DF1160/60F2690B/6100D3B1" Ref="R?"  Part="1"
 AR Path="/60DF1160/6100D3B1" Ref="R?"  Part="1"
-AR Path="/60F197D4/6100D3B1" Ref="R?"  Part="1"
-F 0 "R?" H 5070 4796 50  0000 L CNN
+AR Path="/60F197D4/6100D3B1" Ref="R48"  Part="1"
+F 0 "R48" H 5070 4796 50  0000 L CNN
 F 1 "1k" H 5070 4705 50  0000 L CNN
 F 2 "Resistor_SMD:R_0603_1608Metric_Pad0.98x0.95mm_HandSolder" V 4930 4750 50  0001 C CNN
@@
 AR Path="/60DF1160/60F2690B/6100EF4A" Ref="R?"  Part="1"
 AR Path="/60DF1160/6100EF4A" Ref="R?"  Part="1"
-AR Path="/60F197D4/6100EF4A" Ref="R?"  Part="1"
-F 0 "R?" V 6350 4450 50  0000 L CNN
-F 1 "10k" V 6150 4400 50  0000 L CNN
+AR Path="/60F197D4/6100EF4A" Ref="R49"  Part="1"
+F 0 "R49" V 6350 4450 50  0000 L CNN
+F 1 "4.7k" V 6150 4400 50  0000 L CNN
 F 2 "Resistor_SMD:R_0603_1608Metric_Pad0.98x0.95mm_HandSolder" V 6180 4500 50  0001 C CNN
 F 3 "~" H 6250 4500 50  0001 C CNN
@@
 AR Path="/60DF196E/61013214" Ref="TP?"  Part="1"
 AR Path="/60DF212D/61013214" Ref="TP?"  Part="1"
-AR Path="/60F197D4/61013214" Ref="TP?"  Part="1"
+AR Path="/60F197D4/61013214" Ref="TP23"  Part="1"
 AR Path="/60F1A0E6/61013214" Ref="TP?"  Part="1"
-F 0 "TP?" H 7058 4618 50  0000 L CNN
+F 0 "TP23" H 7058 4618 50  0000 L CNN
 F 1 "TestPoint" H 7058 4527 50  0001 L CNN
 F 2 "" H 7200 4500 50  0001 C CNN

Commit message: Add files via upload
Parts:
- C54: symbol Device:C -> rata-rescue:C-Device
- Q3: symbol Sensor_Optical:SFH300 -> rata-rescue:SFH300-Sensor_Optical
- R48, R49: symbol Device:R -> rata-rescue:R-Device
- TP22, TP23: symbol Connector:TestPoint -> rata-rescue:TestPoint-Connector
Changed lines of the file:
@@
 $EndDescr
 $Comp
-L Device:C C?
+L rata-rescue:C-Device C?
 U 1 1 60F26C9D
 P 6500 4750
@@
 $EndComp
 $Comp
-L Connector:TestPoint TP?
+L rata-rescue:TestPoint-Connector TP?
 U 1 1 60F1A12F
 P 5500 4500
@@
 VOLT
 $Comp
-L Sensor_Optical:SFH300 Q3
+L rata-rescue:SFH300-Sensor_Optical Q3
 U 1 1 60F482D9
 P 4900 4200
@@
 $EndComp
 $Comp
-L Device:R R?
+L rata-rescue:R-Device R?
 U 1 1 6100D3B1
 P 5000 4750
@@
 $EndComp
 $Comp
-L Device:R R?
+L rata-rescue:R-Device R?
 U 1 1 6100EF4A
 P 6250 4500
@@
 $EndComp
 $Comp
-L Connector:TestPoint TP?
+L rata-rescue:TestPoint-Connector TP?
 U 1 1 61013214
 P 7000 4500

Commit message: Add files via upload
Parts:
- added C54: 0.1u, Capacitor_SMD:C_0603_1608Metric_Pad1.08x0.95mm_HandSolder, symbol rata-rescue:C-Device
- Q3: footprint LED_THT:LED_D5.0mm_Clear -> LED_THT:LED_D3.0mm_Horizontal_O1.27mm_Z2.0mm_Clear
- TP22, TP23: footprint (none) -> rata:TP
- renumbered C54 to C55, R48 to R49, R49 to R50
Connections:
- net +3V3: now also C54.1
- net GND: now also C54.2
Other:
- moved on the sheet: C55, Q3, R49, R50, TP22, TP23
Changed lines of the file:
@@
 encoding utf-8
 Sheet 15 23
-Title ""
-Date ""
-Rev ""
-Comp ""
+Title "rata"
+Date "2021-09-25"
+Rev "1.0"
+Comp "Yuriy Volkov"
 Comment1 ""
 Comment2 ""
@@
 L rata-rescue:C-Device C?
 U 1 1 60F26C9D
-P 6500 4750
+P 7000 4750
 AR Path="/60F26C9D" Ref="C?"  Part="1"
 AR Path="/609CA6A8/609D24C0/60F26C9D" Ref="C?"  Part="1"
@@
 AR Path="/60DF196E/60F26C9D" Ref="C?"  Part="1"
 AR Path="/60DF212D/60F26C9D" Ref="C?"  Part="1"
-AR Path="/60F197D4/60F26C9D" Ref="C54"  Part="1"
+AR Path="/60F197D4/60F26C9D" Ref="C55"  Part="1"
 AR Path="/60F1A0E6/60F26C9D" Ref="C?"  Part="1"
-F 0 "C54" H 6615 4796 50  0000 L CNN
-F 1 "1u" H 6615 4705 50  0000 L CNN
-F 2 "Capacitor_SMD:C_0603_1608Metric_Pad1.08x0.95mm_HandSolder" H 6538 4600 50  0001 C CNN
-F 3 "~" H 6500 4750 50  0001 C CNN
-	1    6500 4750
+F 0 "C55" H 7115 4796 50  0000 L CNN
+F 1 "1u" H 7115 4705 50  0000 L CNN
+F 2 "Capacitor_SMD:C_0603_1608Metric_Pad1.08x0.95mm_HandSolder" H 7038 4600 50  0001 C CNN
+F 3 "~" H 7000 4750 50  0001 C CNN
+	1    7000 4750
 	1    0    0    -1
 $EndComp
@@
 L rata-rescue:TestPoint-Connector TP?
 U 1 1 60F1A12F
-P 5500 4500
+P 6000 4500
 AR Path="/60F1A12F" Ref="TP?"  Part="1"
 AR Path="/609FED99/60F1A12F" Ref="TP?"  Part="1"
@@
 AR Path="/60F197D4/60F1A12F" Ref="TP22"  Part="1"
 AR Path="/60F1A0E6/60F1A12F" Ref="TP?"  Part="1"
-F 0 "TP22" H 5558 4618 50  0000 L CNN
-F 1 "TestPoint" H 5558 4527 50  0001 L CNN
-F 2 "" H 5700 4500 50  0001 C CNN
-F 3 "~" H 5700 4500 50  0001 C CNN
-	1    5500 4500
-	1    0    0    -1
-$EndComp
-Text HLabel 4000 3500 0    50   Input ~ 0
-+3V3
-Text HLabel 4000 5000 0    50   Input ~ 0
+F 0 "TP22" H 6058 4618 50  0000 L CNN
+F 1 "TestPoint" H 6058 4527 50  0001 L CNN
+F 2 "rata:TP" H 6200 4500 50  0001 C CNN
+F 3 "~" H 6200 4500 50  0001 C CNN
+	1    6000 4500
+	1    0    0    -1
+$EndComp
+Text HLabel 3500 5000 0    50   Input ~ 0
 GND
 Text Notes 6900 2250 2    197  ~ 0
 Light level sensor
-Text HLabel 7500 4500 2    50   Output ~ 0
+Text HLabel 8000 4500 2    50   Output ~ 0
 VOLT
 $Comp
 L rata-rescue:SFH300-Sensor_Optical Q3
 U 1 1 60F482D9
-P 4900 4200
-F 0 "Q3" H 5090 4246 50  0000 L CNN
-F 1 "SFH3310" H 5090 4155 50  0000 L CNN
-F 2 "LED_THT:LED_D5.0mm_Clear" H 5380 4060 50  0001 C CNN
-F 3 "http://www.osram-os.com/Graphics/XPic2/00101785_0.pdf" H 4900 4200 50  0001 C CNN
-	1    4900 4200
+P 5400 4200
+F 0 "Q3" H 5590 4246 50  0000 L CNN
+F 1 "SFH3310" H 5590 4155 50  0000 L CNN
+F 2 "LED_THT:LED_D3.0mm_Horizontal_O1.27mm_Z2.0mm_Clear" H 5880 4060 50  0001 C CNN
+F 3 "http://www.osram-os.com/Graphics/XPic2/00101785_0.pdf" H 5400 4200 50  0001 C CNN
+	1    5400 4200
 	1    0    0    -1
 $EndComp
@@
 L rata-rescue:R-Device R?
 U 1 1 6100D3B1
-P 5000 4750
+P 5500 4750
 AR Path="/6100D3B1" Ref="R?"  Part="1"
 AR Path="/60B39FE1/6100D3B1" Ref="R?"  Part="1"
 AR Path="/60DF1160/60F2690B/6100D3B1" Ref="R?"  Part="1"
 AR Path="/60DF1160/6100D3B1" Ref="R?"  Part="1"
-AR Path="/60F197D4/6100D3B1" Ref="R48"  Part="1"
-F 0 "R48" H 5070 4796 50  0000 L CNN
-F 1 "1k" H 5070 4705 50  0000 L CNN
-F 2 "Resistor_SMD:R_0603_1608Metric_Pad0.98x0.95mm_HandSolder" V 4930 4750 50  0001 C CNN
-F 3 "~" H 5000 4750 50  0001 C CNN
-	1    5000 4750
+AR Path="/60F197D4/6100D3B1" Ref="R49"  Part="1"
+F 0 "R49" H 5570 4796 50  0000 L CNN
+F 1 "1k" H 5570 4705 50  0000 L CNN
+F 2 "Resistor_SMD:R_0603_1608Metric_Pad0.98x0.95mm_HandSolder" V 5430 4750 50  0001 C CNN
+F 3 "~" H 5500 4750 50  0001 C CNN
+	1    5500 4750
 	1    0    0    -1
 $EndComp
@@
 L rata-rescue:R-Device R?
 U 1 1 6100EF4A
-P 6250 4500
+P 6750 4500
 AR Path="/6100EF4A" Ref="R?"  Part="1"
 AR Path="/60B39FE1/6100EF4A" Ref="R?"  Part="1"
 AR Path="/60DF1160/60F2690B/6100EF4A" Ref="R?"  Part="1"
 AR Path="/60DF1160/6100EF4A" Ref="R?"  Part="1"
-AR Path="/60F197D4/6100EF4A" Ref="R49"  Part="1"
-F 0 "R49" V 6350 4450 50  0000 L CNN
-F 1 "4.7k" V 6150 4400 50  0000 L CNN
-F 2 "Resistor_SMD:R_0603_1608Metric_Pad0.98x0.95mm_HandSolder" V 6180 4500 50  0001 C CNN
-F 3 "~" H 6250 4500 50  0001 C CNN
-	1    6250 4500
+AR Path="/60F197D4/6100EF4A" Ref="R50"  Part="1"
+F 0 "R50" V 6850 4450 50  0000 L CNN
+F 1 "4.7k" V 6650 4400 50  0000 L CNN
+F 2 "Resistor_SMD:R_0603_1608Metric_Pad0.98x0.95mm_HandSolder" V 6680 4500 50  0001 C CNN
+F 3 "~" H 6750 4500 50  0001 C CNN
+	1    6750 4500
 	0    -1   -1   0
 $EndComp
@@
 L rata-rescue:TestPoint-Connector TP?
 U 1 1 61013214
-P 7000 4500
+P 7500 4500
 AR Path="/61013214" Ref="TP?"  Part="1"
 AR Path="/609FED99/61013214" Ref="TP?"  Part="1"
@@
 AR Path="/60F197D4/61013214" Ref="TP23"  Part="1"
 AR Path="/60F1A0E6/61013214" Ref="TP?"  Part="1"
-F 0 "TP23" H 7058 4618 50  0000 L CNN
-F 1 "TestPoint" H 7058 4527 50  0001 L CNN
-F 2 "" H 7200 4500 50  0001 C CNN
-F 3 "~" H 7200 4500 50  0001 C CNN
-	1    7000 4500
-	1    0    0    -1
-$EndComp
-Wire Wire Line
-	4000 3500 5000 3500
-Wire Wire Line
-	5000 3500 5000 4000
-Wire Wire Line
-	4000 5000 5000 5000
-Wire Wire Line
-	6500 5000 6500 4900
-Wire Wire Line
-	5000 4900 5000 5000
-Connection ~ 5000 5000
-Wire Wire Line
-	5000 5000 6500 5000
-Wire Wire Line
-	5000 4400 5000 4500
-Wire Wire Line
-	5000 4500 5500 4500
-Connection ~ 5000 4500
-Wire Wire Line
-	5000 4500 5000 4600
+F 0 "TP23" H 7558 4618 50  0000 L CNN
+F 1 "TestPoint" H 7558 4527 50  0001 L CNN
+F 2 "rata:TP" H 7700 4500 50  0001 C CNN
+F 3 "~" H 7700 4500 50  0001 C CNN
+	1    7500 4500
+	1    0    0    -1
+$EndComp
+Wire Wire Line
+	5500 3500 5500 4000
+Wire Wire Line
+	3500 5000 4500 5000
+Wire Wire Line
+	7000 5000 7000 4900
+Wire Wire Line
+	5500 4900 5500 5000
+Connection ~ 5500 5000
+Wire Wire Line
+	5500 5000 7000 5000
+Wire Wire Line
+	5500 4400 5500 4500
+Wire Wire Line
+	5500 4500 6000 4500
 Connection ~ 5500 4500
 Wire Wire Line
-	5500 4500 6100 4500
-Wire Wire Line
-	6400 4500 6500 4500
+	5500 4500 5500 4600
+Connection ~ 6000 4500
+Wire Wire Line
+	6000 4500 6600 4500
+Wire Wire Line
+	6900 4500 7000 4500
+Connection ~ 7500 4500
+Wire Wire Line
+	7500 4500 8000 4500
+Wire Wire Line
+	7000 4600 7000 4500
 Connection ~ 7000 4500
 Wire Wire Line
 	7000 4500 7500 4500
-Wire Wire Line
-	6500 4600 6500 4500
-Connection ~ 6500 4500
-Wire Wire Line
-	6500 4500 7000 4500
+$Comp
+L rata-rescue:C-Device C?
+U 1 1 61C54722
+P 4500 3850
+AR Path="/61C54722" Ref="C?"  Part="1"
+AR Path="/609CA6A8/609D24C0/61C54722" Ref="C?"  Part="1"
+AR Path="/609CA6A8/60A08E0B/61C54722" Ref="C?"  Part="1"
+AR Path="/609CA6A8/60A0A46E/61C54722" Ref="C?"  Part="1"
+AR Path="/609CA6A8/60A0A500/61C54722" Ref="C?"  Part="1"
+AR Path="/609CA6A8/60A0A922/61C54722" Ref="C?"  Part="1"
+AR Path="/609CA6A8/61C54722" Ref="C?"  Part="1"
+AR Path="/609CA6A8/60AE5653/61C54722" Ref="C?"  Part="1"
+AR Path="/609FED99/61C54722" Ref="C?"  Part="1"
+AR Path="/60DF07DE/61C54722" Ref="C?"  Part="1"
+AR Path="/60DF0860/61C54722" Ref="C?"  Part="1"
+AR Path="/60DF1072/61C54722" Ref="C?"  Part="1"
+AR Path="/60DF1160/61C54722" Ref="C?"  Part="1"
+AR Path="/60DF196E/61C54722" Ref="C?"  Part="1"
+AR Path="/60DF212D/61C54722" Ref="C?"  Part="1"
+AR Path="/60F197D4/61C54722" Ref="C54"  Part="1"
+AR Path="/60F1A0E6/61C54722" Ref="C?"  Part="1"
+F 0 "C54" H 4615 3896 50  0000 L CNN
+F 1 "0.1u" H 4615 3805 50  0000 L CNN
+F 2 "Capacitor_SMD:C_0603_1608Metric_Pad1.08x0.95mm_HandSolder" H 4538 3700 50  0001 C CNN
+F 3 "~" H 4500 3850 50  0001 C CNN
+	1    4500 3850
+	1    0    0    -1
+$EndComp
+Text HLabel 3500 3500 0    50   Input ~ 0
++3V3
+Wire Wire Line
+	3500 3500 4500 3500
+Wire Wire Line
+	4500 3700 4500 3500
+Connection ~ 4500 3500
+Wire Wire Line
+	4500 3500 5500 3500
+Wire Wire Line
+	4500 4000 4500 5000
+Connection ~ 4500 5000
+Wire Wire Line
+	4500 5000 5500 5000
 $EndSCHEMATC
