File: MCU.sch (KiCad schematic (older format))
At the start: 22 parts

Commit message: Add files via upload
Parts:
- removed C?: 0,01, Capacitor_SMD:C_0603_1608Metric_Pad1.08x0.95mm_HandSolder, symbol Device:C
- removed J?: PLS-6, symbol Connector:Conn_01x06_Male
- removed Q?: BC847, Package_TO_SOT_SMD:SOT-23, symbol Transistor_BJT:BC847
- removed R? (x2): 3,3k, Resistor_SMD:R_0603_1608Metric_Pad0.98x0.95mm_HandSolder, symbol Device:R
- removed R?: 150, Resistor_SMD:R_0603_1608Metric_Pad0.98x0.95mm_HandSolder, symbol Device:R
- removed R?: 56k, Resistor_SMD:R_0603_1608Metric_Pad0.98x0.95mm_HandSolder, symbol Device:R
- removed R?: 1k, Resistor_SMD:R_0603_1608Metric_Pad0.98x0.95mm_HandSolder, symbol Device:R
- added J?: PLS-5, symbol Connector:Conn_01x05_Male
Connections:
- net labels added: +3V3A, ALARM, AMP_EN, BRG0N, BRG0P, BRG1N, BRG1P, COL0, COL1, COL2, DAC_I2C_SCK, DAC_I2C_SDA, I2C2_SCK, I2C2_SDA, I2C_SCK, I2C_SDA, LIGHT, ROW0, ROW1, ROW2, SPI1_MOSI, T1C1, T1C1N, T1C2, T1C2N, UART2_RX, UART2_TX, USBDM, USBDP, USB_ON, ~SPI1_CS
- net labels removed: CHARGE_PUMP_CLK, DPY_I2C_SCK, DPY_I2C_SDA, DPY_PWR_EN, EXT_UART_RX, HEATER_CTRL, KYBD, KYBD0, KYBD1, KYBD2, KYBD3, KYBD4, KYBD5, KYBD6, KYBD7, KYBD8, KYBD9, SPI2_MISO, SPI2_MOSI, SPI2_SCK, SWO, TEMP_SPI_MISO, TEMP_SPI_SCK, UART1_RX, UART1_TX, ~DPY_RST, ~SPI2__CS, ~TEMP_CS0, ~TEMP_CS1, ~TEMP_CS2, ~TEMP_CS3, ~TEMP_CS4, ~TEMP_SPI_CS
- wire segments 101 -> 123
- no-connect marks 0 -> 6
Other:
- note added: "Matrix keyboard"
- note removed: "5V to 3V level converter"
- moved on the sheet: C?, J?, R?, Y?

Commit message: Add files via upload
Parts:
- gave numbers to parts that had none: 15
Connections:
- net ROW0: now also U2.25 (PB12); no longer U2.18 (PB0)
- net HEATER_PWR_EN: now reaches U2.2 (PC13)
- new net HEATER_VOLT: U2.18 (PB0)
- no-connect marks 6 -> 4
Other:
- moved on the sheet: C1, C4, R1, Y1

Commit message: Add files via upload
Parts:
- C1, C2, C3, C4, C5, C6, C7, C8, C9: symbol Device:C -> rata-rescue:C-Device
- J3: symbol Connector:Conn_01x05_Male -> rata-rescue:Conn_01x05_Male-Connector
- J4: symbol Connector:Conn_01x03_Male -> rata-rescue:Conn_01x03_Male-Connector
- R1, R2: symbol Device:R -> rata-rescue:R-Device
- U2: symbol MCU_ST_STM32F1:STM32F103C6Tx -> rata-rescue:STM32F103C6Tx-MCU_ST_STM32F1
- Y1: symbol Device:Crystal -> rata-rescue:Crystal-Device
Changed lines of the file:
@@
 	5300 4400 5400 4400
 $Comp
-L Connector:Conn_01x05_Male J3
+L rata-rescue:Conn_01x05_Male-Connector J3
 U 1 1 6101E732
 P 2500 2900
@@
 	5000 2800 5000 2850
 $Comp
-L Device:C C?
+L rata-rescue:C-Device C?
 U 1 1 60A7599F
 P 5000 3050
@@
 $EndComp
 $Comp
-L Device:R R?
+L rata-rescue:R-Device R?
 U 1 1 60A5E844
 P 4250 3700
@@
 	4100 3700 3950 3700
 $Comp
-L Device:C C?
+L rata-rescue:C-Device C?
 U 1 1 60A56506
 P 3950 3850
@@
 $EndComp
 $Comp
-L Device:C C?
+L rata-rescue:C-Device C?
 U 1 1 60A55C72
 P 3200 3850
@@
 $EndComp
 $Comp
-L Device:Crystal Y1
+L rata-rescue:Crystal-Device Y1
 U 1 1 60A53D72
 P 3650 3700
@@
 $EndComp
 $Comp
-L Device:C C?
+L rata-rescue:C-Device C?
 U 1 1 60A4D379
 P 5600 2150
@@
 $EndComp
 $Comp
-L Device:C C?
+L rata-rescue:C-Device C?
 U 1 1 60A4D2CE
 P 6000 2150
@@
 $EndComp
 $Comp
-L Device:C C?
+L rata-rescue:C-Device C?
 U 1 1 60A4D090
 P 4700 2150
@@
 $EndComp
 $Comp
-L Device:C C?
+L rata-rescue:C-Device C?
 U 1 1 60A4CF16
 P 4300 2150
@@
 $EndComp
 $Comp
-L Device:C C?
+L rata-rescue:C-Device C?
 U 1 1 60B4CB8E
 P 3900 2150
@@
 $EndComp
 $Comp
-L Device:R R?
+L rata-rescue:R-Device R?
 U 1 1 60B4CB82
 P 5000 2650
@@
 $EndComp
 $Comp
-L Connector:Conn_01x03_Male J4
+L rata-rescue:Conn_01x03_Male-Connector J4
 U 1 1 60B5D67E
 P 8200 4500
@@
 $EndComp
 $Comp
-L MCU_ST_STM32F1:STM32F103C6Tx U?
+L rata-rescue:STM32F103C6Tx-MCU_ST_STM32F1 U?
 U 1 1 609CC27B
 P 6100 4400
@@
 $EndComp
 $Comp
-L Device:C C?
+L rata-rescue:C-Device C?
 U 1 1 60B4F8D6
 P 3500 2150

Commit message: Add files via upload
Parts:
- J3: footprint (none) -> Connector_PinHeader_2.54mm:PinHeader_1x05_P2.54mm_Vertical
- J4: footprint (none) -> Connector_PinHeader_2.54mm:PinHeader_1x03_P2.54mm_Vertical
- Y1: footprint (none) -> Crystal:Crystal_SMD_HC49-SD
Connections:
- net LIGHT is gone; now on net AMP_EN: U2.11 (PA1)
- net ALARM: now also U2.43 (PB7); no longer U2.45 (PB8)
- net AMP_EN: no longer U2.46 (PB9)
- net BZ_EN: now also U2.2 (PC13); no longer U2.10 (PA0)
- net COL0: now also U2.15 (PA5); no longer U2.39 (PB3)
- net COL1: now also U2.16 (PA6); no longer U2.40 (PB4)
- net COL2: now also U2.17 (PA7); no longer U2.41 (PB5)
- net DAC_I2C_SCK: now also U2.21 (PB10); no longer U2.42 (PB6)
- net DAC_I2C_SDA: now also U2.22 (PB11); no longer U2.43 (PB7)
- net HEATER_PWR_EN: now also U2.28 (PB15); no longer U2.2 (PC13)
- net HEATER_VOLT: now also U2.19 (PB1); no longer U2.18 (PB0)
- net I2C_SCK: now also U2.45 (PB8); no longer U2.21 (PB10)
- net I2C_SDA: now also U2.46 (PB9); no longer U2.22 (PB11)
- net ROW1: now also U2.20 (PB2); no longer U2.19 (PB1)
- net ROW2: now also U2.18 (PB0); no longer U2.20 (PB2)
- net SD_SPI_MISO: now also U2.40 (PB4); no longer U2.16 (PA6)
- net SD_SPI_MOSI: now also U2.41 (PB5); no longer U2.17 (PA7)
- net SD_SPI_SCK: now also U2.39 (PB3); no longer U2.15 (PA5)
- net ~SD_SPI_CS: now also U2.38 (PA15); no longer U2.14 (PA4)
- new net LIGHT_VOLT: U2.10 (PA0)
- new net SD_CARD_DET: U2.42 (PB6)
- no-connect marks 4 -> 3
Other:
- moved on the sheet: C1, C2, C3, C4, C5, C6, C7, C8, C9, J3, J4, R1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
