File: Micro_SD_card.sch (KiCad schematic (older format))
At the start: 7 parts

Commit message: Add files via upload
Changed lines of the file:
@@
 $Descr A4 11693 8268
 encoding utf-8
-Sheet 3 11
+Sheet 3 15
 Title ""
 Date ""
@@
 $EndComp
 $Comp
-L power:GND #PWR?
-U 1 1 60B1D1D7
-P 8000 5300
-AR Path="/60B1D1D7" Ref="#PWR?"  Part="1"
-AR Path="/609C9D41/60B1D1D7" Ref="#PWR?"  Part="1"
-AR Path="/60B1951B/60B1D1D7" Ref="#PWR?"  Part="1"
-F 0 "#PWR?" H 8000 5050 50  0001 C CNN
-F 1 "GND" H 8005 5127 50  0000 C CNN
-F 2 "" H 8000 5300 50  0001 C CNN
-F 3 "" H 8000 5300 50  0001 C CNN
-	1    8000 5300
-	1    0    0    -1
-$EndComp
-$Comp
 L Device:C C?
 U 1 1 60B1D1DD
@@
 	1    0    0    -1
 $EndComp
-$Comp
-L power:GND #PWR?
-U 1 1 60B1D1E3
-P 5500 5250
-AR Path="/60B1D1E3" Ref="#PWR?"  Part="1"
-AR Path="/609C9D41/60B1D1E3" Ref="#PWR?"  Part="1"
-AR Path="/60B1951B/60B1D1E3" Ref="#PWR?"  Part="1"
-F 0 "#PWR?" H 5500 5000 50  0001 C CNN
-F 1 "GND" H 5505 5077 50  0000 C CNN
-F 2 "" H 5500 5250 50  0001 C CNN
-F 3 "" H 5500 5250 50  0001 C CNN
-	1    5500 5250
-	1    0    0    -1
-$EndComp
-$Comp
-L power:+3V3 #PWR?
-U 1 1 60B1D1E9
-P 5500 3250
-AR Path="/609FED99/60B1D1E9" Ref="#PWR?"  Part="1"
-AR Path="/609C9D41/60B1D1E9" Ref="#PWR?"  Part="1"
-AR Path="/60B1951B/60B1D1E9" Ref="#PWR?"  Part="1"
-F 0 "#PWR?" H 5500 3100 50  0001 C CNN
-F 1 "+3V3" H 5515 3423 50  0000 C CNN
-F 2 "" H 5500 3250 50  0001 C CNN
-F 3 "" H 5500 3250 50  0001 C CNN
-	1    5500 3250
-	1    0    0    -1
-$EndComp
-$Comp
-L power:GND #PWR?
-U 1 1 60B1D1EF
-P 5800 3950
-AR Path="/60B1D1EF" Ref="#PWR?"  Part="1"
-AR Path="/609C9D41/60B1D1EF" Ref="#PWR?"  Part="1"
-AR Path="/60B1951B/60B1D1EF" Ref="#PWR?"  Part="1"
-F 0 "#PWR?" H 5800 3700 50  0001 C CNN
-F 1 "GND" H 5805 3777 50  0000 C CNN
-F 2 "" H 5800 3950 50  0001 C CNN
-F 3 "" H 5800 3950 50  0001 C CNN
-	1    5800 3950
-	1    0    0    -1
-$EndComp
-Wire Wire Line
-	8000 5200 8000 5300
-Wire Wire Line
-	5500 4800 5500 5250
 Wire Wire Line
 	5500 4600 5500 3500
@@
 Wire Wire Line
 	5800 3800 5800 3950
-Connection ~ 5500 3400
-Wire Wire Line
-	5500 3400 5500 3250
 Wire Wire Line
 	5000 3750 5000 3400
@@
 Wire Wire Line
 	6200 3950 5800 3950
-Connection ~ 5800 3950
 Wire Wire Line
 	4100 4400 4900 4400
@@
 Wire Wire Line
 	4600 4900 5000 4900
+Text HLabel 4100 3400 0    50   Input ~ 0
++3V3
+Text HLabel 4100 6000 0    50   Input ~ 0
+GND
+Wire Wire Line
+	8000 5200 8000 6000
+Wire Wire Line
+	5500 4800 5500 6000
+Connection ~ 5500 6000
+Wire Wire Line
+	5500 6000 5800 6000
 Wire Wire Line
 	5000 5900 4900 5900
-$Comp
-L power:GND #PWR?
-U 1 1 60B38C7E
-P 4900 5900
-AR Path="/60B38C7E" Ref="#PWR?"  Part="1"
-AR Path="/609C9D41/60B38C7E" Ref="#PWR?"  Part="1"
-AR Path="/60B1951B/60B38C7E" Ref="#PWR?"  Part="1"
-F 0 "#PWR?" H 4900 5650 50  0001 C CNN
-F 1 "GND" H 4905 5727 50  0000 C CNN
-F 2 "" H 4900 5900 50  0001 C CNN
-F 3 "" H 4900 5900 50  0001 C CNN
-	1    4900 5900
-	1    0    0    -1
-$EndComp
+Wire Wire Line
+	4900 5900 4900 6000
+Wire Wire Line
+	4900 6000 5500 6000
+Wire Wire Line
+	5800 3950 5800 6000
+Connection ~ 5800 3950
+Connection ~ 5800 6000
+Wire Wire Line
+	5800 6000 8000 6000
+Wire Wire Line
+	4100 3400 4400 3400
+Connection ~ 4400 3400
+Wire Wire Line
+	4100 6000 4900 6000
+Connection ~ 4900 6000
 $EndSCHEMATC

Commit message: Add files via upload
Parts:
- gave numbers to parts that had none: 7
Changed lines of the file:
@@
 AR Path="/60B1D1CB" Ref="J?"  Part="1"
 AR Path="/609C9D41/60B1D1CB" Ref="J?"  Part="1"
-AR Path="/60B1951B/60B1D1CB" Ref="J?"  Part="1"
-F 0 "J?" H 7150 5317 50  0000 C CNN
+AR Path="/60B1951B/60B1D1CB" Ref="J6"  Part="1"
+F 0 "J6" H 7150 5317 50  0000 C CNN
 F 1 "Micro_SD_Card" H 7150 5226 50  0000 C CNN
 F 2 "" H 8350 4900 50  0001 C CNN
@@
 AR Path="/60B1D1D1" Ref="R?"  Part="1"
 AR Path="/609C9D41/60B1D1D1" Ref="R?"  Part="1"
-AR Path="/60B1951B/60B1D1D1" Ref="R?"  Part="1"
-F 0 "R?" H 5070 3946 50  0000 L CNN
+AR Path="/60B1951B/60B1D1D1" Ref="R5"  Part="1"
+F 0 "R5" H 5070 3946 50  0000 L CNN
 F 1 "10k" H 5070 3855 50  0000 L CNN
 F 2 "Resistor_SMD:R_0603_1608Metric_Pad0.98x0.95mm_HandSolder" V 4930 3900 50  0001 C CNN
@@
 AR Path="/60B1D1DD" Ref="C?"  Part="1"
 AR Path="/609C9D41/60B1D1DD" Ref="C?"  Part="1"
-AR Path="/60B1951B/60B1D1DD" Ref="C?"  Part="1"
-F 0 "C?" H 5915 3696 50  0000 L CNN
+AR Path="/60B1951B/60B1D1DD" Ref="C10"  Part="1"
+F 0 "C10" H 5915 3696 50  0000 L CNN
 F 1 "0,1" H 5915 3605 50  0000 L CNN
 F 2 "Capacitor_SMD:C_0603_1608Metric_Pad1.08x0.95mm_HandSolder" H 5838 3500 50  0001 C CNN
@@
 AR Path="/60B1D208" Ref="R?"  Part="1"
 AR Path="/609C9D41/60B1D208" Ref="R?"  Part="1"
-AR Path="/60B1951B/60B1D208" Ref="R?"  Part="1"
-F 0 "R?" H 4770 3946 50  0000 L CNN
+AR Path="/60B1951B/60B1D208" Ref="R4"  Part="1"
+F 0 "R4" H 4770 3946 50  0000 L CNN
 F 1 "10k" H 4770 3855 50  0000 L CNN
 F 2 "Resistor_SMD:R_0603_1608Metric_Pad0.98x0.95mm_HandSolder" V 4630 3900 50  0001 C CNN
@@
 AR Path="/60B1D20E" Ref="R?"  Part="1"
 AR Path="/609C9D41/60B1D20E" Ref="R?"  Part="1"
-AR Path="/60B1951B/60B1D20E" Ref="R?"  Part="1"
-F 0 "R?" H 4470 3946 50  0000 L CNN
+AR Path="/60B1951B/60B1D20E" Ref="R3"  Part="1"
+F 0 "R3" H 4470 3946 50  0000 L CNN
 F 1 "10k" H 4470 3855 50  0000 L CNN
 F 2 "Resistor_SMD:R_0603_1608Metric_Pad0.98x0.95mm_HandSolder" V 4330 3900 50  0001 C CNN
@@
 AR Path="/609FED99/60B1D21E" Ref="C?"  Part="1"
 AR Path="/609C9D41/60B1D21E" Ref="C?"  Part="1"
-AR Path="/60B1951B/60B1D21E" Ref="C?"  Part="1"
-F 0 "C?" H 6315 3696 50  0000 L CNN
+AR Path="/60B1951B/60B1D21E" Ref="C11"  Part="1"
+F 0 "C11" H 6315 3696 50  0000 L CNN
 F 1 "10u" H 6315 3605 50  0000 L CNN
 F 2 "Capacitor_SMD:C_1206_3216Metric_Pad1.33x1.80mm_HandSolder" H 6238 3500 50  0001 C CNN
@@
 MISO
 $Comp
-L Connector:Conn_01x05_Male J?
+L Connector:Conn_01x05_Male J5
 U 1 1 60B35003
 P 5200 5700
-F 0 "J?" H 5172 5724 50  0000 R CNN
+F 0 "J5" H 5172 5724 50  0000 R CNN
 F 1 "Conn_01x05_Male" H 5172 5633 50  0000 R CNN
 F 2 "" H 5200 5700 50  0001 C CNN

Commit message: Add files via upload
Parts:
- C10, C11: symbol Device:C -> rata-rescue:C-Device
- J5: symbol Connector:Conn_01x05_Male -> rata-rescue:Conn_01x05_Male-Connector
- J6: symbol Connector:Micro_SD_Card -> rata-rescue:Micro_SD_Card-Connector
- R3, R4, R5: symbol Device:R -> rata-rescue:R-Device
Changed lines of the file:
@@
 $EndDescr
 $Comp
-L Connector:Micro_SD_Card J?
+L rata-rescue:Micro_SD_Card-Connector J?
 U 1 1 60B1D1CB
 P 7200 4600
@@
 $EndComp
 $Comp
-L Device:R R?
+L rata-rescue:R-Device R?
 U 1 1 60B1D1D1
 P 5000 3900
@@
 $EndComp
 $Comp
-L Device:C C?
+L rata-rescue:C-Device C?
 U 1 1 60B1D1DD
 P 5800 3650
@@
 	5000 4050 5000 4900
 $Comp
-L Device:R R?
+L rata-rescue:R-Device R?
 U 1 1 60B1D208
 P 4700 3900
@@
 $EndComp
 $Comp
-L Device:R R?
+L rata-rescue:R-Device R?
 U 1 1 60B1D20E
 P 4400 3900
@@
 	4700 3400 5000 3400
 $Comp
-L Device:C C?
+L rata-rescue:C-Device C?
 U 1 1 60B1D21E
 P 6200 3650
@@
 MISO
 $Comp
-L Connector:Conn_01x05_Male J5
+L rata-rescue:Conn_01x05_Male-Connector J5
 U 1 1 60B35003
 P 5200 5700

Commit message: Add files via upload
Parts:
- removed J6: Micro_SD_Card, symbol rata-rescue:Micro_SD_Card-Connector
- added J6: CTF-11081-P, rata:CTF-11081-P, symbol rata:CTF-11081-P
- added R3: 10k, Resistor_SMD:R_0603_1608Metric_Pad0.98x0.95mm_HandSolder, symbol rata-rescue:R-Device
- J5: value Conn_01x05_Male -> PLS-5; footprint (none) -> Connector_PinHeader_2.54mm:PinHeader_1x05_P2.54mm_Vertical
- renumbered R3 to R4, R4 to R5, R5 to R6
Connections:
- net +3V3: now also J6.4 (VDD), R3.1
- net GND: now also J6.6 (VSS), J6.G (GROUND)
- net MISO: now also J6.7 (DAT0)
- net MOSI: now also J6.3 (CMD)
- net SCK: now also J6.5 (CLK)
- net ~CS~: now also J6.2 (DAT3/CD)
- net at R5.2: now also J6.1 (DAT2)
- net at R4.2: now also J6.8 (DAT1)
- new net CARD_DET: J6.Cd (CARD_DETECTION), R3.2
Changed lines of the file:
@@
 encoding utf-8
 Sheet 3 23
-Title ""
-Date ""
-Rev ""
-Comp ""
+Title "rata"
+Date "2021-09-25"
+Rev "1.0"
+Comp "Yuriy Volkov"
 Comment1 ""
 Comment2 ""
@@
 $EndDescr
 $Comp
-L rata-rescue:Micro_SD_Card-Connector J?
-U 1 1 60B1D1CB
-P 7200 4600
-AR Path="/60B1D1CB" Ref="J?"  Part="1"
-AR Path="/609C9D41/60B1D1CB" Ref="J?"  Part="1"
-AR Path="/60B1951B/60B1D1CB" Ref="J6"  Part="1"
-F 0 "J6" H 7150 5317 50  0000 C CNN
-F 1 "Micro_SD_Card" H 7150 5226 50  0000 C CNN
-F 2 "" H 8350 4900 50  0001 C CNN
-F 3 "http://katalog.we-online.de/em/datasheet/693072010801.pdf" H 7200 4600 50  0001 C CNN
-	1    7200 4600
-	1    0    0    -1
-$EndComp
-$Comp
 L rata-rescue:R-Device R?
 U 1 1 60B1D1D1
@@
 AR Path="/60B1D1D1" Ref="R?"  Part="1"
 AR Path="/609C9D41/60B1D1D1" Ref="R?"  Part="1"
-AR Path="/60B1951B/60B1D1D1" Ref="R5"  Part="1"
-F 0 "R5" H 5070 3946 50  0000 L CNN
+AR Path="/60B1951B/60B1D1D1" Ref="R6"  Part="1"
+F 0 "R6" H 5070 3946 50  0000 L CNN
 F 1 "10k" H 5070 3855 50  0000 L CNN
 F 2 "Resistor_SMD:R_0603_1608Metric_Pad0.98x0.95mm_HandSolder" V 4930 3900 50  0001 C CNN
@@
 AR Path="/60B1D208" Ref="R?"  Part="1"
 AR Path="/609C9D41/60B1D208" Ref="R?"  Part="1"
-AR Path="/60B1951B/60B1D208" Ref="R4"  Part="1"
-F 0 "R4" H 4770 3946 50  0000 L CNN
+AR Path="/60B1951B/60B1D208" Ref="R5"  Part="1"
+F 0 "R5" H 4770 3946 50  0000 L CNN
 F 1 "10k" H 4770 3855 50  0000 L CNN
 F 2 "Resistor_SMD:R_0603_1608Metric_Pad0.98x0.95mm_HandSolder" V 4630 3900 50  0001 C CNN
@@
 AR Path="/60B1D20E" Ref="R?"  Part="1"
 AR Path="/609C9D41/60B1D20E" Ref="R?"  Part="1"
-AR Path="/60B1951B/60B1D20E" Ref="R3"  Part="1"
-F 0 "R3" H 4470 3946 50  0000 L CNN
+AR Path="/60B1951B/60B1D20E" Ref="R4"  Part="1"
+F 0 "R4" H 4470 3946 50  0000 L CNN
 F 1 "10k" H 4470 3855 50  0000 L CNN
 F 2 "Resistor_SMD:R_0603_1608Metric_Pad0.98x0.95mm_HandSolder" V 4330 3900 50  0001 C CNN
@@
 	6200 3950 5800 3950
 Wire Wire Line
-	4100 4400 4900 4400
-Wire Wire Line
-	4100 4500 4700 4500
-Wire Wire Line
-	4100 4700 4800 4700
-Wire Wire Line
-	4100 4900 4600 4900
+	3500 4400 4900 4400
+Wire Wire Line
+	3500 4500 4700 4500
+Wire Wire Line
+	3500 4700 4800 4700
+Wire Wire Line
+	3500 4900 4600 4900
 Connection ~ 5000 4900
 Text Notes 7600 2450 2    197  ~ 0
 Micro-SD card connector
-Text HLabel 4100 4400 0    50   Input ~ 0
+Text HLabel 3500 4400 0    50   Input ~ 0
 ~CS~
-Text HLabel 4100 4500 0    50   Input ~ 0
+Text HLabel 3500 4500 0    50   Input ~ 0
 MOSI
-Text HLabel 4100 4700 0    50   Input ~ 0
+Text HLabel 3500 4700 0    50   Input ~ 0
 SCK
-Text HLabel 4100 4900 0    50   Output ~ 0
+Text HLabel 3500 4900 0    50   Output ~ 0
 MISO
 $Comp
@@
 P 5200 5700
 F 0 "J5" H 5172 5724 50  0000 R CNN
-F 1 "Conn_01x05_Male" H 5172 5633 50  0000 R CNN
-F 2 "" H 5200 5700 50  0001 C CNN
+F 1 "PLS-5" H 5172 5633 50  0000 R CNN
+F 2 "Connector_PinHeader_2.54mm:PinHeader_1x05_P2.54mm_Vertical" H 5200 5700 50  0001 C CNN
 F 3 "~" H 5200 5700 50  0001 C CNN
 	1    5200 5700
@@
 Wire Wire Line
 	4600 4900 5000 4900
-Text HLabel 4100 3400 0    50   Input ~ 0
+Text HLabel 3500 3400 0    50   Input ~ 0
 +3V3
-Text HLabel 4100 6000 0    50   Input ~ 0
+Text HLabel 3500 6000 0    50   Input ~ 0
 GND
 Wire Wire Line
@@
 	5800 6000 8000 6000
 Wire Wire Line
+	3500 3400 4100 3400
+Connection ~ 4400 3400
+Wire Wire Line
+	3500 6000 4900 6000
+Connection ~ 4900 6000
+$Comp
+L rata:CTF-11081-P J6
+U 1 1 6159A21C
+P 7200 4600
+F 0 "J6" H 7150 5317 50  0000 C CNN
+F 1 "CTF-11081-P" H 7150 5226 50  0000 C CNN
+F 2 "rata:CTF-11081-P" H 8350 4900 50  0001 C CNN
+F 3 "" H 7200 4600 50  0001 C CNN
+	1    7200 4600
+	1    0    0    -1
+$EndComp
+$Comp
+L rata-rescue:R-Device R?
+U 1 1 615A4AAC
+P 4100 3900
+AR Path="/615A4AAC" Ref="R?"  Part="1"
+AR Path="/609C9D41/615A4AAC" Ref="R?"  Part="1"
+AR Path="/60B1951B/615A4AAC" Ref="R3"  Part="1"
+F 0 "R3" H 4170 3946 50  0000 L CNN
+F 1 "10k" H 4170 3855 50  0000 L CNN
+F 2 "Resistor_SMD:R_0603_1608Metric_Pad0.98x0.95mm_HandSolder" V 4030 3900 50  0001 C CNN
+F 3 "~" H 4100 3900 50  0001 C CNN
+	1    4100 3900
+	1    0    0    -1
+$EndComp
+Text HLabel 3500 5100 0    50   Output ~ 0
+CARD_DET
+Wire Wire Line
+	3500 5100 4100 5100
+Wire Wire Line
+	4100 4050 4100 5100
+Connection ~ 4100 5100
+Wire Wire Line
+	4100 5100 6300 5100
+Wire Wire Line
+	4100 3750 4100 3400
+Connection ~ 4100 3400
+Wire Wire Line
 	4100 3400 4400 3400
-Connection ~ 4400 3400
-Wire Wire Line
-	4100 6000 4900 6000
-Connection ~ 4900 6000
 $EndSCHEMATC
