File: Power_+25V.sch (KiCad schematic (older format))
At the start: 31 parts

Commit message: Add files via upload
Parts:
- removed C? (x6): 10u, Capacitor_SMD:C_1206_3216Metric_Pad1.33x1.80mm_HandSolder, symbol Device:C
- removed C?: 1u, Capacitor_SMD:C_0603_1608Metric_Pad1.08x0.95mm_HandSolder, symbol Device:C
- removed D? (x3): BAT54S, Package_TO_SOT_SMD:SOT-23, symbol Diode:BAT54S
- removed D?: SMAJ5.0CA, symbol Device:D_TVS
- removed Q?: IRLML6402, Package_TO_SOT_SMD:SOT-23, symbol Transistor_FET:IRLML6402
- removed Q?: IRLML2402, Package_TO_SOT_SMD:SOT-23, symbol Transistor_FET:IRLML2060
- removed Q?: BC847, Package_TO_SOT_SMD:SOT-23, symbol Transistor_BJT:BC847
- removed R?: 100, Resistor_SMD:R_0603_1608Metric_Pad0.98x0.95mm_HandSolder, symbol Device:R
- removed R? (x2): 1,2k, Resistor_SMD:R_0603_1608Metric_Pad0.98x0.95mm_HandSolder, symbol Device:R
- removed R? (x2): 56k, Resistor_SMD:R_0603_1608Metric_Pad0.98x0.95mm_HandSolder, symbol Device:R
- removed R?: 3,3k, Resistor_SMD:R_0603_1608Metric_Pad0.98x0.95mm_HandSolder, symbol Device:R
- removed TP?: TestPoint, symbol Connector:TestPoint
- removed U?: AMS1117-3.3, Package_TO_SOT_SMD:SOT-223-3_TabPin2, symbol Regulator_Linear:AMS1117-3.3
- added C?: 470u, symbol Device:CP
- added C?: 1000, Capacitor_SMD:C_0603_1608Metric_Pad1.08x0.95mm_HandSolder, symbol Device:C
- added D?: MBR0540, symbol Device:D_Schottky
- added L?: 330u, symbol Device:L
- added R?: 47k 1%, Resistor_SMD:R_0603_1608Metric_Pad0.98x0.95mm_HandSolder, symbol Device:R
- R?: value 680 -> 0,47 2010; footprint Resistor_SMD:R_0603_1608Metric_Pad0.98x0.95mm_HandSolder -> (none)
- R?: value 330 -> 200
- R?: value 56k -> 2,4k 1%
Connections:
- net labels added: +25V_OUT
- net labels removed: +10V, +3V3, +5V, CHARGE_PUMP_CLK, GND_IN
- wire segments 77 -> 42
- no-connect marks 2 -> 0
Other:
- note added: "Power source +25V"
- note removed: "Power sources 3V3 and 10V"
- moved on the sheet: C?, R?, TP?, U?

Commit message: Add files via upload
Parts:
- C?: value 1000 -> 500
Changed lines of the file:
@@
 AR Path="/60DF0860/60E81588" Ref="C?"  Part="1"
 F 0 "C?" H 4615 4596 50  0000 L CNN
-F 1 "1000" H 4615 4505 50  0000 L CNN
+F 1 "500" H 4615 4505 50  0000 L CNN
 F 2 "Capacitor_SMD:C_0603_1608Metric_Pad1.08x0.95mm_HandSolder" H 4538 4400 50  0001 C CNN
 F 3 "~" H 4500 4550 50  0001 C CNN

Commit message: Add files via upload
Other:
- note added: "Boost converter +25V"
- note removed: "Power source +25V"
Changed lines of the file:
@@
 $Descr A4 11693 8268
 encoding utf-8
-Sheet 7 15
+Sheet 7 20
 Title ""
 Date ""
@@
 $EndDescr
 Text Notes 7000 2250 2    197  ~ 0
-Power source +25V
+Boost converter +25V
 $Comp
 L Device:C C?

Commit message: Add files via upload
Parts:
- removed C?: 100u, symbol Device:CP
- removed TP?: TestPoint, symbol Connector:TestPoint
- added C?: 100u, symbol Device:CP
- added TP?: TestPoint, symbol Connector:TestPoint
Connections:
- net +5V_IN: now also C?.1
- net GND: now also C?.2
- net at L?.1, R?.1, R?.1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: now also TP?.1
Changed lines of the file:
@@
 $Descr A4 11693 8268
 encoding utf-8
-Sheet 7 20
+Sheet 7 24
 Title ""
 Date ""
@@
 $Comp
 L Connector:TestPoint TP?
-U 1 1 60ACAEBE
+U 1 1 60F5917B
 P 5600 3500
-AR Path="/60ACAEBE" Ref="TP?"  Part="1"
-AR Path="/609FED99/60ACAEBE" Ref="TP?"  Part="1"
-AR Path="/60DF0860/60ACAEBE" Ref="TP?"  Part="1"
+AR Path="/60F5917B" Ref="TP?"  Part="1"
+AR Path="/609FED99/60F5917B" Ref="TP?"  Part="1"
+AR Path="/60DF0860/60F5917B" Ref="TP?"  Part="1"
 F 0 "TP?" H 5658 3618 50  0000 L CNN
 F 1 "TestPoint" H 5658 3527 50  0001 L CNN
@@
 $Comp
 L Device:CP C?
-U 1 1 60ADA476
+U 1 1 60F5917D
 P 3500 4150
 F 0 "C?" H 3618 4196 50  0000 L CNN

Commit message: Add files via upload
Parts:
- gave numbers to parts that had none: 14
Changed lines of the file:
@@
 AR Path="/609CA6A8/60AE5653/60A0DAB2" Ref="C?"  Part="1"
 AR Path="/609FED99/60A0DAB2" Ref="C?"  Part="1"
-AR Path="/60DF0860/60A0DAB2" Ref="C?"  Part="1"
-F 0 "C?" H 4115 4196 50  0000 L CNN
+AR Path="/60DF0860/60A0DAB2" Ref="C23"  Part="1"
+F 0 "C23" H 4115 4196 50  0000 L CNN
 F 1 "0,1" H 4115 4105 50  0000 L CNN
 F 2 "Capacitor_SMD:C_0603_1608Metric_Pad1.08x0.95mm_HandSolder" H 4038 4000 50  0001 C CNN
@@
 AR Path="/60A440E9" Ref="R?"  Part="1"
 AR Path="/609FED99/60A440E9" Ref="R?"  Part="1"
-AR Path="/60DF0860/60A440E9" Ref="R?"  Part="1"
-F 0 "R?" V 5200 3450 50  0000 L CNN
+AR Path="/60DF0860/60A440E9" Ref="R12"  Part="1"
+F 0 "R12" V 5200 3450 50  0000 L CNN
 F 1 "0,47 2010" V 5400 3300 50  0000 L CNN
 F 2 "" V 5230 3500 50  0001 C CNN
@@
 AR Path="/60DF11BE" Ref="R?"  Part="1"
 AR Path="/609FED99/60DF11BE" Ref="R?"  Part="1"
-AR Path="/60DF0860/60DF11BE" Ref="R?"  Part="1"
-F 0 "R?" H 6320 3696 50  0000 L CNN
+AR Path="/60DF0860/60DF11BE" Ref="R13"  Part="1"
+F 0 "R13" H 6320 3696 50  0000 L CNN
 F 1 "200" H 6320 3605 50  0000 L CNN
 F 2 "Resistor_SMD:R_0603_1608Metric_Pad0.98x0.95mm_HandSolder" V 6180 3650 50  0001 C CNN
@@
 AR Path="/60DF11BF" Ref="TP?"  Part="1"
 AR Path="/609FED99/60DF11BF" Ref="TP?"  Part="1"
-AR Path="/60DF0860/60DF11BF" Ref="TP?"  Part="1"
-F 0 "TP?" H 8308 4118 50  0000 L CNN
+AR Path="/60DF0860/60DF11BF" Ref="TP11"  Part="1"
+F 0 "TP11" H 8308 4118 50  0000 L CNN
 F 1 "TestPoint" H 8308 4027 50  0001 L CNN
 F 2 "" H 8450 4000 50  0001 C CNN
@@
 AR Path="/60F5917B" Ref="TP?"  Part="1"
 AR Path="/609FED99/60F5917B" Ref="TP?"  Part="1"
-AR Path="/60DF0860/60F5917B" Ref="TP?"  Part="1"
-F 0 "TP?" H 5658 3618 50  0000 L CNN
+AR Path="/60DF0860/60F5917B" Ref="TP10"  Part="1"
+F 0 "TP10" H 5658 3618 50  0000 L CNN
 F 1 "TestPoint" H 5658 3527 50  0001 L CNN
 F 2 "" H 5800 3500 50  0001 C CNN
@@
 $EndComp
 $Comp
-L Device:CP C?
+L Device:CP C22
 U 1 1 60F5917D
 P 3500 4150
-F 0 "C?" H 3618 4196 50  0000 L CNN
+F 0 "C22" H 3618 4196 50  0000 L CNN
 F 1 "100u" H 3618 4105 50  0000 L CNN
 F 2 "" H 3538 4000 50  0001 C CNN
@@
 AR Path="/60AFF250" Ref="TP?"  Part="1"
 AR Path="/609FED99/60AFF250" Ref="TP?"  Part="1"
-AR Path="/60DF0860/60AFF250" Ref="TP?"  Part="1"
-F 0 "TP?" H 5058 3618 50  0000 L CNN
+AR Path="/60DF0860/60AFF250" Ref="TP9"  Part="1"
+F 0 "TP9" H 5058 3618 50  0000 L CNN
 F 1 "TestPoint" H 5058 3527 50  0001 L CNN
 F 2 "" H 5200 3500 50  0001 C CNN
@@
 AR Path="/60B39FE1/60DF11CA" Ref="R?"  Part="1"
 AR Path="/609FED99/60DF11CA" Ref="R?"  Part="1"
-AR Path="/60DF0860/60DF11CA" Ref="R?"  Part="1"
-F 0 "R?" H 8070 4696 50  0000 L CNN
+AR Path="/60DF0860/60DF11CA" Ref="R15"  Part="1"
+F 0 "R15" H 8070 4696 50  0000 L CNN
 F 1 "2,4k 1%" H 8070 4605 50  0000 L CNN
 F 2 "Resistor_SMD:R_0603_1608Metric_Pad0.98x0.95mm_HandSolder" V 7930 4650 50  0001 C CNN
@@
 $EndComp
 $Comp
-L Regulator_Switching:MC34063AD U?
+L Regulator_Switching:MC34063AD U5
 U 1 1 60DF4135
 P 5300 4200
-F 0 "U?" H 5300 4667 50  0000 C CNN
+F 0 "U5" H 5300 4667 50  0000 C CNN
 F 1 "MC34063AD" H 5300 4576 50  0000 C CNN
 F 2 "Package_SO:SOIC-8_3.9x4.9mm_P1.27mm" H 5350 3750 50  0001 L CNN
@@
 $EndComp
 $Comp
-L Device:CP C?
+L Device:CP C25
 U 1 1 60E7FC90
 P 8500 4150
-F 0 "C?" H 8618 4196 50  0000 L CNN
+F 0 "C25" H 8618 4196 50  0000 L CNN
 F 1 "470u" H 8618 4105 50  0000 L CNN
 F 2 "" H 8538 4000 50  0001 C CNN
@@
 AR Path="/60B39FE1/60E80DA1" Ref="R?"  Part="1"
 AR Path="/609FED99/60E80DA1" Ref="R?"  Part="1"
-AR Path="/60DF0860/60E80DA1" Ref="R?"  Part="1"
-F 0 "R?" H 8070 4196 50  0000 L CNN
+AR Path="/60DF0860/60E80DA1" Ref="R14"  Part="1"
+F 0 "R14" H 8070 4196 50  0000 L CNN
 F 1 "47k 1%" H 8070 4105 50  0000 L CNN
 F 2 "Resistor_SMD:R_0603_1608Metric_Pad0.98x0.95mm_HandSolder" V 7930 4150 50  0001 C CNN
@@
 AR Path="/609CA6A8/60AE5653/60E81588" Ref="C?"  Part="1"
 AR Path="/609FED99/60E81588" Ref="C?"  Part="1"
-AR Path="/60DF0860/60E81588" Ref="C?"  Part="1"
-F 0 "C?" H 4615 4596 50  0000 L CNN
+AR Path="/60DF0860/60E81588" Ref="C24"  Part="1"
+F 0 "C24" H 4615 4596 50  0000 L CNN
 F 1 "500" H 4615 4505 50  0000 L CNN
 F 2 "Capacitor_SMD:C_0603_1608Metric_Pad1.08x0.95mm_HandSolder" H 4538 4400 50  0001 C CNN
@@
 $EndComp
 $Comp
-L Device:L L?
+L Device:L L3
 U 1 1 60E8569C
 P 6650 3500
-F 0 "L?" V 6750 3500 50  0000 C CNN
+F 0 "L3" V 6750 3500 50  0000 C CNN
 F 1 "330u" V 6600 3500 50  0000 C CNN
 F 2 "" H 6650 3500 50  0001 C CNN
@@
 	8500 5000 8000 5000
 $Comp
-L Device:D_Schottky D?
+L Device:D_Schottky D2
 U 1 1 60EBDE25
 P 7350 4000
-F 0 "D?" H 7350 3900 50  0000 C CNN
+F 0 "D2" H 7350 3900 50  0000 C CNN
 F 1 "MBR0540" H 7300 4100 50  0000 C CNN
 F 2 "" H 7350 4000 50  0001 C CNN

Commit message: Add files via upload
Parts:
- C22, C25: symbol Device:CP -> rata-rescue:CP-Device
- C23, C24: symbol Device:C -> rata-rescue:C-Device
- D2: symbol Device:D_Schottky -> rata-rescue:D_Schottky-Device
- L3: symbol Device:L -> rata-rescue:L-Device
- R12, R13, R14, R15: symbol Device:R -> rata-rescue:R-Device
- TP10, TP11, TP9: symbol Connector:TestPoint -> rata-rescue:TestPoint-Connector
- U5: symbol Regulator_Switching:MC34063AD -> rata-rescue:MC34063AD-Regulator_Switching
Changed lines of the file:
@@
 Boost converter +25V
 $Comp
-L Device:C C?
+L rata-rescue:C-Device C?
 U 1 1 60A0DAB2
 P 4000 4150
@@
 $EndComp
 $Comp
-L Device:R R?
+L rata-rescue:R-Device R?
 U 1 1 60A440E9
 P 5300 3500
@@
 $EndComp
 $Comp
-L Device:R R?
+L rata-rescue:R-Device R?
 U 1 1 60DF11BE
 P 6250 3650
@@
 $EndComp
 $Comp
-L Connector:TestPoint TP?
+L rata-rescue:TestPoint-Connector TP?
 U 1 1 60DF11BF
 P 8250 4000
@@
 $EndComp
 $Comp
-L Connector:TestPoint TP?
+L rata-rescue:TestPoint-Connector TP?
 U 1 1 60F5917B
 P 5600 3500
@@
 $EndComp
 $Comp
-L Device:CP C22
+L rata-rescue:CP-Device C22
 U 1 1 60F5917D
 P 3500 4150
@@
 +5V_IN
 $Comp
-L Connector:TestPoint TP?
+L rata-rescue:TestPoint-Connector TP?
 U 1 1 60AFF250
 P 5000 3500
@@
 GND
 $Comp
-L Device:R R?
+L rata-rescue:R-Device R?
 U 1 1 60DF11CA
 P 8000 4650
@@
 $EndComp
 $Comp
-L Regulator_Switching:MC34063AD U5
+L rata-rescue:MC34063AD-Regulator_Switching U5
 U 1 1 60DF4135
 P 5300 4200
@@
 $EndComp
 $Comp
-L Device:CP C25
+L rata-rescue:CP-Device C25
 U 1 1 60E7FC90
 P 8500 4150
@@
 $EndComp
 $Comp
-L Device:R R?
+L rata-rescue:R-Device R?
 U 1 1 60E80DA1
 P 8000 4150
@@
 $EndComp
 $Comp
-L Device:C C?
+L rata-rescue:C-Device C?
 U 1 1 60E81588
 P 4500 4550
@@
 $EndComp
 $Comp
-L Device:L L3
+L rata-rescue:L-Device L3
 U 1 1 60E8569C
 P 6650 3500
@@
 	8500 5000 8000 5000
 $Comp
-L Device:D_Schottky D2
+L rata-rescue:D_Schottky-Device D2
 U 1 1 60EBDE25
 P 7350 4000

Commit message: Add files via upload
Parts:
- C22: footprint (none) -> Capacitor_SMD:CP_Elec_6.3x7.7
- C25: footprint (none) -> Capacitor_SMD:CP_Elec_10x10.5
- D2: footprint (none) -> Diode_SMD:D_SOD-123
- L3: footprint (none) -> rata:L_12x12mm_H8mm
- R13: renamed from R12; footprint (none) -> Resistor_SMD:R_2010_5025Metric_Pad1.40x2.65mm_HandSolder
- TP10, TP11, TP9: footprint (none) -> rata:TP
- renumbered R13 to R14, R14 to R15, R15 to R16
Changed lines of the file:
@@
 encoding utf-8
 Sheet 7 23
-Title ""
-Date ""
-Rev ""
-Comp ""
+Title "rata"
+Date "2021-09-25"
+Rev "1.0"
+Comp "Yuriy Volkov"
 Comment1 ""
 Comment2 ""
@@
 AR Path="/60A440E9" Ref="R?"  Part="1"
 AR Path="/609FED99/60A440E9" Ref="R?"  Part="1"
-AR Path="/60DF0860/60A440E9" Ref="R12"  Part="1"
-F 0 "R12" V 5200 3450 50  0000 L CNN
+AR Path="/60DF0860/60A440E9" Ref="R13"  Part="1"
+F 0 "R13" V 5200 3450 50  0000 L CNN
 F 1 "0,47 2010" V 5400 3300 50  0000 L CNN
-F 2 "" V 5230 3500 50  0001 C CNN
+F 2 "Resistor_SMD:R_2010_5025Metric_Pad1.40x2.65mm_HandSolder" V 5230 3500 50  0001 C CNN
 F 3 "~" H 5300 3500 50  0001 C CNN
 	1    5300 3500
@@
 AR Path="/60DF11BE" Ref="R?"  Part="1"
 AR Path="/609FED99/60DF11BE" Ref="R?"  Part="1"
-AR Path="/60DF0860/60DF11BE" Ref="R13"  Part="1"
-F 0 "R13" H 6320 3696 50  0000 L CNN
+AR Path="/60DF0860/60DF11BE" Ref="R14"  Part="1"
+F 0 "R14" H 6320 3696 50  0000 L CNN
 F 1 "200" H 6320 3605 50  0000 L CNN
 F 2 "Resistor_SMD:R_0603_1608Metric_Pad0.98x0.95mm_HandSolder" V 6180 3650 50  0001 C CNN
@@
 F 0 "TP11" H 8308 4118 50  0000 L CNN
 F 1 "TestPoint" H 8308 4027 50  0001 L CNN
-F 2 "" H 8450 4000 50  0001 C CNN
+F 2 "rata:TP" H 8450 4000 50  0001 C CNN
 F 3 "~" H 8450 4000 50  0001 C CNN
 	1    8250 4000
@@
 F 0 "TP10" H 5658 3618 50  0000 L CNN
 F 1 "TestPoint" H 5658 3527 50  0001 L CNN
-F 2 "" H 5800 3500 50  0001 C CNN
+F 2 "rata:TP" H 5800 3500 50  0001 C CNN
 F 3 "~" H 5800 3500 50  0001 C CNN
 	1    5600 3500
@@
 F 0 "C22" H 3618 4196 50  0000 L CNN
 F 1 "100u" H 3618 4105 50  0000 L CNN
-F 2 "" H 3538 4000 50  0001 C CNN
+F 2 "Capacitor_SMD:CP_Elec_6.3x7.7" H 3538 4000 50  0001 C CNN
 F 3 "~" H 3500 4150 50  0001 C CNN
 	1    3500 4150
@@
 F 0 "TP9" H 5058 3618 50  0000 L CNN
 F 1 "TestPoint" H 5058 3527 50  0001 L CNN
-F 2 "" H 5200 3500 50  0001 C CNN
+F 2 "rata:TP" H 5200 3500 50  0001 C CNN
 F 3 "~" H 5200 3500 50  0001 C CNN
 	1    5000 3500
@@
 AR Path="/60B39FE1/60DF11CA" Ref="R?"  Part="1"
 AR Path="/609FED99/60DF11CA" Ref="R?"  Part="1"
-AR Path="/60DF0860/60DF11CA" Ref="R15"  Part="1"
-F 0 "R15" H 8070 4696 50  0000 L CNN
+AR Path="/60DF0860/60DF11CA" Ref="R16"  Part="1"
+F 0 "R16" H 8070 4696 50  0000 L CNN
 F 1 "2,4k 1%" H 8070 4605 50  0000 L CNN
 F 2 "Resistor_SMD:R_0603_1608Metric_Pad0.98x0.95mm_HandSolder" V 7930 4650 50  0001 C CNN
@@
 F 0 "C25" H 8618 4196 50  0000 L CNN
 F 1 "470u" H 8618 4105 50  0000 L CNN
-F 2 "" H 8538 4000 50  0001 C CNN
+F 2 "Capacitor_SMD:CP_Elec_10x10.5" H 8538 4000 50  0001 C CNN
 F 3 "~" H 8500 4150 50  0001 C CNN
 	1    8500 4150
@@
 AR Path="/60B39FE1/60E80DA1" Ref="R?"  Part="1"
 AR Path="/609FED99/60E80DA1" Ref="R?"  Part="1"
-AR Path="/60DF0860/60E80DA1" Ref="R14"  Part="1"
-F 0 "R14" H 8070 4196 50  0000 L CNN
+AR Path="/60DF0860/60E80DA1" Ref="R15"  Part="1"
+F 0 "R15" H 8070 4196 50  0000 L CNN
 F 1 "47k 1%" H 8070 4105 50  0000 L CNN
 F 2 "Resistor_SMD:R_0603_1608Metric_Pad0.98x0.95mm_HandSolder" V 7930 4150 50  0001 C CNN
@@
 F 0 "L3" V 6750 3500 50  0000 C CNN
 F 1 "330u" V 6600 3500 50  0000 C CNN
-F 2 "" H 6650 3500 50  0001 C CNN
+F 2 "rata:L_12x12mm_H8mm" H 6650 3500 50  0001 C CNN
 F 3 "~" H 6650 3500 50  0001 C CNN
 	1    6650 3500
@@
 Connection ~ 8500 4000
 Wire Wire Line
-	8500 4000 9500 4000
+	8500 4000 9000 4000
 Wire Wire Line
 	8500 4300 8500 5000
@@
 F 0 "D2" H 7350 3900 50  0000 C CNN
 F 1 "MBR0540" H 7300 4100 50  0000 C CNN
-F 2 "" H 7350 4000 50  0001 C CNN
+F 2 "Diode_SMD:D_SOD-123" H 7350 4000 50  0001 C CNN
 F 3 "~" H 7350 4000 50  0001 C CNN
 	1    7350 4000
@@
 Connection ~ 6000 5000
 Connection ~ 8000 5000
+$Comp
+L power:PWR_FLAG #FLG02
+U 1 1 615A480A
+P 9000 4000
+F 0 "#FLG02" H 9000 4075 50  0001 C CNN
+F 1 "PWR_FLAG" H 9000 4173 50  0000 C CNN
+F 2 "" H 9000 4000 50  0001 C CNN
+F 3 "~" H 9000 4000 50  0001 C CNN
+	1    9000 4000
+	1    0    0    -1
+$EndComp
+Connection ~ 9000 4000
+Wire Wire Line
+	9000 4000 9500 4000
 $EndSCHEMATC
