File: Power_+25V.sch (KiCad schematic (older format))
At the start: 14 parts, among them U5 MC34063AD

Commit message: Resistors values corrected to correspond actual values
Parts:
- R15: value 47k 1% -> 27k 1%
Connections:
- net +25V_OUT renamed +15V_OUT
Other:
- note added: "Boost converter +15V"
- note removed: "Boost converter +25V"
Changed lines of the file:
@@
 $Descr A4 11693 8268
 encoding utf-8
-Sheet 7 23
+Sheet 23 23
 Title "rata"
 Date "2021-09-25"
@@
 $EndDescr
 Text Notes 7000 2250 2    197  ~ 0
-Boost converter +25V
+Boost converter +15V
 $Comp
 L rata-rescue:C-Device C?
@@
 AR Path="/60DF0860/60E80DA1" Ref="R15"  Part="1"
 F 0 "R15" H 8070 4196 50  0000 L CNN
-F 1 "47k 1%" H 8070 4105 50  0000 L CNN
+F 1 "27k 1%" H 8070 4105 50  0000 L CNN
 F 2 "Resistor_SMD:R_0603_1608Metric_Pad0.98x0.95mm_HandSolder" V 7930 4150 50  0001 C CNN
 F 3 "~" H 8000 4150 50  0001 C CNN
@@
 $EndComp
 Text HLabel 9500 4000 2    50   Output ~ 0
-+25V_OUT
++15V_OUT
 Wire Wire Line
 	2500 4000 3500 4000
