File: Power_+3V3A.sch (KiCad schematic (older format))
At the start: 12 parts, among them U17 AMS1117-3.3

Commit message: Add files via upload
Parts:
- C61, C63: symbol Device:CP -> rata-rescue:CP-Device
- C62, C64, C65, C66: symbol Device:C -> rata-rescue:C-Device
- FB4: symbol Device:Ferrite_Bead -> rata-rescue:Ferrite_Bead-Device
- L4: symbol Device:L -> rata-rescue:L-Device
- TP30, TP31, TP32: symbol Connector:TestPoint -> rata-rescue:TestPoint-Connector
- U17: symbol Regulator_Linear:AMS1117-3.3 -> rata-rescue:AMS1117-3.3-Regulator_Linear
Other:
- moved on the sheet: C61, C62, C63, C64, C65, C66, TP31
Changed lines of the file:
@@
 $EndDescr
 $Comp
-L Regulator_Linear:AMS1117-3.3 U?
+L rata-rescue:AMS1117-3.3-Regulator_Linear U?
 U 1 1 611C22D7
 P 6800 3500
@@
 $EndComp
 $Comp
-L Device:C C?
+L rata-rescue:C-Device C?
 U 1 1 60E73024
-P 7400 3650
+P 7400 3750
 AR Path="/60E73024" Ref="C?"  Part="1"
 AR Path="/609CA6A8/609D24C0/60E73024" Ref="C?"  Part="1"
@@
 AR Path="/60DF212D/60E73024" Ref="C?"  Part="1"
 AR Path="/60E6F2E9/60E73024" Ref="C65"  Part="1"
-F 0 "C65" H 7515 3696 50  0000 L CNN
-F 1 "10u" H 7515 3605 50  0000 L CNN
-F 2 "Capacitor_SMD:C_1206_3216Metric_Pad1.33x1.80mm_HandSolder" H 7438 3500 50  0001 C CNN
-F 3 "~" H 7400 3650 50  0001 C CNN
-	1    7400 3650
-	1    0    0    -1
-$EndComp
-$Comp
-L Device:C C?
+F 0 "C65" H 7515 3796 50  0000 L CNN
+F 1 "10u" H 7515 3705 50  0000 L CNN
+F 2 "Capacitor_SMD:C_1206_3216Metric_Pad1.33x1.80mm_HandSolder" H 7438 3600 50  0001 C CNN
+F 3 "~" H 7400 3750 50  0001 C CNN
+	1    7400 3750
+	1    0    0    -1
+$EndComp
+$Comp
+L rata-rescue:C-Device C?
 U 1 1 611C22D9
-P 6200 3650
+P 6200 3750
 AR Path="/611C22D9" Ref="C?"  Part="1"
 AR Path="/609CA6A8/609D24C0/611C22D9" Ref="C?"  Part="1"
@@
 AR Path="/60DF212D/611C22D9" Ref="C?"  Part="1"
 AR Path="/60E6F2E9/611C22D9" Ref="C64"  Part="1"
-F 0 "C64" H 6315 3696 50  0000 L CNN
-F 1 "0,1" H 6315 3605 50  0000 L CNN
-F 2 "Capacitor_SMD:C_0603_1608Metric_Pad1.08x0.95mm_HandSolder" H 6238 3500 50  0001 C CNN
-F 3 "~" H 6200 3650 50  0001 C CNN
-	1    6200 3650
-	1    0    0    -1
-$EndComp
-$Comp
-L Device:C C?
+F 0 "C64" H 6315 3796 50  0000 L CNN
+F 1 "0,1" H 6315 3705 50  0000 L CNN
+F 2 "Capacitor_SMD:C_0603_1608Metric_Pad1.08x0.95mm_HandSolder" H 6238 3600 50  0001 C CNN
+F 3 "~" H 6200 3750 50  0001 C CNN
+	1    6200 3750
+	1    0    0    -1
+$EndComp
+$Comp
+L rata-rescue:C-Device C?
 U 1 1 60E7301F
-P 7800 3650
+P 7800 3750
 AR Path="/60E7301F" Ref="C?"  Part="1"
 AR Path="/609CA6A8/609D24C0/60E7301F" Ref="C?"  Part="1"
@@
 AR Path="/60DF212D/60E7301F" Ref="C?"  Part="1"
 AR Path="/60E6F2E9/60E7301F" Ref="C66"  Part="1"
-F 0 "C66" H 7915 3696 50  0000 L CNN
-F 1 "10u" H 7915 3605 50  0000 L CNN
-F 2 "Capacitor_SMD:C_1206_3216Metric_Pad1.33x1.80mm_HandSolder" H 7838 3500 50  0001 C CNN
-F 3 "~" H 7800 3650 50  0001 C CNN
-	1    7800 3650
-	1    0    0    -1
-$EndComp
-Wire Wire Line
-	6200 3500 6500 3500
-Wire Wire Line
-	7100 3500 7400 3500
-Wire Wire Line
-	7800 3800 7400 3800
-Connection ~ 6800 3800
-Wire Wire Line
-	6800 3800 6200 3800
-Connection ~ 7400 3800
-$Comp
-L Connector:TestPoint TP?
+F 0 "C66" H 7915 3796 50  0000 L CNN
+F 1 "10u" H 7915 3705 50  0000 L CNN
+F 2 "Capacitor_SMD:C_1206_3216Metric_Pad1.33x1.80mm_HandSolder" H 7838 3600 50  0001 C CNN
+F 3 "~" H 7800 3750 50  0001 C CNN
+	1    7800 3750
+	1    0    0    -1
+$EndComp
+$Comp
+L rata-rescue:TestPoint-Connector TP?
 U 1 1 60DF19BA
 P 7550 3500
@@
 $EndComp
 $Comp
-L Connector:TestPoint TP?
+L rata-rescue:TestPoint-Connector TP?
 U 1 1 60E73021
 P 5400 3500
@@
 Text HLabel 2000 3500 0    50   Input ~ 0
 +5V_IN
-Connection ~ 6200 3500
-Connection ~ 6200 3800
-Wire Wire Line
-	6800 3800 7400 3800
-$Comp
-L Connector:TestPoint TP?
+$Comp
+L rata-rescue:TestPoint-Connector TP?
 U 1 1 611C22D3
-P 5400 3800
+P 5400 4000
 AR Path="/611C22D3" Ref="TP?"  Part="1"
 AR Path="/609FED99/611C22D3" Ref="TP?"  Part="1"
@@
 AR Path="/60DF212D/611C22D3" Ref="TP?"  Part="1"
 AR Path="/60E6F2E9/611C22D3" Ref="TP31"  Part="1"
-F 0 "TP31" H 5458 3918 50  0000 L CNN
-F 1 "TestPoint" H 5458 3827 50  0001 L CNN
-F 2 "" H 5600 3800 50  0001 C CNN
-F 3 "~" H 5600 3800 50  0001 C CNN
-	1    5400 3800
-	1    0    0    -1
-$EndComp
-Wire Wire Line
-	7400 3500 7550 3500
-Connection ~ 7400 3500
-Wire Wire Line
-	7550 3500 7800 3500
+F 0 "TP31" H 5458 4118 50  0000 L CNN
+F 1 "TestPoint" H 5458 4027 50  0001 L CNN
+F 2 "" H 5600 4000 50  0001 C CNN
+F 3 "~" H 5600 4000 50  0001 C CNN
+	1    5400 4000
+	1    0    0    -1
+$EndComp
 Connection ~ 7550 3500
-Text HLabel 2000 3800 0    50   Input ~ 0
+Text HLabel 2000 4000 0    50   Input ~ 0
 GND
 Text Notes 6900 2250 2    197  ~ 0
 Power source +3V3 analog\n
-Wire Wire Line
-	5400 3500 6200 3500
-Wire Wire Line
-	5400 3800 6200 3800
 Text HLabel 8500 3500 2    50   Output ~ 0
 +3V3_OUT
-Wire Wire Line
-	7800 3500 8500 3500
-Connection ~ 7800 3500
-$Comp
-L Device:C C?
+$Comp
+L rata-rescue:C-Device C?
 U 1 1 60FB3F89
-P 3000 3650
+P 3000 3750
 AR Path="/60FB3F89" Ref="C?"  Part="1"
 AR Path="/609CA6A8/609D24C0/60FB3F89" Ref="C?"  Part="1"
@@
 AR Path="/60E6F2E9/60FB3F89" Ref="C62"  Part="1"
 AR Path="/60EE89A9/60FB3F89" Ref="C?"  Part="1"
-F 0 "C62" H 3115 3696 50  0000 L CNN
-F 1 "1u" H 3115 3605 50  0000 L CNN
-F 2 "Capacitor_SMD:C_0603_1608Metric_Pad1.08x0.95mm_HandSolder" H 3038 3500 50  0001 C CNN
-F 3 "~" H 3000 3650 50  0001 C CNN
-	1    3000 3650
-	1    0    0    -1
-$EndComp
-$Comp
-L Device:CP C?
+F 0 "C62" H 3115 3796 50  0000 L CNN
+F 1 "1u" H 3115 3705 50  0000 L CNN
+F 2 "Capacitor_SMD:C_0603_1608Metric_Pad1.08x0.95mm_HandSolder" H 3038 3600 50  0001 C CNN
+F 3 "~" H 3000 3750 50  0001 C CNN
+	1    3000 3750
+	1    0    0    -1
+$EndComp
+$Comp
+L rata-rescue:CP-Device C?
 U 1 1 60FB3F8F
-P 2500 3650
+P 2500 3750
 AR Path="/609FED99/60FB3F8F" Ref="C?"  Part="1"
 AR Path="/60DF07DE/60FB3F8F" Ref="C?"  Part="1"
@@
 AR Path="/60E6F2E9/60FB3F8F" Ref="C61"  Part="1"
 AR Path="/60EE89A9/60FB3F8F" Ref="C?"  Part="1"
-F 0 "C61" H 2618 3696 50  0000 L CNN
-F 1 "100u" H 2618 3605 50  0000 L CNN
-F 2 "" H 2538 3500 50  0001 C CNN
-F 3 "~" H 2500 3650 50  0001 C CNN
-	1    2500 3650
-	1    0    0    -1
-$EndComp
-$Comp
-L Device:CP C?
+F 0 "C61" H 2618 3796 50  0000 L CNN
+F 1 "100u" H 2618 3705 50  0000 L CNN
+F 2 "" H 2538 3600 50  0001 C CNN
+F 3 "~" H 2500 3750 50  0001 C CNN
+	1    2500 3750
+	1    0    0    -1
+$EndComp
+$Comp
+L rata-rescue:CP-Device C?
 U 1 1 60FC0F28
-P 5000 3650
+P 5000 3750
 AR Path="/609FED99/60FC0F28" Ref="C?"  Part="1"
 AR Path="/60DF07DE/60FC0F28" Ref="C?"  Part="1"
@@
 AR Path="/60E6F2E9/60FC0F28" Ref="C63"  Part="1"
 AR Path="/60EE89A9/60FC0F28" Ref="C?"  Part="1"
-F 0 "C63" H 5118 3696 50  0000 L CNN
-F 1 "100u" H 5118 3605 50  0000 L CNN
-F 2 "" H 5038 3500 50  0001 C CNN
-F 3 "~" H 5000 3650 50  0001 C CNN
-	1    5000 3650
-	1    0    0    -1
-$EndComp
-$Comp
-L Device:Ferrite_Bead FB?
+F 0 "C63" H 5118 3796 50  0000 L CNN
+F 1 "100u" H 5118 3705 50  0000 L CNN
+F 2 "" H 5038 3600 50  0001 C CNN
+F 3 "~" H 5000 3750 50  0001 C CNN
+	1    5000 3750
+	1    0    0    -1
+$EndComp
+$Comp
+L rata-rescue:Ferrite_Bead-Device FB?
 U 1 1 60FC2E70
 P 4250 3500
@@
 $EndComp
 $Comp
-L Device:L L?
+L rata-rescue:L-Device L?
 U 1 1 60FC380F
 P 3750 3500
@@
 $EndComp
 Wire Wire Line
+	3900 3500 4100 3500
+Connection ~ 5400 3500
+Wire Wire Line
+	7550 3500 7800 3500
+Wire Wire Line
+	7100 3500 7400 3500
+Wire Wire Line
+	5400 3500 6200 3500
+Wire Wire Line
+	4400 3500 5000 3500
+Wire Wire Line
 	2000 3500 2500 3500
+Wire Wire Line
+	2000 4000 2500 4000
+Wire Wire Line
+	7800 4000 7800 3900
+Wire Wire Line
+	7800 3600 7800 3500
+Connection ~ 7800 3500
+Wire Wire Line
+	7800 3500 8500 3500
+Wire Wire Line
+	7400 3600 7400 3500
+Connection ~ 7400 3500
+Wire Wire Line
+	7400 3500 7550 3500
+Wire Wire Line
+	7400 3900 7400 4000
+Connection ~ 7400 4000
+Wire Wire Line
+	7400 4000 7800 4000
+Wire Wire Line
+	6800 3800 6800 4000
+Connection ~ 6800 4000
+Wire Wire Line
+	6800 4000 7400 4000
+Wire Wire Line
+	6200 3600 6200 3500
+Connection ~ 6200 3500
+Wire Wire Line
+	6200 3500 6500 3500
+Wire Wire Line
+	6200 3900 6200 4000
+Connection ~ 6200 4000
+Wire Wire Line
+	6200 4000 6800 4000
+Connection ~ 5400 4000
+Wire Wire Line
+	5400 4000 6200 4000
+Wire Wire Line
+	5000 3600 5000 3500
+Connection ~ 5000 3500
+Wire Wire Line
+	5000 3500 5400 3500
+Wire Wire Line
+	5000 3900 5000 4000
+Connection ~ 5000 4000
+Wire Wire Line
+	5000 4000 5400 4000
+Wire Wire Line
+	3000 3600 3000 3500
+Connection ~ 3000 3500
+Wire Wire Line
+	3000 3500 3600 3500
+Wire Wire Line
+	3000 3900 3000 4000
+Connection ~ 3000 4000
+Wire Wire Line
+	3000 4000 5000 4000
+Wire Wire Line
+	2500 3600 2500 3500
 Connection ~ 2500 3500
 Wire Wire Line
 	2500 3500 3000 3500
-Connection ~ 3000 3500
-Wire Wire Line
-	3000 3500 3600 3500
-Wire Wire Line
-	3900 3500 4100 3500
-Wire Wire Line
-	4400 3500 5000 3500
-Connection ~ 5400 3500
-Connection ~ 5000 3500
-Wire Wire Line
-	5000 3500 5400 3500
-Wire Wire Line
-	2000 3800 2500 3800
-Connection ~ 5400 3800
-Connection ~ 2500 3800
-Wire Wire Line
-	2500 3800 3000 3800
-Connection ~ 3000 3800
-Wire Wire Line
-	3000 3800 5000 3800
-Connection ~ 5000 3800
-Wire Wire Line
-	5000 3800 5400 3800
+Wire Wire Line
+	2500 3900 2500 4000
+Connection ~ 2500 4000
+Wire Wire Line
+	2500 4000 3000 4000
 $EndSCHEMATC

Commit message: Add files via upload
Parts:
- C58: renamed from C61; footprint (none) -> Capacitor_SMD:CP_Elec_6.3x7.7
- C60: renamed from C63; footprint (none) -> Capacitor_SMD:CP_Elec_6.3x7.7
- FB4: footprint (none) -> Inductor_SMD:L_0805_2012Metric_Pad1.05x1.20mm_HandSolder
- L4: footprint (none) -> rata:L_12x12mm_H8mm
- TP30, TP31, TP32: footprint (none) -> rata:TP
- renumbered C62 to C59, C64 to C61, C65 to C62, C66 to C63, U17 to U13
Changed lines of the file:
@@
 $Descr A4 11693 8268
 encoding utf-8
-Sheet 23 23
-Title ""
-Date ""
-Rev ""
-Comp ""
+Sheet 22 23
+Title "rata"
+Date "2021-09-25"
+Rev "1.0"
+Comp "Yuriy Volkov"
 Comment1 ""
 Comment2 ""
@@
 AR Path="/60DF196E/611C22D7" Ref="U?"  Part="1"
 AR Path="/60DF212D/611C22D7" Ref="U?"  Part="1"
-AR Path="/60E6F2E9/611C22D7" Ref="U17"  Part="1"
-F 0 "U17" H 6800 3742 50  0000 C CNN
+AR Path="/60E6F2E9/611C22D7" Ref="U13"  Part="1"
+F 0 "U13" H 6800 3742 50  0000 C CNN
 F 1 "AMS1117-3.3" H 6800 3651 50  0000 C CNN
 F 2 "Package_TO_SOT_SMD:SOT-223-3_TabPin2" H 6800 3700 50  0001 C CNN
@@
 AR Path="/60DF196E/60E73024" Ref="C?"  Part="1"
 AR Path="/60DF212D/60E73024" Ref="C?"  Part="1"
-AR Path="/60E6F2E9/60E73024" Ref="C65"  Part="1"
-F 0 "C65" H 7515 3796 50  0000 L CNN
+AR Path="/60E6F2E9/60E73024" Ref="C62"  Part="1"
+F 0 "C62" H 7515 3796 50  0000 L CNN
 F 1 "10u" H 7515 3705 50  0000 L CNN
 F 2 "Capacitor_SMD:C_1206_3216Metric_Pad1.33x1.80mm_HandSolder" H 7438 3600 50  0001 C CNN
@@
 AR Path="/60DF196E/611C22D9" Ref="C?"  Part="1"
 AR Path="/60DF212D/611C22D9" Ref="C?"  Part="1"
-AR Path="/60E6F2E9/611C22D9" Ref="C64"  Part="1"
-F 0 "C64" H 6315 3796 50  0000 L CNN
+AR Path="/60E6F2E9/611C22D9" Ref="C61"  Part="1"
+F 0 "C61" H 6315 3796 50  0000 L CNN
 F 1 "0,1" H 6315 3705 50  0000 L CNN
 F 2 "Capacitor_SMD:C_0603_1608Metric_Pad1.08x0.95mm_HandSolder" H 6238 3600 50  0001 C CNN
@@
 AR Path="/60DF196E/60E7301F" Ref="C?"  Part="1"
 AR Path="/60DF212D/60E7301F" Ref="C?"  Part="1"
-AR Path="/60E6F2E9/60E7301F" Ref="C66"  Part="1"
-F 0 "C66" H 7915 3796 50  0000 L CNN
+AR Path="/60E6F2E9/60E7301F" Ref="C63"  Part="1"
+F 0 "C63" H 7915 3796 50  0000 L CNN
 F 1 "10u" H 7915 3705 50  0000 L CNN
 F 2 "Capacitor_SMD:C_1206_3216Metric_Pad1.33x1.80mm_HandSolder" H 7838 3600 50  0001 C CNN
@@
 F 0 "TP32" H 7608 3618 50  0000 L CNN
 F 1 "TestPoint" H 7608 3527 50  0001 L CNN
-F 2 "" H 7750 3500 50  0001 C CNN
+F 2 "rata:TP" H 7750 3500 50  0001 C CNN
 F 3 "~" H 7750 3500 50  0001 C CNN
 	1    7550 3500
@@
 F 0 "TP30" H 5458 3618 50  0000 L CNN
 F 1 "TestPoint" H 5458 3527 50  0001 L CNN
-F 2 "" H 5600 3500 50  0001 C CNN
+F 2 "rata:TP" H 5600 3500 50  0001 C CNN
 F 3 "~" H 5600 3500 50  0001 C CNN
 	1    5400 3500
@@
 F 0 "TP31" H 5458 4118 50  0000 L CNN
 F 1 "TestPoint" H 5458 4027 50  0001 L CNN
-F 2 "" H 5600 4000 50  0001 C CNN
+F 2 "rata:TP" H 5600 4000 50  0001 C CNN
 F 3 "~" H 5600 4000 50  0001 C CNN
 	1    5400 4000
@@
 AR Path="/60DF196E/60FB3F89" Ref="C?"  Part="1"
 AR Path="/60DF212D/60FB3F89" Ref="C?"  Part="1"
-AR Path="/60E6F2E9/60FB3F89" Ref="C62"  Part="1"
+AR Path="/60E6F2E9/60FB3F89" Ref="C59"  Part="1"
 AR Path="/60EE89A9/60FB3F89" Ref="C?"  Part="1"
-F 0 "C62" H 3115 3796 50  0000 L CNN
+F 0 "C59" H 3115 3796 50  0000 L CNN
 F 1 "1u" H 3115 3705 50  0000 L CNN
 F 2 "Capacitor_SMD:C_0603_1608Metric_Pad1.08x0.95mm_HandSolder" H 3038 3600 50  0001 C CNN
@@
 AR Path="/60DF196E/60FB3F8F" Ref="C?"  Part="1"
 AR Path="/60DF212D/60FB3F8F" Ref="C?"  Part="1"
-AR Path="/60E6F2E9/60FB3F8F" Ref="C61"  Part="1"
+AR Path="/60E6F2E9/60FB3F8F" Ref="C58"  Part="1"
 AR Path="/60EE89A9/60FB3F8F" Ref="C?"  Part="1"
-F 0 "C61" H 2618 3796 50  0000 L CNN
+F 0 "C58" H 2618 3796 50  0000 L CNN
 F 1 "100u" H 2618 3705 50  0000 L CNN
-F 2 "" H 2538 3600 50  0001 C CNN
+F 2 "Capacitor_SMD:CP_Elec_6.3x7.7" H 2538 3600 50  0001 C CNN
 F 3 "~" H 2500 3750 50  0001 C CNN
 	1    2500 3750
@@
 AR Path="/60DF196E/60FC0F28" Ref="C?"  Part="1"
 AR Path="/60DF212D/60FC0F28" Ref="C?"  Part="1"
-AR Path="/60E6F2E9/60FC0F28" Ref="C63"  Part="1"
+AR Path="/60E6F2E9/60FC0F28" Ref="C60"  Part="1"
 AR Path="/60EE89A9/60FC0F28" Ref="C?"  Part="1"
-F 0 "C63" H 5118 3796 50  0000 L CNN
+F 0 "C60" H 5118 3796 50  0000 L CNN
 F 1 "100u" H 5118 3705 50  0000 L CNN
-F 2 "" H 5038 3600 50  0001 C CNN
+F 2 "Capacitor_SMD:CP_Elec_6.3x7.7" H 5038 3600 50  0001 C CNN
 F 3 "~" H 5000 3750 50  0001 C CNN
 	1    5000 3750
@@
 F 0 "FB4" V 3976 3500 50  0000 C CNN
 F 1 "Ferrite_Bead" V 4067 3500 50  0000 C CNN
-F 2 "" V 4180 3500 50  0001 C CNN
+F 2 "Inductor_SMD:L_0805_2012Metric_Pad1.05x1.20mm_HandSolder" V 4180 3500 50  0001 C CNN
 F 3 "~" H 4250 3500 50  0001 C CNN
 	1    4250 3500
@@
 F 0 "L4" V 3850 3500 50  0000 C CNN
 F 1 "330u" V 3700 3500 50  0000 C CNN
-F 2 "" H 3750 3500 50  0001 C CNN
+F 2 "rata:L_12x12mm_H8mm" H 3750 3500 50  0001 C CNN
 F 3 "~" H 3750 3500 50  0001 C CNN
 	1    3750 3500
@@
 	7100 3500 7400 3500
 Wire Wire Line
-	5400 3500 6200 3500
+	5400 3500 6000 3500
 Wire Wire Line
 	4400 3500 5000 3500
@@
 Wire Wire Line
 	2500 4000 3000 4000
+$Comp
+L power:PWR_FLAG #FLG09
+U 1 1 615BF45A
+P 6000 3500
+F 0 "#FLG09" H 6000 3575 50  0001 C CNN
+F 1 "PWR_FLAG" H 6000 3673 50  0000 C CNN
+F 2 "" H 6000 3500 50  0001 C CNN
+F 3 "~" H 6000 3500 50  0001 C CNN
+	1    6000 3500
+	1    0    0    -1
+$EndComp
+Connection ~ 6000 3500
+Wire Wire Line
+	6000 3500 6200 3500
 $EndSCHEMATC
