File: Power_+4.5V.sch (KiCad schematic (older format))
At the start: 19 parts

Commit message: Add files via upload
Parts:
- removed C? (x2): 0,1, Capacitor_SMD:C_0603_1608Metric_Pad1.08x0.95mm_HandSolder, symbol Device:C
- removed C?: 500, Capacitor_SMD:C_0603_1608Metric_Pad1.08x0.95mm_HandSolder, symbol Device:C
- removed C?: 100u, symbol Device:CP
- removed C? (x2): 470u, symbol Device:CP
- removed D?: MBR0540, symbol Device:D_Schottky
- removed L? (x2): 330u, symbol Device:L
- removed R?: 0,47 2010, symbol Device:R
- removed R?: 200, Resistor_SMD:R_0603_1608Metric_Pad0.98x0.95mm_HandSolder, symbol Device:R
- removed R?: 2,4k 1%, Resistor_SMD:R_0603_1608Metric_Pad0.98x0.95mm_HandSolder, symbol Device:R
- removed R?: 47k 1%, Resistor_SMD:R_0603_1608Metric_Pad0.98x0.95mm_HandSolder, symbol Device:R
- removed TP? (x5): TestPoint, symbol Connector:TestPoint
- removed U?: MC34063AD, Package_SO:SOIC-8_3.9x4.9mm_P1.27mm, symbol Regulator_Switching:MC34063AD
- added C?: 100u, symbol Device:CP
- added C? (x2): 470u, symbol Device:CP
- added C? (x2): 0,1, Capacitor_SMD:C_0603_1608Metric_Pad1.08x0.95mm_HandSolder, symbol Device:C
- added C?: 500, Capacitor_SMD:C_0603_1608Metric_Pad1.08x0.95mm_HandSolder, symbol Device:C
- added D?: MBR0540, symbol Device:D_Schottky
- added L? (x2): 330u, symbol Device:L
- added R?: 47k 1%, Resistor_SMD:R_0603_1608Metric_Pad0.98x0.95mm_HandSolder, symbol Device:R
- added R?: 0,47 2010, symbol Device:R
- added R?: 200, Resistor_SMD:R_0603_1608Metric_Pad0.98x0.95mm_HandSolder, symbol Device:R
- added R?: 2,4k 1%, Resistor_SMD:R_0603_1608Metric_Pad0.98x0.95mm_HandSolder, symbol Device:R
- added TP? (x5): TestPoint, symbol Connector:TestPoint
- added U?: MC34063AD, Package_SO:SOIC-8_3.9x4.9mm_P1.27mm, symbol Regulator_Switching:MC34063AD
Connections:
- net +10V_OUT: now also C?.1, C?.1, L?.2, TP?.1
- net +5V_IN: now also C?.1, C?.1, R?.2, TP?.1, U?.6 (Vin)
- net GND: now also C?.2, C?.2, C?.2, C?.2, C?.2, C?.2, R?.2, TP?.1, U?.2 (SwE), U?.4 (GND)
- new net: C?.1, D?.1 (K), L?.1, R?.1, TP?.1
- new net: R?.1, R?.2, U?.5 (Vfb)
- new net: L?.1, R?.1, R?.1, TP?.1, U?.7 (Ipk)
- new net: D?.2 (A), L?.2, U?.1 (SwC)
- new net: R?.2, U?.8 (DC)
- new net: C?.1, U?.3 (TC)
Other:
- note added: "Power source +10V"
- note removed: "Boost converter +10V"

Commit message: Add files via upload
Parts:
- removed C?: 100u, symbol Device:CP
- removed C? (x2): 470u, symbol Device:CP
- removed C? (x2): 0,1, Capacitor_SMD:C_0603_1608Metric_Pad1.08x0.95mm_HandSolder, symbol Device:C
- removed C?: 500, Capacitor_SMD:C_0603_1608Metric_Pad1.08x0.95mm_HandSolder, symbol Device:C
- removed D?: MBR0540, symbol Device:D_Schottky
- removed L? (x2): 330u, symbol Device:L
- removed R?: 47k 1%, Resistor_SMD:R_0603_1608Metric_Pad0.98x0.95mm_HandSolder, symbol Device:R
- removed R?: 0,47 2010, symbol Device:R
- removed R?: 200, Resistor_SMD:R_0603_1608Metric_Pad0.98x0.95mm_HandSolder, symbol Device:R
- removed R?: 2,4k 1%, Resistor_SMD:R_0603_1608Metric_Pad0.98x0.95mm_HandSolder, symbol Device:R
- removed TP? (x4): TestPoint, symbol Connector:TestPoint
- removed U?: MC34063AD, Package_SO:SOIC-8_3.9x4.9mm_P1.27mm, symbol Regulator_Switching:MC34063AD
- added C?: 4.7u, Capacitor_SMD:C_1206_3216Metric_Pad1.33x1.80mm_HandSolder, symbol Device:C
- added C?: 0,1, Capacitor_SMD:C_0603_1608Metric_Pad1.08x0.95mm_HandSolder, symbol Device:C
- added C?: 0,01, Capacitor_SMD:C_0603_1608Metric_Pad1.08x0.95mm_HandSolder, symbol Device:C
- added R? (x2): 1k 1%, Resistor_SMD:R_0603_1608Metric_Pad0.98x0.95mm_HandSolder, symbol Device:R
- added R? (x2): 2.7k 1%, Resistor_SMD:R_0603_1608Metric_Pad0.98x0.95mm_HandSolder, symbol Device:R
- added U?: LP2951-5.0_SOIC, Package_SO:SOIC-8_3.9x4.9mm_P1.27mm, symbol Regulator_Linear:LP2951-5.0_SOIC
Connections:
- net +5V_IN: now also C?.1, U?.8 (IN)
- net GND: now also C?.2, C?.2, R?.2, R?.2, U?.4 (GND)
- net +4V5_OUT: now reaches TP?.1
- net +4V5_OUT: now also C?.1, C?.1, R?.1, R?.1, U?.1 (OUT)
- new net: C?.2, R?.1, R?.2, U?.7 (FEEDBACK)
- new net SD: U?.3 (SHUTDOWN)
- new net VOLT: R?.1, R?.2
- no-connect marks 0 -> 3
Other:
- note added: "LDO +4V5"
- note removed: "Power source +10V"
- moved on the sheet: TP?

Commit message: Add files via upload
Parts:
- added R43: 0, symbol Device:R
- added TP19, TP20: TestPoint, symbol Connector:TestPoint
- gave numbers to parts that had none: 9
Connections:
- net +5V_IN: now also R43.1, TP19.1; no longer C51.1, U11.8 (IN)
- new net: C51.1, R43.2, TP20.1, U11.8 (IN)
Changed lines of the file:
@@
 $Descr A4 11693 8268
 encoding utf-8
-Sheet 15 23
+Sheet 14 23
 Title ""
 Date ""
@@
 AR Path="/60DF0860/60F18F0D" Ref="TP?"  Part="1"
 AR Path="/60DF07DE/60F18F0D" Ref="TP?"  Part="1"
-AR Path="/60F1863C/60F18F0D" Ref="TP?"  Part="1"
-F 0 "TP?" H 8558 3118 50  0000 L CNN
+AR Path="/60F1863C/60F18F0D" Ref="TP21"  Part="1"
+F 0 "TP21" H 8558 3118 50  0000 L CNN
 F 1 "TestPoint" H 8558 3027 50  0001 L CNN
 F 2 "" H 8700 3000 50  0001 C CNN
@@
 	1    0    0    -1
 $EndComp
-Text HLabel 3500 3000 0    50   Input ~ 0
+Text HLabel 3000 3000 0    50   Input ~ 0
 +5V_IN
-Text HLabel 3500 4000 0    50   Input ~ 0
+Text HLabel 3000 4000 0    50   Input ~ 0
 GND
 Text HLabel 9000 3000 2    50   Output ~ 0
 +4V5_OUT
 $Comp
-L Regulator_Linear:LP2951-5.0_SOIC U?
+L Regulator_Linear:LP2951-5.0_SOIC U11
 U 1 1 60F560B0
 P 5400 3300
-F 0 "U?" H 5400 3867 50  0000 C CNN
+F 0 "U11" H 5400 3867 50  0000 C CNN
 F 1 "LP2951-5.0_SOIC" H 5400 3776 50  0000 C CNN
 F 2 "Package_SO:SOIC-8_3.9x4.9mm_P1.27mm" H 5400 2650 50  0001 C CNN
@@
 AR Path="/60DF212D/60F593FA" Ref="C?"  Part="1"
 AR Path="/60E6F2E9/60F593FA" Ref="C?"  Part="1"
-AR Path="/60F1863C/60F593FA" Ref="C?"  Part="1"
-F 0 "C?" H 7615 3196 50  0000 L CNN
+AR Path="/60F1863C/60F593FA" Ref="C53"  Part="1"
+F 0 "C53" H 7615 3196 50  0000 L CNN
 F 1 "4.7u" H 7615 3105 50  0000 L CNN
 F 2 "Capacitor_SMD:C_1206_3216Metric_Pad1.33x1.80mm_HandSolder" H 7538 3000 50  0001 C CNN
@@
 AR Path="/60DF212D/60F59400" Ref="C?"  Part="1"
 AR Path="/60E6F2E9/60F59400" Ref="C?"  Part="1"
-AR Path="/60F1863C/60F59400" Ref="C?"  Part="1"
-F 0 "C?" H 4615 3196 50  0000 L CNN
+AR Path="/60F1863C/60F59400" Ref="C51"  Part="1"
+F 0 "C51" H 4615 3196 50  0000 L CNN
 F 1 "0,1" H 4615 3105 50  0000 L CNN
 F 2 "Capacitor_SMD:C_0603_1608Metric_Pad1.08x0.95mm_HandSolder" H 4538 3000 50  0001 C CNN
@@
 AR Path="/60DF0860/60F5D079" Ref="R?"  Part="1"
 AR Path="/60DF07DE/60F5D079" Ref="R?"  Part="1"
-AR Path="/60F1863C/60F5D079" Ref="R?"  Part="1"
-F 0 "R?" H 6820 3796 50  0000 L CNN
+AR Path="/60F1863C/60F5D079" Ref="R45"  Part="1"
+F 0 "R45" H 6820 3796 50  0000 L CNN
 F 1 "1k 1%" H 6820 3705 50  0000 L CNN
 F 2 "Resistor_SMD:R_0603_1608Metric_Pad0.98x0.95mm_HandSolder" V 6680 3750 50  0001 C CNN
@@
 AR Path="/60DF0860/60F5D07F" Ref="R?"  Part="1"
 AR Path="/60DF07DE/60F5D07F" Ref="R?"  Part="1"
-AR Path="/60F1863C/60F5D07F" Ref="R?"  Part="1"
-F 0 "R?" H 6820 3196 50  0000 L CNN
+AR Path="/60F1863C/60F5D07F" Ref="R44"  Part="1"
+F 0 "R44" H 6820 3196 50  0000 L CNN
 F 1 "2.7k 1%" H 6820 3105 50  0000 L CNN
 F 2 "Resistor_SMD:R_0603_1608Metric_Pad0.98x0.95mm_HandSolder" V 6680 3150 50  0001 C CNN
@@
 	1    0    0    -1
 $EndComp
-Text HLabel 3500 3500 0    50   Input ~ 0
+Text HLabel 3000 3500 0    50   Input ~ 0
 SD
 Text HLabel 9000 3500 2    50   Output ~ 0
@@
 AR Path="/60DF212D/60F5ECDF" Ref="C?"  Part="1"
 AR Path="/60E6F2E9/60F5ECDF" Ref="C?"  Part="1"
-AR Path="/60F1863C/60F5ECDF" Ref="C?"  Part="1"
-F 0 "C?" H 6365 3196 50  0000 L CNN
+AR Path="/60F1863C/60F5ECDF" Ref="C52"  Part="1"
+F 0 "C52" H 6365 3196 50  0000 L CNN
 F 1 "0,01" H 6365 3105 50  0000 L CNN
 F 2 "Capacitor_SMD:C_0603_1608Metric_Pad1.08x0.95mm_HandSolder" H 6288 3000 50  0001 C CNN
@@
 $EndComp
 Wire Wire Line
-	3500 4000 4500 4000
+	3000 4000 4500 4000
 Wire Wire Line
 	7500 4000 7500 3300
@@
 	4900 3200 4900 3500
 Wire Wire Line
-	4900 3500 3500 3500
-Wire Wire Line
-	3500 3000 4500 3000
-Connection ~ 4500 3000
+	4900 3500 3000 3500
 Wire Wire Line
 	4500 3000 5000 3000
@@
 AR Path="/60DF0860/60F633BE" Ref="R?"  Part="1"
 AR Path="/60DF07DE/60F633BE" Ref="R?"  Part="1"
-AR Path="/60F1863C/60F633BE" Ref="R?"  Part="1"
-F 0 "R?" H 8070 3796 50  0000 L CNN
+AR Path="/60F1863C/60F633BE" Ref="R47"  Part="1"
+F 0 "R47" H 8070 3796 50  0000 L CNN
 F 1 "1k 1%" H 8070 3705 50  0000 L CNN
 F 2 "Resistor_SMD:R_0603_1608Metric_Pad0.98x0.95mm_HandSolder" V 7930 3750 50  0001 C CNN
@@
 AR Path="/60DF0860/60F633C4" Ref="R?"  Part="1"
 AR Path="/60DF07DE/60F633C4" Ref="R?"  Part="1"
-AR Path="/60F1863C/60F633C4" Ref="R?"  Part="1"
-F 0 "R?" H 8070 3196 50  0000 L CNN
+AR Path="/60F1863C/60F633C4" Ref="R46"  Part="1"
+F 0 "R46" H 8070 3196 50  0000 L CNN
 F 1 "2.7k 1%" H 8070 3105 50  0000 L CNN
 F 2 "Resistor_SMD:R_0603_1608Metric_Pad0.98x0.95mm_HandSolder" V 7930 3150 50  0001 C CNN
@@
 NoConn ~ 5800 3100
 NoConn ~ 5800 3500
+$Comp
+L Device:R R?
+U 1 1 60FD8AD9
+P 3900 3000
+AR Path="/60FD8AD9" Ref="R?"  Part="1"
+AR Path="/60B39FE1/60FD8AD9" Ref="R?"  Part="1"
+AR Path="/60DF1160/60F2690B/60FD8AD9" Ref="R?"  Part="1"
+AR Path="/60DF1160/60FD8AD9" Ref="R?"  Part="1"
+AR Path="/60DF212D/60FD8AD9" Ref="R?"  Part="1"
+AR Path="/60F1863C/60FD8AD9" Ref="R43"  Part="1"
+F 0 "R43" V 4000 2900 50  0000 L CNN
+F 1 "0" V 3800 2950 50  0000 L CNN
+F 2 "" V 3830 3000 50  0001 C CNN
+F 3 "~" H 3900 3000 50  0001 C CNN
+	1    3900 3000
+	0    -1   -1   0
+$EndComp
+Wire Wire Line
+	4050 3000 4250 3000
+Connection ~ 4500 3000
+$Comp
+L Connector:TestPoint TP?
+U 1 1 611C47E1
+P 4250 3000
+AR Path="/611C47E1" Ref="TP?"  Part="1"
+AR Path="/609FED99/611C47E1" Ref="TP?"  Part="1"
+AR Path="/60DF0860/611C47E1" Ref="TP?"  Part="1"
+AR Path="/60DF07DE/611C47E1" Ref="TP?"  Part="1"
+AR Path="/60F1863C/611C47E1" Ref="TP20"  Part="1"
+F 0 "TP20" H 4308 3118 50  0000 L CNN
+F 1 "TestPoint" H 4308 3027 50  0001 L CNN
+F 2 "" H 4450 3000 50  0001 C CNN
+F 3 "~" H 4450 3000 50  0001 C CNN
+	1    4250 3000
+	1    0    0    -1
+$EndComp
+Connection ~ 4250 3000
+Wire Wire Line
+	4250 3000 4500 3000
+$Comp
+L Connector:TestPoint TP?
+U 1 1 611C4C71
+P 3500 3000
+AR Path="/611C4C71" Ref="TP?"  Part="1"
+AR Path="/609FED99/611C4C71" Ref="TP?"  Part="1"
+AR Path="/60DF0860/611C4C71" Ref="TP?"  Part="1"
+AR Path="/60DF07DE/611C4C71" Ref="TP?"  Part="1"
+AR Path="/60F1863C/611C4C71" Ref="TP19"  Part="1"
+F 0 "TP19" H 3558 3118 50  0000 L CNN
+F 1 "TestPoint" H 3558 3027 50  0001 L CNN
+F 2 "" H 3700 3000 50  0001 C CNN
+F 3 "~" H 3700 3000 50  0001 C CNN
+	1    3500 3000
+	1    0    0    -1
+$EndComp
+Connection ~ 3500 3000
+Wire Wire Line
+	3500 3000 3000 3000
+Wire Wire Line
+	3500 3000 3750 3000
 $EndSCHEMATC

Commit message: Add files via upload
Parts:
- C51, C52, C53: symbol Device:C -> rata-rescue:C-Device
- R43, R44, R45, R46, R47: symbol Device:R -> rata-rescue:R-Device
- TP19, TP20, TP21: symbol Connector:TestPoint -> rata-rescue:TestPoint-Connector
- U11: symbol Regulator_Linear:LP2951-5.0_SOIC -> rata-rescue:LP2951-5.0_SOIC-Regulator_Linear
Changed lines of the file:
@@
 LDO +4V5
 $Comp
-L Connector:TestPoint TP?
+L rata-rescue:TestPoint-Connector TP?
 U 1 1 60F18F0D
 P 8500 3000
@@
 +4V5_OUT
 $Comp
-L Regulator_Linear:LP2951-5.0_SOIC U11
+L rata-rescue:LP2951-5.0_SOIC-Regulator_Linear U11
 U 1 1 60F560B0
 P 5400 3300
@@
 $EndComp
 $Comp
-L Device:C C?
+L rata-rescue:C-Device C?
 U 1 1 60F593FA
 P 7500 3150
@@
 $EndComp
 $Comp
-L Device:C C?
+L rata-rescue:C-Device C?
 U 1 1 60F59400
 P 4500 3150
@@
 $EndComp
 $Comp
-L Device:R R?
+L rata-rescue:R-Device R?
 U 1 1 60F5D079
 P 6750 3750
@@
 $EndComp
 $Comp
-L Device:R R?
+L rata-rescue:R-Device R?
 U 1 1 60F5D07F
 P 6750 3150
@@
 VOLT
 $Comp
-L Device:C C?
+L rata-rescue:C-Device C?
 U 1 1 60F5ECDF
 P 6250 3150
@@
 	6750 3400 6750 3600
 $Comp
-L Device:R R?
+L rata-rescue:R-Device R?
 U 1 1 60F633BE
 P 8000 3750
@@
 $EndComp
 $Comp
-L Device:R R?
+L rata-rescue:R-Device R?
 U 1 1 60F633C4
 P 8000 3150
@@
 NoConn ~ 5800 3500
 $Comp
-L Device:R R?
+L rata-rescue:R-Device R?
 U 1 1 60FD8AD9
 P 3900 3000
@@
 Connection ~ 4500 3000
 $Comp
-L Connector:TestPoint TP?
+L rata-rescue:TestPoint-Connector TP?
 U 1 1 611C47E1
 P 4250 3000
@@
 	4250 3000 4500 3000
 $Comp
-L Connector:TestPoint TP?
+L rata-rescue:TestPoint-Connector TP?
 U 1 1 611C4C71
 P 3500 3000

Commit message: Add files via upload
Parts:
- R44: renamed from R43; footprint (none) -> Resistor_SMD:R_0805_2012Metric_Pad1.20x1.40mm_HandSolder
- TP19, TP20, TP21: footprint (none) -> rata:TP
- renumbered R44 to R45, R45 to R46, R46 to R47, R47 to R48
Changed lines of the file:
@@
 encoding utf-8
 Sheet 14 23
-Title ""
-Date ""
-Rev ""
-Comp ""
+Title "rata"
+Date "2021-09-25"
+Rev "1.0"
+Comp "Yuriy Volkov"
 Comment1 ""
 Comment2 ""
@@
 F 0 "TP21" H 8558 3118 50  0000 L CNN
 F 1 "TestPoint" H 8558 3027 50  0001 L CNN
-F 2 "" H 8700 3000 50  0001 C CNN
+F 2 "rata:TP" H 8700 3000 50  0001 C CNN
 F 3 "~" H 8700 3000 50  0001 C CNN
 	1    8500 3000
@@
 AR Path="/60DF0860/60F5D079" Ref="R?"  Part="1"
 AR Path="/60DF07DE/60F5D079" Ref="R?"  Part="1"
-AR Path="/60F1863C/60F5D079" Ref="R45"  Part="1"
-F 0 "R45" H 6820 3796 50  0000 L CNN
+AR Path="/60F1863C/60F5D079" Ref="R46"  Part="1"
+F 0 "R46" H 6820 3796 50  0000 L CNN
 F 1 "1k 1%" H 6820 3705 50  0000 L CNN
 F 2 "Resistor_SMD:R_0603_1608Metric_Pad0.98x0.95mm_HandSolder" V 6680 3750 50  0001 C CNN
@@
 AR Path="/60DF0860/60F5D07F" Ref="R?"  Part="1"
 AR Path="/60DF07DE/60F5D07F" Ref="R?"  Part="1"
-AR Path="/60F1863C/60F5D07F" Ref="R44"  Part="1"
-F 0 "R44" H 6820 3196 50  0000 L CNN
+AR Path="/60F1863C/60F5D07F" Ref="R45"  Part="1"
+F 0 "R45" H 6820 3196 50  0000 L CNN
 F 1 "2.7k 1%" H 6820 3105 50  0000 L CNN
 F 2 "Resistor_SMD:R_0603_1608Metric_Pad0.98x0.95mm_HandSolder" V 6680 3150 50  0001 C CNN
@@
 	4900 3500 3000 3500
 Wire Wire Line
-	4500 3000 5000 3000
+	4500 3000 4800 3000
 Wire Wire Line
 	5800 3000 6250 3000
@@
 AR Path="/60DF0860/60F633BE" Ref="R?"  Part="1"
 AR Path="/60DF07DE/60F633BE" Ref="R?"  Part="1"
-AR Path="/60F1863C/60F633BE" Ref="R47"  Part="1"
-F 0 "R47" H 8070 3796 50  0000 L CNN
+AR Path="/60F1863C/60F633BE" Ref="R48"  Part="1"
+F 0 "R48" H 8070 3796 50  0000 L CNN
 F 1 "1k 1%" H 8070 3705 50  0000 L CNN
 F 2 "Resistor_SMD:R_0603_1608Metric_Pad0.98x0.95mm_HandSolder" V 7930 3750 50  0001 C CNN
@@
 AR Path="/60DF0860/60F633C4" Ref="R?"  Part="1"
 AR Path="/60DF07DE/60F633C4" Ref="R?"  Part="1"
-AR Path="/60F1863C/60F633C4" Ref="R46"  Part="1"
-F 0 "R46" H 8070 3196 50  0000 L CNN
+AR Path="/60F1863C/60F633C4" Ref="R47"  Part="1"
+F 0 "R47" H 8070 3196 50  0000 L CNN
 F 1 "2.7k 1%" H 8070 3105 50  0000 L CNN
 F 2 "Resistor_SMD:R_0603_1608Metric_Pad0.98x0.95mm_HandSolder" V 7930 3150 50  0001 C CNN
@@
 AR Path="/60DF1160/60FD8AD9" Ref="R?"  Part="1"
 AR Path="/60DF212D/60FD8AD9" Ref="R?"  Part="1"
-AR Path="/60F1863C/60FD8AD9" Ref="R43"  Part="1"
-F 0 "R43" V 4000 2900 50  0000 L CNN
+AR Path="/60F1863C/60FD8AD9" Ref="R44"  Part="1"
+F 0 "R44" V 4000 2900 50  0000 L CNN
 F 1 "0" V 3800 2950 50  0000 L CNN
-F 2 "" V 3830 3000 50  0001 C CNN
+F 2 "Resistor_SMD:R_0805_2012Metric_Pad1.20x1.40mm_HandSolder" V 3830 3000 50  0001 C CNN
 F 3 "~" H 3900 3000 50  0001 C CNN
 	1    3900 3000
@@
 F 0 "TP20" H 4308 3118 50  0000 L CNN
 F 1 "TestPoint" H 4308 3027 50  0001 L CNN
-F 2 "" H 4450 3000 50  0001 C CNN
+F 2 "rata:TP" H 4450 3000 50  0001 C CNN
 F 3 "~" H 4450 3000 50  0001 C CNN
 	1    4250 3000
@@
 F 0 "TP19" H 3558 3118 50  0000 L CNN
 F 1 "TestPoint" H 3558 3027 50  0001 L CNN
-F 2 "" H 3700 3000 50  0001 C CNN
+F 2 "rata:TP" H 3700 3000 50  0001 C CNN
 F 3 "~" H 3700 3000 50  0001 C CNN
 	1    3500 3000
@@
 Wire Wire Line
 	3500 3000 3750 3000
+$Comp
+L power:PWR_FLAG #FLG07
+U 1 1 615BADF8
+P 4800 3000
+F 0 "#FLG07" H 4800 3075 50  0001 C CNN
+F 1 "PWR_FLAG" H 4800 3173 50  0000 C CNN
+F 2 "" H 4800 3000 50  0001 C CNN
+F 3 "~" H 4800 3000 50  0001 C CNN
+	1    4800 3000
+	1    0    0    -1
+$EndComp
+Connection ~ 4800 3000
+Wire Wire Line
+	4800 3000 5000 3000
 $EndSCHEMATC
