File: RTC.sch (KiCad schematic (older format))
At the start: 10 parts

Commit message: Add files via upload
Parts:
- removed C?: 0,1, Capacitor_SMD:C_0603_1608Metric_Pad1.08x0.95mm_HandSolder, symbol Device:C
- added C?: 0,1, Capacitor_SMD:C_0603_1608Metric_Pad1.08x0.95mm_HandSolder, symbol Device:C
Connections:
- net GND: now also C?.2
- net at U?.14 (BBS), U?.5 (IFS): now also C?.1
Changed lines of the file:
@@
 $Descr A4 11693 8268
 encoding utf-8
-Sheet 15 15
+Sheet 15 20
 Title ""
 Date ""
@@
 $Comp
 L Device:C C?
-U 1 1 60DF1217
+U 1 1 60F186C3
 P 7250 3950
-AR Path="/60DF1217" Ref="C?"  Part="1"
-AR Path="/609CA6A8/609D24C0/60DF1217" Ref="C?"  Part="1"
-AR Path="/609CA6A8/60A08E0B/60DF1217" Ref="C?"  Part="1"
-AR Path="/609CA6A8/60A0A46E/60DF1217" Ref="C?"  Part="1"
-AR Path="/609CA6A8/60A0A500/60DF1217" Ref="C?"  Part="1"
-AR Path="/609CA6A8/60A0A922/60DF1217" Ref="C?"  Part="1"
-AR Path="/609CA6A8/60DF1217" Ref="C?"  Part="1"
-AR Path="/609CA6A8/60AE5653/60DF1217" Ref="C?"  Part="1"
-AR Path="/609FED99/60DF1217" Ref="C?"  Part="1"
-AR Path="/60DF07DE/60DF1217" Ref="C?"  Part="1"
-AR Path="/60DF0860/60DF1217" Ref="C?"  Part="1"
-AR Path="/60DF1072/60DF1217" Ref="C?"  Part="1"
-AR Path="/60DF1160/60DF1217" Ref="C?"  Part="1"
-AR Path="/60E72FD7/60DF1217" Ref="C?"  Part="1"
-AR Path="/60EF6B1B/60DF1217" Ref="C?"  Part="1"
+AR Path="/60F186C3" Ref="C?"  Part="1"
+AR Path="/609CA6A8/609D24C0/60F186C3" Ref="C?"  Part="1"
+AR Path="/609CA6A8/60A08E0B/60F186C3" Ref="C?"  Part="1"
+AR Path="/609CA6A8/60A0A46E/60F186C3" Ref="C?"  Part="1"
+AR Path="/609CA6A8/60A0A500/60F186C3" Ref="C?"  Part="1"
+AR Path="/609CA6A8/60A0A922/60F186C3" Ref="C?"  Part="1"
+AR Path="/609CA6A8/60F186C3" Ref="C?"  Part="1"
+AR Path="/609CA6A8/60AE5653/60F186C3" Ref="C?"  Part="1"
+AR Path="/609FED99/60F186C3" Ref="C?"  Part="1"
+AR Path="/60DF07DE/60F186C3" Ref="C?"  Part="1"
+AR Path="/60DF0860/60F186C3" Ref="C?"  Part="1"
+AR Path="/60DF1072/60F186C3" Ref="C?"  Part="1"
+AR Path="/60DF1160/60F186C3" Ref="C?"  Part="1"
+AR Path="/60E72FD7/60F186C3" Ref="C?"  Part="1"
+AR Path="/60EF6B1B/60F186C3" Ref="C?"  Part="1"
 F 0 "C?" H 7365 3996 50  0000 L CNN
 F 1 "0,1" H 7365 3905 50  0000 L CNN

Commit message: Add files via upload
Parts:
- gave numbers to parts that had none: 10
Changed lines of the file:
@@
 $Descr A4 11693 8268
 encoding utf-8
-Sheet 14 23
+Sheet 13 23
 Title ""
 Date ""
@@
 AR Path="/60DF1160/60EE8A0B" Ref="C?"  Part="1"
 AR Path="/60E72FD7/60EE8A0B" Ref="C?"  Part="1"
-AR Path="/60EF6B1B/60EE8A0B" Ref="C?"  Part="1"
-F 0 "C?" H 5115 3296 50  0000 L CNN
+AR Path="/60EF6B1B/60EE8A0B" Ref="C47"  Part="1"
+F 0 "C47" H 5115 3296 50  0000 L CNN
 F 1 "10u" H 5115 3205 50  0000 L CNN
 F 2 "Capacitor_SMD:C_1206_3216Metric_Pad1.33x1.80mm_HandSolder" H 5038 3100 50  0001 C CNN
@@
 AR Path="/60DF1160/60F186C3" Ref="C?"  Part="1"
 AR Path="/60E72FD7/60F186C3" Ref="C?"  Part="1"
-AR Path="/60EF6B1B/60F186C3" Ref="C?"  Part="1"
-F 0 "C?" H 7365 3996 50  0000 L CNN
+AR Path="/60EF6B1B/60F186C3" Ref="C49"  Part="1"
+F 0 "C49" H 7365 3996 50  0000 L CNN
 F 1 "0,1" H 7365 3905 50  0000 L CNN
 F 2 "Capacitor_SMD:C_0603_1608Metric_Pad1.08x0.95mm_HandSolder" H 7288 3800 50  0001 C CNN
@@
 Battery powered RTC
 $Comp
-L rata:PCF2129T_2,518 U?
+L rata:PCF2129T_2,518 U10
 U 1 1 60E75075
 P 6400 3800
-F 0 "U?" H 6600 3250 50  0000 C CNN
+F 0 "U10" H 6600 3250 50  0000 C CNN
 F 1 "PCF2129T_2,518" H 6850 3150 50  0000 C CNN
 F 2 "" H 6300 3800 50  0001 C CNN
@@
 AR Path="/60DF07DE/60E783E4" Ref="R?"  Part="1"
 AR Path="/60EE89A9/60E783E4" Ref="R?"  Part="1"
-AR Path="/60EF6B1B/60E783E4" Ref="R?"  Part="1"
-F 0 "R?" H 4070 3296 50  0000 L CNN
+AR Path="/60EF6B1B/60E783E4" Ref="R41"  Part="1"
+F 0 "R41" H 4070 3296 50  0000 L CNN
 F 1 "4,7k" H 4070 3205 50  0000 L CNN
 F 2 "Resistor_SMD:R_0603_1608Metric_Pad0.98x0.95mm_HandSolder" V 3930 3250 50  0001 C CNN
@@
 AR Path="/60B39FE1/60E783EA" Ref="R?"  Part="1"
 AR Path="/60EE89A9/60E783EA" Ref="R?"  Part="1"
-AR Path="/60EF6B1B/60E783EA" Ref="R?"  Part="1"
-F 0 "R?" V 4600 2950 50  0000 L CNN
+AR Path="/60EF6B1B/60E783EA" Ref="R42"  Part="1"
+F 0 "R42" V 4600 2950 50  0000 L CNN
 F 1 "330" V 4400 2950 50  0000 L CNN
 F 2 "Resistor_SMD:R_0603_1608Metric_Pad0.98x0.95mm_HandSolder" V 4430 3000 50  0001 C CNN
@@
 AR Path="/60DF07DE/60E784A4" Ref="R?"  Part="1"
 AR Path="/60EE89A9/60E784A4" Ref="R?"  Part="1"
-AR Path="/60EF6B1B/60E784A4" Ref="R?"  Part="1"
-F 0 "R?" H 3570 3296 50  0000 L CNN
+AR Path="/60EF6B1B/60E784A4" Ref="R40"  Part="1"
+F 0 "R40" H 3570 3296 50  0000 L CNN
 F 1 "4,7k" H 3570 3205 50  0000 L CNN
 F 2 "Resistor_SMD:R_0603_1608Metric_Pad0.98x0.95mm_HandSolder" V 3430 3250 50  0001 C CNN
@@
 AR Path="/60DF1160/60E7980C" Ref="C?"  Part="1"
 AR Path="/60E72FD7/60E7980C" Ref="C?"  Part="1"
-AR Path="/60EF6B1B/60E7980C" Ref="C?"  Part="1"
-F 0 "C?" H 7615 3296 50  0000 L CNN
+AR Path="/60EF6B1B/60E7980C" Ref="C50"  Part="1"
+F 0 "C50" H 7615 3296 50  0000 L CNN
 F 1 "0,1" H 7615 3205 50  0000 L CNN
 F 2 "Capacitor_SMD:C_0603_1608Metric_Pad1.08x0.95mm_HandSolder" H 7538 3100 50  0001 C CNN
@@
 AR Path="/60DF1160/60E79A99" Ref="C?"  Part="1"
 AR Path="/60E72FD7/60E79A99" Ref="C?"  Part="1"
-AR Path="/60EF6B1B/60E79A99" Ref="C?"  Part="1"
-F 0 "C?" H 5615 3296 50  0000 L CNN
+AR Path="/60EF6B1B/60E79A99" Ref="C48"  Part="1"
+F 0 "C48" H 5615 3296 50  0000 L CNN
 F 1 "0,1" H 5615 3205 50  0000 L CNN
 F 2 "Capacitor_SMD:C_0603_1608Metric_Pad1.08x0.95mm_HandSolder" H 5538 3100 50  0001 C CNN
@@
 SCK
 $Comp
-L Device:Battery_Cell BT?
+L Device:Battery_Cell BT1
 U 1 1 60E7F687
 P 8500 3300
-F 0 "BT?" H 8618 3396 50  0000 L CNN
+F 0 "BT1" H 8618 3396 50  0000 L CNN
 F 1 "Battery_Cell" H 8618 3305 50  0000 L CNN
 F 2 "" V 8500 3360 50  0001 C CNN
@@
 NoConn ~ 7000 3600
 $Comp
-L Connector:Conn_01x03_Male J?
+L Connector:Conn_01x03_Male J9
 U 1 1 60E973C8
 P 4200 4900
-F 0 "J?" H 4172 4924 50  0000 R CNN
+F 0 "J9" H 4172 4924 50  0000 R CNN
 F 1 "Conn_01x03_Male" H 4172 4833 50  0000 R CNN
 F 2 "" H 4200 4900 50  0001 C CNN

Commit message: Add files via upload
Parts:
- BT1: symbol Device:Battery_Cell -> rata-rescue:Battery_Cell-Device
- C47, C48, C49, C50: symbol Device:C -> rata-rescue:C-Device
- J9: symbol Connector:Conn_01x03_Male -> rata-rescue:Conn_01x03_Male-Connector
- R40, R41, R42: symbol Device:R -> rata-rescue:R-Device
Changed lines of the file:
@@
 $EndDescr
 $Comp
-L Device:C C?
+L rata-rescue:C-Device C?
 U 1 1 60EE8A0B
 P 5000 3250
@@
 $EndComp
 $Comp
-L Device:C C?
+L rata-rescue:C-Device C?
 U 1 1 60F186C3
 P 7250 3950
@@
 $EndComp
 $Comp
-L Device:R R?
+L rata-rescue:R-Device R?
 U 1 1 60E783E4
 P 4000 3250
@@
 $EndComp
 $Comp
-L Device:R R?
+L rata-rescue:R-Device R?
 U 1 1 60E783EA
 P 4500 3000
@@
 $EndComp
 $Comp
-L Device:R R?
+L rata-rescue:R-Device R?
 U 1 1 60E784A4
 P 3500 3250
@@
 $EndComp
 $Comp
-L Device:C C?
+L rata-rescue:C-Device C?
 U 1 1 60E7980C
 P 7500 3250
@@
 $EndComp
 $Comp
-L Device:C C?
+L rata-rescue:C-Device C?
 U 1 1 60E79A99
 P 5500 3250
@@
 SCK
 $Comp
-L Device:Battery_Cell BT1
+L rata-rescue:Battery_Cell-Device BT1
 U 1 1 60E7F687
 P 8500 3300
@@
 NoConn ~ 7000 3600
 $Comp
-L Connector:Conn_01x03_Male J9
+L rata-rescue:Conn_01x03_Male-Connector J9
 U 1 1 60E973C8
 P 4200 4900

Commit message: Add files via upload
Parts:
- BT1: value Battery_Cell -> CR2032; footprint (none) -> rata:BatteryHolder_CR2032
- J9: value Conn_01x03_Male -> PLS-3; footprint (none) -> Connector_PinHeader_2.54mm:PinHeader_1x03_P2.54mm_Vertical
- U10: footprint (none) -> Package_SO:SOIC-16W_7.5x10.3mm_P1.27mm
- renumbered R40 to R41, R41 to R42, R42 to R43
Changed lines of the file:
@@
 encoding utf-8
 Sheet 13 23
-Title ""
-Date ""
-Rev ""
-Comp ""
+Title "rata"
+Date "2021-09-25"
+Rev "1.0"
+Comp "Yuriy Volkov"
 Comment1 ""
 Comment2 ""
@@
 F 0 "U10" H 6600 3250 50  0000 C CNN
 F 1 "PCF2129T_2,518" H 6850 3150 50  0000 C CNN
-F 2 "" H 6300 3800 50  0001 C CNN
+F 2 "Package_SO:SOIC-16W_7.5x10.3mm_P1.27mm" H 6300 3800 50  0001 C CNN
 F 3 "" H 6300 3800 50  0001 C CNN
 	1    6400 3800
@@
 AR Path="/60DF07DE/60E783E4" Ref="R?"  Part="1"
 AR Path="/60EE89A9/60E783E4" Ref="R?"  Part="1"
-AR Path="/60EF6B1B/60E783E4" Ref="R41"  Part="1"
-F 0 "R41" H 4070 3296 50  0000 L CNN
+AR Path="/60EF6B1B/60E783E4" Ref="R42"  Part="1"
+F 0 "R42" H 4070 3296 50  0000 L CNN
 F 1 "4,7k" H 4070 3205 50  0000 L CNN
 F 2 "Resistor_SMD:R_0603_1608Metric_Pad0.98x0.95mm_HandSolder" V 3930 3250 50  0001 C CNN
@@
 AR Path="/60B39FE1/60E783EA" Ref="R?"  Part="1"
 AR Path="/60EE89A9/60E783EA" Ref="R?"  Part="1"
-AR Path="/60EF6B1B/60E783EA" Ref="R42"  Part="1"
-F 0 "R42" V 4600 2950 50  0000 L CNN
+AR Path="/60EF6B1B/60E783EA" Ref="R43"  Part="1"
+F 0 "R43" V 4600 2950 50  0000 L CNN
 F 1 "330" V 4400 2950 50  0000 L CNN
 F 2 "Resistor_SMD:R_0603_1608Metric_Pad0.98x0.95mm_HandSolder" V 4430 3000 50  0001 C CNN
@@
 AR Path="/60DF07DE/60E784A4" Ref="R?"  Part="1"
 AR Path="/60EE89A9/60E784A4" Ref="R?"  Part="1"
-AR Path="/60EF6B1B/60E784A4" Ref="R40"  Part="1"
-F 0 "R40" H 3570 3296 50  0000 L CNN
+AR Path="/60EF6B1B/60E784A4" Ref="R41"  Part="1"
+F 0 "R41" H 3570 3296 50  0000 L CNN
 F 1 "4,7k" H 3570 3205 50  0000 L CNN
 F 2 "Resistor_SMD:R_0603_1608Metric_Pad0.98x0.95mm_HandSolder" V 3430 3250 50  0001 C CNN
@@
 P 8500 3300
 F 0 "BT1" H 8618 3396 50  0000 L CNN
-F 1 "Battery_Cell" H 8618 3305 50  0000 L CNN
-F 2 "" V 8500 3360 50  0001 C CNN
+F 1 "CR2032" H 8618 3305 50  0000 L CNN
+F 2 "rata:BatteryHolder_CR2032" V 8500 3360 50  0001 C CNN
 F 3 "~" V 8500 3360 50  0001 C CNN
 	1    8500 3300
@@
 	6500 3400 6500 3000
 Wire Wire Line
-	6500 3000 7500 3000
+	6500 3000 7000 3000
 Wire Wire Line
 	8500 3000 8500 3100
@@
 	6400 3400 6400 3000
 Wire Wire Line
-	6400 3000 5500 3000
+	6400 3000 6000 3000
 Wire Wire Line
 	5000 3100 5000 3000
@@
 P 4200 4900
 F 0 "J9" H 4172 4924 50  0000 R CNN
-F 1 "Conn_01x03_Male" H 4172 4833 50  0000 R CNN
-F 2 "" H 4200 4900 50  0001 C CNN
+F 1 "PLS-3" H 4172 4833 50  0000 R CNN
+F 2 "Connector_PinHeader_2.54mm:PinHeader_1x03_P2.54mm_Vertical" H 4200 4900 50  0001 C CNN
 F 3 "~" H 4200 4900 50  0001 C CNN
 	1    4200 4900
@@
 Wire Wire Line
 	3700 3500 4500 3500
+$Comp
+L power:PWR_FLAG #FLG06
+U 1 1 615B5B5C
+P 7000 3000
+F 0 "#FLG06" H 7000 3075 50  0001 C CNN
+F 1 "PWR_FLAG" H 7000 3173 50  0000 C CNN
+F 2 "" H 7000 3000 50  0001 C CNN
+F 3 "~" H 7000 3000 50  0001 C CNN
+	1    7000 3000
+	1    0    0    -1
+$EndComp
+Connection ~ 7000 3000
+Wire Wire Line
+	7000 3000 7500 3000
+$Comp
+L power:PWR_FLAG #FLG05
+U 1 1 615B6DFE
+P 6000 3000
+F 0 "#FLG05" H 6000 3075 50  0001 C CNN
+F 1 "PWR_FLAG" H 6000 3173 50  0000 C CNN
+F 2 "" H 6000 3000 50  0001 C CNN
+F 3 "~" H 6000 3000 50  0001 C CNN
+	1    6000 3000
+	1    0    0    -1
+$EndComp
+Connection ~ 6000 3000
+Wire Wire Line
+	6000 3000 5500 3000
 $EndSCHEMATC
