File: Switch.sch (KiCad schematic (older format))
At the start: 10 parts

Commit message: Add files via upload
Parts:
- removed C?: 100u, symbol Device:CP
- removed TP? (x2): TestPoint, symbol Connector:TestPoint
- added C?: 100u, symbol Device:CP
- added TP? (x2): TestPoint, symbol Connector:TestPoint
Changed lines of the file:
@@
 $Descr A4 11693 8268
 encoding utf-8
-Sheet 5 11
+Sheet 11 15
 Title ""
 Date ""
@@
 $Comp
 L Connector:TestPoint TP?
-U 1 1 60DF19BA
+U 1 1 60E73026
 P 7550 3500
-AR Path="/60DF19BA" Ref="TP?"  Part="1"
-AR Path="/609FED99/60DF19BA" Ref="TP?"  Part="1"
-AR Path="/60DF07DE/60DF19BA" Ref="TP?"  Part="1"
-AR Path="/60DF0860/60DF19BA" Ref="TP?"  Part="1"
-AR Path="/60DF1072/60DF19BA" Ref="TP?"  Part="1"
-AR Path="/60DF1160/60DF19BA" Ref="TP?"  Part="1"
-AR Path="/60DF196E/60DF19BA" Ref="TP?"  Part="1"
-AR Path="/60DF212D/60DF19BA" Ref="TP?"  Part="1"
+AR Path="/60E73026" Ref="TP?"  Part="1"
+AR Path="/609FED99/60E73026" Ref="TP?"  Part="1"
+AR Path="/60DF07DE/60E73026" Ref="TP?"  Part="1"
+AR Path="/60DF0860/60E73026" Ref="TP?"  Part="1"
+AR Path="/60DF1072/60E73026" Ref="TP?"  Part="1"
+AR Path="/60DF1160/60E73026" Ref="TP?"  Part="1"
+AR Path="/60DF196E/60E73026" Ref="TP?"  Part="1"
+AR Path="/60DF212D/60E73026" Ref="TP?"  Part="1"
 F 0 "TP?" H 7608 3618 50  0000 L CNN
 F 1 "TestPoint" H 7608 3527 50  0001 L CNN
@@
 $Comp
 L Device:CP C?
-U 1 1 60DF19BC
+U 1 1 60E73027
 P 3800 3650
-AR Path="/609FED99/60DF19BC" Ref="C?"  Part="1"
-AR Path="/60DF07DE/60DF19BC" Ref="C?"  Part="1"
-AR Path="/60DF0860/60DF19BC" Ref="C?"  Part="1"
-AR Path="/60DF1072/60DF19BC" Ref="C?"  Part="1"
-AR Path="/60DF1160/60DF19BC" Ref="C?"  Part="1"
-AR Path="/60DF196E/60DF19BC" Ref="C?"  Part="1"
-AR Path="/60DF212D/60DF19BC" Ref="C?"  Part="1"
+AR Path="/609FED99/60E73027" Ref="C?"  Part="1"
+AR Path="/60DF07DE/60E73027" Ref="C?"  Part="1"
+AR Path="/60DF0860/60E73027" Ref="C?"  Part="1"
+AR Path="/60DF1072/60E73027" Ref="C?"  Part="1"
+AR Path="/60DF1160/60E73027" Ref="C?"  Part="1"
+AR Path="/60DF196E/60E73027" Ref="C?"  Part="1"
+AR Path="/60DF212D/60E73027" Ref="C?"  Part="1"
 F 0 "C?" H 3918 3696 50  0000 L CNN
 F 1 "100u" H 3918 3605 50  0000 L CNN
@@
 $Comp
 L Connector:TestPoint TP?
-U 1 1 60DF0A64
+U 1 1 60E73020
 P 5400 3800
-AR Path="/60DF0A64" Ref="TP?"  Part="1"
-AR Path="/609FED99/60DF0A64" Ref="TP?"  Part="1"
-AR Path="/60DF07DE/60DF0A64" Ref="TP?"  Part="1"
-AR Path="/60DF0860/60DF0A64" Ref="TP?"  Part="1"
-AR Path="/60DF1072/60DF0A64" Ref="TP?"  Part="1"
-AR Path="/60DF1160/60DF0A64" Ref="TP?"  Part="1"
-AR Path="/60DF196E/60DF0A64" Ref="TP?"  Part="1"
-AR Path="/60DF212D/60DF0A64" Ref="TP?"  Part="1"
+AR Path="/60E73020" Ref="TP?"  Part="1"
+AR Path="/609FED99/60E73020" Ref="TP?"  Part="1"
+AR Path="/60DF07DE/60E73020" Ref="TP?"  Part="1"
+AR Path="/60DF0860/60E73020" Ref="TP?"  Part="1"
+AR Path="/60DF1072/60E73020" Ref="TP?"  Part="1"
+AR Path="/60DF1160/60E73020" Ref="TP?"  Part="1"
+AR Path="/60DF196E/60E73020" Ref="TP?"  Part="1"
+AR Path="/60DF212D/60E73020" Ref="TP?"  Part="1"
 F 0 "TP?" H 5458 3918 50  0000 L CNN
 F 1 "TestPoint" H 5458 3827 50  0001 L CNN

Commit message: Add files via upload
Parts:
- removed C? (x2): 10u, Capacitor_SMD:C_1206_3216Metric_Pad1.33x1.80mm_HandSolder, symbol Device:C
- removed C?: 0,1, Capacitor_SMD:C_0603_1608Metric_Pad1.08x0.95mm_HandSolder, symbol Device:C
- removed C?: 1u, Capacitor_SMD:C_0603_1608Metric_Pad1.08x0.95mm_HandSolder, symbol Device:C
- removed TP?: TestPoint, symbol Connector:TestPoint
- removed U?: AMS1117-3.3, Package_TO_SOT_SMD:SOT-223-3_TabPin2, symbol Regulator_Linear:AMS1117-3.3
- added C? (x2): 10u, Capacitor_SMD:C_1206_3216Metric_Pad1.33x1.80mm_HandSolder, symbol Device:C
- added C?: 0,1, Capacitor_SMD:C_0603_1608Metric_Pad1.08x0.95mm_HandSolder, symbol Device:C
- added C?: 1u, Capacitor_SMD:C_0603_1608Metric_Pad1.08x0.95mm_HandSolder, symbol Device:C
- added TP?: TestPoint, symbol Connector:TestPoint
- added U?: AMS1117-3.3, Package_TO_SOT_SMD:SOT-223-3_TabPin2, symbol Regulator_Linear:AMS1117-3.3

Commit message: Add files via upload
Parts:
- removed C?: 100u, symbol Device:CP
- removed C? (x2): 10u, Capacitor_SMD:C_1206_3216Metric_Pad1.33x1.80mm_HandSolder, symbol Device:C
- removed C?: 0,1, Capacitor_SMD:C_0603_1608Metric_Pad1.08x0.95mm_HandSolder, symbol Device:C
- removed C?: 1u, Capacitor_SMD:C_0603_1608Metric_Pad1.08x0.95mm_HandSolder, symbol Device:C
- removed D?: SMAJ5.0CA, symbol Device:D_TVS
- removed TP? (x3): TestPoint, symbol Connector:TestPoint
- removed U?: AMS1117-3.3, Package_TO_SOT_SMD:SOT-223-3_TabPin2, symbol Regulator_Linear:AMS1117-3.3
- added R?: 10k, Resistor_SMD:R_0603_1608Metric_Pad0.98x0.95mm_HandSolder, symbol Device:R
- added SW? (x2): SW_DPDT_x2, symbol Switch:SW_DPDT_x2
Connections:
- net labels added: +3V3, ALARM
- net labels removed: +3V3_OUT, +5V_IN
- wire segments 18 -> 8
- no-connect marks 0 -> 3
Other:
- note added: "Alarm switch"
- note removed: "Power source +3V3"

Commit message: Add files via upload
Parts:
- R25: renamed from R?; value 10k -> 4.7k
- gave numbers to parts that had none: 1
Changed lines of the file:
@@
 ALARM
 $Comp
-L Switch:SW_DPDT_x2 SW?
+L Switch:SW_DPDT_x2 SW10
 U 1 1 60F712E0
 P 6800 4000
-F 0 "SW?" H 6800 4285 50  0000 C CNN
+F 0 "SW10" H 6800 4285 50  0000 C CNN
 F 1 "SW_DPDT_x2" H 6800 4194 50  0000 C CNN
 F 2 "" H 6800 4000 50  0001 C CNN
@@
 $EndComp
 $Comp
-L Switch:SW_DPDT_x2 SW?
+L Switch:SW_DPDT_x2 SW10
 U 2 1 60F71AB8
 P 6800 5000
-F 0 "SW?" H 6800 5285 50  0000 C CNN
+F 0 "SW10" H 6800 5285 50  0000 C CNN
 F 1 "SW_DPDT_x2" H 6800 5194 50  0000 C CNN
 F 2 "" H 6800 5000 50  0001 C CNN
@@
 AR Path="/60DF1160/60F2690B/60F73202" Ref="R?"  Part="1"
 AR Path="/60DF1160/60F73202" Ref="R?"  Part="1"
-AR Path="/60DF212D/60F73202" Ref="R?"  Part="1"
-F 0 "R?" V 5850 3450 50  0000 L CNN
-F 1 "10k" V 5650 3400 50  0000 L CNN
+AR Path="/60DF212D/60F73202" Ref="R25"  Part="1"
+F 0 "R25" V 5850 3450 50  0000 L CNN
+F 1 "4.7k" V 5650 3400 50  0000 L CNN
 F 2 "Resistor_SMD:R_0603_1608Metric_Pad0.98x0.95mm_HandSolder" V 5680 3500 50  0001 C CNN
 F 3 "~" H 5750 3500 50  0001 C CNN

Commit message: Add files via upload
Parts:
- R25: symbol Device:R -> rata-rescue:R-Device
- SW10: symbol Switch:SW_DPDT_x2 -> rata-rescue:SW_DPDT_x2-Switch
Changed lines of the file:
@@
 ALARM
 $Comp
-L Switch:SW_DPDT_x2 SW10
+L rata-rescue:SW_DPDT_x2-Switch SW10
 U 1 1 60F712E0
 P 6800 4000
@@
 $EndComp
 $Comp
-L Switch:SW_DPDT_x2 SW10
+L rata-rescue:SW_DPDT_x2-Switch SW10
 U 2 1 60F71AB8
 P 6800 5000
@@
 $EndComp
 $Comp
-L Device:R R?
+L rata-rescue:R-Device R?
 U 1 1 60F73202
 P 5750 3500

Commit message: Add files via upload
Parts:
- SW10: value SW_DPDT_x2 -> PKN-61; footprint (none) -> rata:PKN-61
- renumbered R25 to R26
Changed lines of the file:
@@
 encoding utf-8
 Sheet 10 23
-Title ""
-Date ""
-Rev ""
-Comp ""
+Title "rata"
+Date "2021-09-25"
+Rev "1.0"
+Comp "Yuriy Volkov"
 Comment1 ""
 Comment2 ""
@@
 P 6800 4000
 F 0 "SW10" H 6800 4285 50  0000 C CNN
-F 1 "SW_DPDT_x2" H 6800 4194 50  0000 C CNN
-F 2 "" H 6800 4000 50  0001 C CNN
+F 1 "PKN-61" H 6800 4194 50  0000 C CNN
+F 2 "rata:PKN-61" H 6800 4000 50  0001 C CNN
 F 3 "~" H 6800 4000 50  0001 C CNN
 	1    6800 4000
@@
 P 6800 5000
 F 0 "SW10" H 6800 5285 50  0000 C CNN
-F 1 "SW_DPDT_x2" H 6800 5194 50  0000 C CNN
-F 2 "" H 6800 5000 50  0001 C CNN
+F 1 "PKN-61" H 6800 5194 50  0000 C CNN
+F 2 "rata:PKN-61" H 6800 5000 50  0001 C CNN
 F 3 "~" H 6800 5000 50  0001 C CNN
 	2    6800 5000
@@
 AR Path="/60DF1160/60F2690B/60F73202" Ref="R?"  Part="1"
 AR Path="/60DF1160/60F73202" Ref="R?"  Part="1"
-AR Path="/60DF212D/60F73202" Ref="R25"  Part="1"
-F 0 "R25" V 5850 3450 50  0000 L CNN
+AR Path="/60DF212D/60F73202" Ref="R26"  Part="1"
+F 0 "R26" V 5850 3450 50  0000 L CNN
 F 1 "4.7k" V 5650 3400 50  0000 L CNN
 F 2 "Resistor_SMD:R_0603_1608Metric_Pad0.98x0.95mm_HandSolder" V 5680 3500 50  0001 C CNN
