File: Temp_sensor.sch (KiCad schematic (older format))
At the start: 11 parts

Commit message: Add files via upload
Parts:
- removed C? (x2): 10u, Capacitor_SMD:C_1206_3216Metric_Pad1.33x1.80mm_HandSolder, symbol Device:C
- removed C?: 0,1, Capacitor_SMD:C_0603_1608Metric_Pad1.08x0.95mm_HandSolder, symbol Device:C
- removed C?: 1u, Capacitor_SMD:C_0603_1608Metric_Pad1.08x0.95mm_HandSolder, symbol Device:C
- removed C?: 100u, symbol Device:CP
- removed D?: SMAJ5.0CA, symbol Device:D_TVS
- removed TP? (x3): TestPoint, symbol Connector:TestPoint
- removed U?: AMS1117-3.3, Package_TO_SOT_SMD:SOT-223-3_TabPin2, symbol Regulator_Linear:AMS1117-3.3
- added C? (x2): 0,1, Capacitor_SMD:C_0603_1608Metric_Pad1.08x0.95mm_HandSolder, symbol Device:C
- added J?: Conn_01x03_Male, symbol Connector:Conn_01x03_Male
- added R? (x2): 4,7k, Resistor_SMD:R_0603_1608Metric_Pad0.98x0.95mm_HandSolder, symbol Device:R
- added R? (x2): 0, Resistor_SMD:R_0603_1608Metric_Pad0.98x0.95mm_HandSolder, symbol Device:R
Connections:
- net labels added: +3V3, +3V3A, SCK, SDA
- net labels removed: +3V3_OUT, +5V_IN
- wire segments 18 -> 44
Other:
- note added: "BME280 humiduty and temperature sensor"
- note removed: "Power source +3V3"
- moved on the sheet: U?

Commit message: Add files via upload
Parts:
- gave numbers to parts that had none: 8
Changed lines of the file:
@@
 $Descr A4 11693 8268
 encoding utf-8
-Sheet 17 23
+Sheet 16 23
 Title ""
 Date ""
@@
 BME280 humiduty and temperature sensor
 $Comp
-L Sensor:BME280 U?
+L Sensor:BME280 U12
 U 1 1 60F46B21
 P 4900 4800
-F 0 "U?" H 4471 4846 50  0000 R CNN
+F 0 "U12" H 4471 4846 50  0000 R CNN
 F 1 "BME280" H 4471 4755 50  0000 R CNN
 F 2 "Package_LGA:Bosch_LGA-8_2.5x2.5mm_P0.65mm_ClockwisePinNumbering" H 6400 4350 50  0001 C CNN
@@
 AR Path="/60EF6B1B/60FE7830" Ref="R?"  Part="1"
 AR Path="/60DF196E/60FE7830" Ref="R?"  Part="1"
-AR Path="/60F1A0E6/60FE7830" Ref="R?"  Part="1"
-F 0 "R?" H 7570 4296 50  0000 L CNN
+AR Path="/60F1A0E6/60FE7830" Ref="R53"  Part="1"
+F 0 "R53" H 7570 4296 50  0000 L CNN
 F 1 "4,7k" H 7570 4205 50  0000 L CNN
 F 2 "Resistor_SMD:R_0603_1608Metric_Pad0.98x0.95mm_HandSolder" V 7430 4250 50  0001 C CNN
@@
 AR Path="/60EF6B1B/60FE7836" Ref="R?"  Part="1"
 AR Path="/60DF196E/60FE7836" Ref="R?"  Part="1"
-AR Path="/60F1A0E6/60FE7836" Ref="R?"  Part="1"
-F 0 "R?" H 7070 4296 50  0000 L CNN
+AR Path="/60F1A0E6/60FE7836" Ref="R52"  Part="1"
+F 0 "R52" H 7070 4296 50  0000 L CNN
 F 1 "4,7k" H 7070 4205 50  0000 L CNN
 F 2 "Resistor_SMD:R_0603_1608Metric_Pad0.98x0.95mm_HandSolder" V 6930 4250 50  0001 C CNN
@@
 AR Path="/60F18EC1/60F77470/60FE8694" Ref="R?"  Part="1"
 AR Path="/60F18EC1/60F77508/60FE8694" Ref="R?"  Part="1"
-AR Path="/60F1A0E6/60FE8694" Ref="R?"  Part="1"
-F 0 "R?" V 6000 3450 50  0000 L CNN
+AR Path="/60F1A0E6/60FE8694" Ref="R51"  Part="1"
+F 0 "R51" V 6000 3450 50  0000 L CNN
 F 1 "0" V 5800 3500 50  0000 L CNN
 F 2 "Resistor_SMD:R_0603_1608Metric_Pad0.98x0.95mm_HandSolder" V 5830 3500 50  0001 C CNN
@@
 P 7200 5400
 AR Path="/60EF6B1B/60FEC4F6" Ref="J?"  Part="1"
-AR Path="/60F1A0E6/60FEC4F6" Ref="J?"  Part="1"
-F 0 "J?" H 7172 5424 50  0000 R CNN
+AR Path="/60F1A0E6/60FEC4F6" Ref="J10"  Part="1"
+F 0 "J10" H 7172 5424 50  0000 R CNN
 F 1 "Conn_01x03_Male" H 7172 5333 50  0000 R CNN
 F 2 "" H 7200 5400 50  0001 C CNN
@@
 AR Path="/60DF212D/60FF5E30" Ref="C?"  Part="1"
 AR Path="/60F197D4/60FF5E30" Ref="C?"  Part="1"
-AR Path="/60F1A0E6/60FF5E30" Ref="C?"  Part="1"
-F 0 "C?" H 5615 3696 50  0000 L CNN
+AR Path="/60F1A0E6/60FF5E30" Ref="C56"  Part="1"
+F 0 "C56" H 5615 3696 50  0000 L CNN
 F 1 "0,1" H 5615 3605 50  0000 L CNN
 F 2 "Capacitor_SMD:C_0603_1608Metric_Pad1.08x0.95mm_HandSolder" H 5538 3500 50  0001 C CNN
@@
 AR Path="/60DF212D/60FF5F7B" Ref="C?"  Part="1"
 AR Path="/60F197D4/60FF5F7B" Ref="C?"  Part="1"
-AR Path="/60F1A0E6/60FF5F7B" Ref="C?"  Part="1"
-F 0 "C?" H 4615 3696 50  0000 L CNN
+AR Path="/60F1A0E6/60FF5F7B" Ref="C55"  Part="1"
+F 0 "C55" H 4615 3696 50  0000 L CNN
 F 1 "0,1" H 4615 3605 50  0000 L CNN
 F 2 "Capacitor_SMD:C_0603_1608Metric_Pad1.08x0.95mm_HandSolder" H 4538 3500 50  0001 C CNN
@@
 AR Path="/60F18EC1/60F77470/60FF4BFC" Ref="R?"  Part="1"
 AR Path="/60F18EC1/60F77508/60FF4BFC" Ref="R?"  Part="1"
-AR Path="/60F1A0E6/60FF4BFC" Ref="R?"  Part="1"
-F 0 "R?" V 5150 3450 50  0000 L CNN
+AR Path="/60F1A0E6/60FF4BFC" Ref="R50"  Part="1"
+F 0 "R50" V 5150 3450 50  0000 L CNN
 F 1 "0" V 4950 3500 50  0000 L CNN
 F 2 "Resistor_SMD:R_0603_1608Metric_Pad0.98x0.95mm_HandSolder" V 4980 3500 50  0001 C CNN

Commit message: Add files via upload
Parts:
- C55, C56: symbol Device:C -> rata-rescue:C-Device
- J10: symbol Connector:Conn_01x03_Male -> rata-rescue:Conn_01x03_Male-Connector
- R50, R51, R52, R53: symbol Device:R -> rata-rescue:R-Device
- U12: symbol Sensor:BME280 -> rata-rescue:BME280-Sensor
Changed lines of the file:
@@
 BME280 humiduty and temperature sensor
 $Comp
-L Sensor:BME280 U12
+L rata-rescue:BME280-Sensor U12
 U 1 1 60F46B21
 P 4900 4800
@@
 $EndComp
 $Comp
-L Device:R R?
+L rata-rescue:R-Device R?
 U 1 1 60FE7830
 P 7500 4250
@@
 $EndComp
 $Comp
-L Device:R R?
+L rata-rescue:R-Device R?
 U 1 1 60FE7836
 P 7000 4250
@@
 $EndComp
 $Comp
-L Device:R R?
+L rata-rescue:R-Device R?
 U 1 1 60FE8694
 P 5900 3500
@@
 $EndComp
 $Comp
-L Connector:Conn_01x03_Male J?
+L rata-rescue:Conn_01x03_Male-Connector J?
 U 1 1 60FEC4F6
 P 7200 5400
@@
 SCK
 $Comp
-L Device:C C?
+L rata-rescue:C-Device C?
 U 1 1 60FF5E30
 P 5500 3650
@@
 $EndComp
 $Comp
-L Device:C C?
+L rata-rescue:C-Device C?
 U 1 1 60FF5F7B
 P 4500 3650
@@
 $EndComp
 $Comp
-L Device:R R?
+L rata-rescue:R-Device R?
 U 1 1 60FF4BFC
 P 5050 3500

Commit message: Add files via upload
Parts:
- J10: value Conn_01x03_Male -> PLS-3; footprint (none) -> Connector_PinHeader_2.54mm:PinHeader_1x03_P2.54mm_Vertical
- R51: renamed from R50; footprint Resistor_SMD:R_0603_1608Metric_Pad0.98x0.95mm_HandSolder -> Resistor_SMD:R_0805_2012Metric_Pad1.20x1.40mm_HandSolder
- R52: renamed from R51; footprint Resistor_SMD:R_0603_1608Metric_Pad0.98x0.95mm_HandSolder -> Resistor_SMD:R_0805_2012Metric_Pad1.20x1.40mm_HandSolder
- renumbered C55 to C56, C56 to C57, R52 to R53, R53 to R54
Changed lines of the file:
@@
 encoding utf-8
 Sheet 16 23
-Title ""
-Date ""
-Rev ""
-Comp ""
+Title "rata"
+Date "2021-09-25"
+Rev "1.0"
+Comp "Yuriy Volkov"
 Comment1 ""
 Comment2 ""
@@
 AR Path="/60EF6B1B/60FE7830" Ref="R?"  Part="1"
 AR Path="/60DF196E/60FE7830" Ref="R?"  Part="1"
-AR Path="/60F1A0E6/60FE7830" Ref="R53"  Part="1"
-F 0 "R53" H 7570 4296 50  0000 L CNN
+AR Path="/60F1A0E6/60FE7830" Ref="R54"  Part="1"
+F 0 "R54" H 7570 4296 50  0000 L CNN
 F 1 "4,7k" H 7570 4205 50  0000 L CNN
 F 2 "Resistor_SMD:R_0603_1608Metric_Pad0.98x0.95mm_HandSolder" V 7430 4250 50  0001 C CNN
@@
 AR Path="/60EF6B1B/60FE7836" Ref="R?"  Part="1"
 AR Path="/60DF196E/60FE7836" Ref="R?"  Part="1"
-AR Path="/60F1A0E6/60FE7836" Ref="R52"  Part="1"
-F 0 "R52" H 7070 4296 50  0000 L CNN
+AR Path="/60F1A0E6/60FE7836" Ref="R53"  Part="1"
+F 0 "R53" H 7070 4296 50  0000 L CNN
 F 1 "4,7k" H 7070 4205 50  0000 L CNN
 F 2 "Resistor_SMD:R_0603_1608Metric_Pad0.98x0.95mm_HandSolder" V 6930 4250 50  0001 C CNN
@@
 AR Path="/60F18EC1/60F77470/60FE8694" Ref="R?"  Part="1"
 AR Path="/60F18EC1/60F77508/60FE8694" Ref="R?"  Part="1"
-AR Path="/60F1A0E6/60FE8694" Ref="R51"  Part="1"
-F 0 "R51" V 6000 3450 50  0000 L CNN
+AR Path="/60F1A0E6/60FE8694" Ref="R52"  Part="1"
+F 0 "R52" V 6000 3450 50  0000 L CNN
 F 1 "0" V 5800 3500 50  0000 L CNN
-F 2 "Resistor_SMD:R_0603_1608Metric_Pad0.98x0.95mm_HandSolder" V 5830 3500 50  0001 C CNN
+F 2 "Resistor_SMD:R_0805_2012Metric_Pad1.20x1.40mm_HandSolder" V 5830 3500 50  0001 C CNN
 F 3 "~" H 5900 3500 50  0001 C CNN
 	1    5900 3500
@@
 AR Path="/60F1A0E6/60FEC4F6" Ref="J10"  Part="1"
 F 0 "J10" H 7172 5424 50  0000 R CNN
-F 1 "Conn_01x03_Male" H 7172 5333 50  0000 R CNN
-F 2 "" H 7200 5400 50  0001 C CNN
+F 1 "PLS-3" H 7172 5333 50  0000 R CNN
+F 2 "Connector_PinHeader_2.54mm:PinHeader_1x03_P2.54mm_Vertical" H 7200 5400 50  0001 C CNN
 F 3 "~" H 7200 5400 50  0001 C CNN
 	1    7200 5400
@@
 AR Path="/60DF212D/60FF5E30" Ref="C?"  Part="1"
 AR Path="/60F197D4/60FF5E30" Ref="C?"  Part="1"
-AR Path="/60F1A0E6/60FF5E30" Ref="C56"  Part="1"
-F 0 "C56" H 5615 3696 50  0000 L CNN
+AR Path="/60F1A0E6/60FF5E30" Ref="C57"  Part="1"
+F 0 "C57" H 5615 3696 50  0000 L CNN
 F 1 "0,1" H 5615 3605 50  0000 L CNN
 F 2 "Capacitor_SMD:C_0603_1608Metric_Pad1.08x0.95mm_HandSolder" H 5538 3500 50  0001 C CNN
@@
 AR Path="/60DF212D/60FF5F7B" Ref="C?"  Part="1"
 AR Path="/60F197D4/60FF5F7B" Ref="C?"  Part="1"
-AR Path="/60F1A0E6/60FF5F7B" Ref="C55"  Part="1"
-F 0 "C55" H 4615 3696 50  0000 L CNN
+AR Path="/60F1A0E6/60FF5F7B" Ref="C56"  Part="1"
+F 0 "C56" H 4615 3696 50  0000 L CNN
 F 1 "0,1" H 4615 3605 50  0000 L CNN
 F 2 "Capacitor_SMD:C_0603_1608Metric_Pad1.08x0.95mm_HandSolder" H 4538 3500 50  0001 C CNN
@@
 AR Path="/60F18EC1/60F77470/60FF4BFC" Ref="R?"  Part="1"
 AR Path="/60F18EC1/60F77508/60FF4BFC" Ref="R?"  Part="1"
-AR Path="/60F1A0E6/60FF4BFC" Ref="R50"  Part="1"
-F 0 "R50" V 5150 3450 50  0000 L CNN
+AR Path="/60F1A0E6/60FF4BFC" Ref="R51"  Part="1"
+F 0 "R51" V 5150 3450 50  0000 L CNN
 F 1 "0" V 4950 3500 50  0000 L CNN
-F 2 "Resistor_SMD:R_0603_1608Metric_Pad0.98x0.95mm_HandSolder" V 4980 3500 50  0001 C CNN
+F 2 "Resistor_SMD:R_0805_2012Metric_Pad1.20x1.40mm_HandSolder" V 4980 3500 50  0001 C CNN
 F 3 "~" H 5050 3500 50  0001 C CNN
 	1    5050 3500
@@
 Connection ~ 5300 3500
 Wire Wire Line
-	5300 3500 5500 3500
+	5300 3500 5400 3500
 Wire Wire Line
 	6050 3500 6250 3500
@@
 Wire Wire Line
 	5750 5500 5000 5500
+$Comp
+L power:PWR_FLAG #FLG08
+U 1 1 615BCBCF
+P 5400 3500
+F 0 "#FLG08" H 5400 3575 50  0001 C CNN
+F 1 "PWR_FLAG" H 5400 3673 50  0000 C CNN
+F 2 "" H 5400 3500 50  0001 C CNN
+F 3 "~" H 5400 3500 50  0001 C CNN
+	1    5400 3500
+	1    0    0    -1
+$EndComp
+Connection ~ 5400 3500
+Wire Wire Line
+	5400 3500 5500 3500
 $EndSCHEMATC
