File: VFD_driver.sch (KiCad schematic (older format))
At the start: 38 parts

Commit message: Add files via upload
Parts:
- gave numbers to parts that had none: 38
Connections:
- net VCC renamed +VCC

Commit message: Add files via upload
Parts:
- C57, C58, C59, C60: symbol Device:C -> rata-rescue:C-Device
- R54, R55, R56, R57, R58, R59, R60, R61, R62, R63, R64, R65, R66, R67, R68, R69, R70, R71, R72, R73, R74, R75, R76, R77, R78, R79, R80, R81, R82, R83: symbol Device:R -> rata-rescue:R-Device
- U13, U14: symbol Interface_Expansion:PCF8574 -> rata-rescue:PCF8574-Interface_Expansion
Changed lines of the file:
@@
 $EndDescr
 $Comp
-L Device:C C?
+L rata-rescue:C-Device C?
 U 1 1 60DF0A5D
 P 2500 2750
@@
 +VCC
 $Comp
-L Interface_Expansion:PCF8574 U13
+L rata-rescue:PCF8574-Interface_Expansion U13
 U 1 1 60F6CDCB
 P 3500 3400
@@
 $EndComp
 $Comp
-L Device:R R?
+L rata-rescue:R-Device R?
 U 1 1 60F845F7
 P 1900 2750
@@
 $EndComp
 $Comp
-L Device:R R?
+L rata-rescue:R-Device R?
 U 1 1 60F84E12
 P 4500 2750
@@
 $EndComp
 $Comp
-L Device:R R?
+L rata-rescue:R-Device R?
 U 1 1 60F858A7
 P 4800 2750
@@
 $EndComp
 $Comp
-L Device:R R?
+L rata-rescue:R-Device R?
 U 1 1 60F85DFA
 P 5100 2750
@@
 $EndComp
 $Comp
-L Device:R R?
+L rata-rescue:R-Device R?
 U 1 1 60F860DE
 P 5400 2750
@@
 $EndComp
 $Comp
-L Device:R R?
+L rata-rescue:R-Device R?
 U 1 1 60F862F9
 P 5700 2750
@@
 $EndComp
 $Comp
-L Device:R R?
+L rata-rescue:R-Device R?
 U 1 1 60F86717
 P 6000 2750
@@
 $EndComp
 $Comp
-L Device:R R?
+L rata-rescue:R-Device R?
 U 1 1 60F86ADC
 P 4800 4750
@@
 $EndComp
 $Comp
-L Device:R R?
+L rata-rescue:R-Device R?
 U 1 1 60F86E0D
 P 5100 4750
@@
 $EndComp
 $Comp
-L Device:R R?
+L rata-rescue:R-Device R?
 U 1 1 60F870C9
 P 5400 4750
@@
 $EndComp
 $Comp
-L Device:R R?
+L rata-rescue:R-Device R?
 U 1 1 60F873E2
 P 5700 4750
@@
 $EndComp
 $Comp
-L Device:R R?
+L rata-rescue:R-Device R?
 U 1 1 60F877BB
 P 6000 4750
@@
 $EndComp
 $Comp
-L Device:R R?
+L rata-rescue:R-Device R?
 U 1 1 60F87A9B
 P 6300 2750
@@
 $EndComp
 $Comp
-L Device:R R?
+L rata-rescue:R-Device R?
 U 1 1 60F87D37
 P 6600 2750
@@
 $EndComp
 $Comp
-L Device:R R?
+L rata-rescue:R-Device R?
 U 1 1 60F88070
 P 4500 4750
@@
 $EndComp
 $Comp
-L Device:C C?
+L rata-rescue:C-Device C?
 U 1 1 60F8C66E
 P 2500 4650
@@
 $EndComp
 $Comp
-L Device:R R?
+L rata-rescue:R-Device R?
 U 1 1 60F8D8C6
 P 1500 2750
@@
 SCK
 $Comp
-L Device:C C?
+L rata-rescue:C-Device C?
 U 1 1 60F9F811
 P 7500 2750
@@
 $EndComp
 $Comp
-L Interface_Expansion:PCF8574 U14
+L rata-rescue:PCF8574-Interface_Expansion U14
 U 1 1 60FA2526
 P 3500 5400
@@
 $EndComp
 $Comp
-L Device:C C?
+L rata-rescue:C-Device C?
 U 1 1 60FAF440
 P 7500 4750
@@
 $EndComp
 $Comp
-L Device:R R?
+L rata-rescue:R-Device R?
 U 1 1 60FB19D3
 P 9850 3000
@@
 $EndComp
 $Comp
-L Device:R R?
+L rata-rescue:R-Device R?
 U 1 1 60FB1D57
 P 9850 3250
@@
 $EndComp
 $Comp
-L Device:R R?
+L rata-rescue:R-Device R?
 U 1 1 60FB1FB6
 P 9850 3500
@@
 $EndComp
 $Comp
-L Device:R R?
+L rata-rescue:R-Device R?
 U 1 1 60FB2169
 P 9850 3750
@@
 $EndComp
 $Comp
-L Device:R R?
+L rata-rescue:R-Device R?
 U 1 1 60FB23D2
 P 9850 4000
@@
 $EndComp
 $Comp
-L Device:R R?
+L rata-rescue:R-Device R?
 U 1 1 60FB260C
 P 9850 4250
@@
 $EndComp
 $Comp
-L Device:R R?
+L rata-rescue:R-Device R?
 U 1 1 60FB27D9
 P 9850 4500
@@
 $EndComp
 $Comp
-L Device:R R?
+L rata-rescue:R-Device R?
 U 1 1 60FB29A6
 P 9850 4750
@@
 $EndComp
 $Comp
-L Device:R R?
+L rata-rescue:R-Device R?
 U 1 1 60FB2BA3
 P 9850 5000
@@
 $EndComp
 $Comp
-L Device:R R?
+L rata-rescue:R-Device R?
 U 1 1 60FB2DC0
 P 9850 5250
@@
 $EndComp
 $Comp
-L Device:R R?
+L rata-rescue:R-Device R?
 U 1 1 60FB2FBC
 P 9850 5500
@@
 $EndComp
 $Comp
-L Device:R R?
+L rata-rescue:R-Device R?
 U 1 1 60FB319F
 P 9850 5750
@@
 $EndComp
 $Comp
-L Device:R R?
+L rata-rescue:R-Device R?
 U 1 1 60FB17A8
 P 9850 2750
@@
 $EndComp
 $Comp
-L Device:R R?
+L rata-rescue:R-Device R?
 U 1 1 60F421DA
 P 9850 2500

Commit message: Add files via upload
Parts:
- U14: renamed from U13; footprint (none) -> Package_SO:SOIC-16W_7.5x10.3mm_P1.27mm
- U15: renamed from U14; footprint (none) -> Package_SO:SOIC-16W_7.5x10.3mm_P1.27mm
- U16: renamed from U15; footprint (none) -> Package_SO:SOIC-18W_7.5x11.6mm_P1.27mm
- U17: renamed from U16; footprint (none) -> Package_SO:SOIC-18W_7.5x11.6mm_P1.27mm
- renumbered C57 to C64, C58 to C65, C59 to C66, C60 to C67, R79 to R100, R80 to R101, R81 to R102, R82 to R103, R83 to R104, R54 to R75, R55 to R76, R56 to R77, R57 to R78, R58 to R79, R59 to R80, R62 to R81, R61 to R82, R64 to R83, R63 to R84, R66 to R85, R65 to R86, R60 to R87, R67 to R88, R68 to R89, R69 to R90, R70 to R91, R71 to R92, R72 to R93, R73 to R94, R74 to R95, R75 to R96, R76 to R97, R77 to R98, R78 to R99
Connections:
- net at R77.2, U14.4 (P0): now also U16.5 (I5); no longer U16.1 (I1)
- net at R79.2, U14.5 (P1): now also U16.6 (I6); no longer U16.2 (I2)
- net at U16.11 (O8): no longer R98.1
- net at U16.12 (O7): no longer R97.1
- net at R80.2, U15.5 (P1): now also U17.6 (I6); no longer U17.2 (I2)
- net at R82.2, U15.6 (P2): now also U17.7 (I7); no longer U17.3 (I3)
- net at R84.2, U15.7 (P3): now also U17.8 (I8); no longer U17.4 (I4)
- net at R86.2, U15.9 (P4): now also U17.1 (I1); no longer U17.5 (I5)
- net at R88.2, U15.10 (P5): now also U17.2 (I2); no longer U17.6 (I6)
- net at R78.2, U15.4 (P0): now also U17.5 (I5); no longer U17.1 (I1)
- net at U15.11 (P6): now also R89.2, U17.3 (I3)
- net at U15.12 (P7): now also R90.2, U17.4 (I4)
- net at U17.11 (O8): now also R104.1
- net at U17.12 (O7): now also R103.1
- net at U17.13 (O6): now also R102.1; no longer R104.1
- net at U17.14 (O5): now also R101.1; no longer R103.1
- net at U17.15 (O4): now also R100.1; no longer R102.1
- net at U17.16 (O3): now also R99.1; no longer R101.1
- net at U17.17 (O2): now also R98.1; no longer R100.1
- net at U17.18 (O1): now also R97.1; no longer R99.1
- new net: R83.2, U14.10 (P5), U16.2 (I2)
- new net: R85.2, U14.11 (P6), U16.3 (I3)
- new net: R87.2, U14.12 (P7), U16.4 (I4)
- new net: R81.2, U14.9 (P4), U16.1 (I1)
- now unconnected: U14.6 (P2), U14.7 (P3), U16.7 (I7), U16.8 (I8)
Other:
- moved on the sheet: C66, C67, R100, R101, R102, R103, R104, R81, R83, R85, R87, R89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
