File: VFD_heater.sch (KiCad schematic (older format))
At the start: 14 parts

Commit message: Add files via upload
Parts:
- gave numbers to parts that had none: 14
Changed lines of the file:
@@
 $Descr A4 11693 8268
 encoding utf-8
-Sheet 19 23
+Sheet 18 23
 Title ""
 Date ""
@@
 OUT0
 $Comp
-L Transistor_FET:IRLML6402 Q?
+L Transistor_FET:IRLML6402 Q4
 U 1 1 60A19F59
 P 5400 2250
-F 0 "Q?" H 5604 2204 50  0000 L CNN
+F 0 "Q4" H 5604 2204 50  0000 L CNN
 F 1 "IRLML6402" H 5604 2295 50  0000 L CNN
 F 2 "Package_TO_SOT_SMD:SOT-23" H 5600 2175 50  0001 L CIN
@@
 $EndComp
 $Comp
-L Transistor_FET:IRLML2060 Q?
+L Transistor_FET:IRLML2060 Q5
 U 1 1 60A1C2D8
 P 5400 3250
-F 0 "Q?" H 5604 3296 50  0000 L CNN
+F 0 "Q5" H 5604 3296 50  0000 L CNN
 F 1 "IRLML2402" H 5604 3205 50  0000 L CNN
 F 2 "Package_TO_SOT_SMD:SOT-23" H 5600 3175 50  0001 L CIN
@@
 AR Path="/60B39FE1/60B13DFF" Ref="R?"  Part="1"
 AR Path="/609FED99/60B13DFF" Ref="R?"  Part="1"
-AR Path="/60F18EC1/60B13DFF" Ref="R?"  Part="1"
-F 0 "R?" H 5070 3546 50  0000 L CNN
+AR Path="/60F18EC1/60B13DFF" Ref="R85"  Part="1"
+F 0 "R85" H 5070 3546 50  0000 L CNN
 F 1 "56k" H 5070 3455 50  0000 L CNN
 F 2 "Resistor_SMD:R_0603_1608Metric_Pad0.98x0.95mm_HandSolder" V 4930 3500 50  0001 C CNN
@@
 AR Path="/60B39FE1/60B1B4E2" Ref="R?"  Part="1"
 AR Path="/609FED99/60B1B4E2" Ref="R?"  Part="1"
-AR Path="/60F18EC1/60B1B4E2" Ref="R?"  Part="1"
-F 0 "R?" H 5070 2046 50  0000 L CNN
+AR Path="/60F18EC1/60B1B4E2" Ref="R84"  Part="1"
+F 0 "R84" H 5070 2046 50  0000 L CNN
 F 1 "56k" H 5070 1955 50  0000 L CNN
 F 2 "Resistor_SMD:R_0603_1608Metric_Pad0.98x0.95mm_HandSolder" V 4930 2000 50  0001 C CNN
@@
 $EndSheet
 $Comp
-L Transistor_FET:IRLML6402 Q?
+L Transistor_FET:IRLML6402 Q6
 U 1 1 60F84C82
 P 8400 4250
-F 0 "Q?" H 8604 4204 50  0000 L CNN
+F 0 "Q6" H 8604 4204 50  0000 L CNN
 F 1 "IRLML6402" H 8604 4295 50  0000 L CNN
 F 2 "Package_TO_SOT_SMD:SOT-23" H 8600 4175 50  0001 L CIN
@@
 $EndComp
 $Comp
-L Transistor_FET:IRLML2060 Q?
+L Transistor_FET:IRLML2060 Q7
 U 1 1 60F84C88
 P 8400 5250
-F 0 "Q?" H 8604 5296 50  0000 L CNN
+F 0 "Q7" H 8604 5296 50  0000 L CNN
 F 1 "IRLML2402" H 8604 5205 50  0000 L CNN
 F 2 "Package_TO_SOT_SMD:SOT-23" H 8600 5175 50  0001 L CIN
@@
 AR Path="/60B39FE1/60F84C8E" Ref="R?"  Part="1"
 AR Path="/609FED99/60F84C8E" Ref="R?"  Part="1"
-AR Path="/60F18EC1/60F84C8E" Ref="R?"  Part="1"
-F 0 "R?" H 8070 5546 50  0000 L CNN
+AR Path="/60F18EC1/60F84C8E" Ref="R87"  Part="1"
+F 0 "R87" H 8070 5546 50  0000 L CNN
 F 1 "56k" H 8070 5455 50  0000 L CNN
 F 2 "Resistor_SMD:R_0603_1608Metric_Pad0.98x0.95mm_HandSolder" V 7930 5500 50  0001 C CNN
@@
 AR Path="/60B39FE1/60F84C94" Ref="R?"  Part="1"
 AR Path="/609FED99/60F84C94" Ref="R?"  Part="1"
-AR Path="/60F18EC1/60F84C94" Ref="R?"  Part="1"
-F 0 "R?" H 8070 4046 50  0000 L CNN
+AR Path="/60F18EC1/60F84C94" Ref="R86"  Part="1"
+F 0 "R86" H 8070 4046 50  0000 L CNN
 F 1 "56k" H 8070 3955 50  0000 L CNN
 F 2 "Resistor_SMD:R_0603_1608Metric_Pad0.98x0.95mm_HandSolder" V 7930 4000 50  0001 C CNN
@@
 AR Path="/60DF196E/60FB0EC1" Ref="TP?"  Part="1"
 AR Path="/60EE89A9/60FB0EC1" Ref="TP?"  Part="1"
-AR Path="/60F18EC1/60FB0EC1" Ref="TP?"  Part="1"
-F 0 "TP?" H 4808 2368 50  0000 L CNN
+AR Path="/60F18EC1/60FB0EC1" Ref="TP24"  Part="1"
+F 0 "TP24" H 4808 2368 50  0000 L CNN
 F 1 "TestPoint" H 4808 2277 50  0001 L CNN
 F 2 "" H 4950 2250 50  0001 C CNN
@@
 AR Path="/60DF196E/60FB22C8" Ref="TP?"  Part="1"
 AR Path="/60EE89A9/60FB22C8" Ref="TP?"  Part="1"
-AR Path="/60F18EC1/60FB22C8" Ref="TP?"  Part="1"
-F 0 "TP?" H 4808 3368 50  0000 L CNN
+AR Path="/60F18EC1/60FB22C8" Ref="TP25"  Part="1"
+F 0 "TP25" H 4808 3368 50  0000 L CNN
 F 1 "TestPoint" H 4808 3277 50  0001 L CNN
 F 2 "" H 4950 3250 50  0001 C CNN
@@
 AR Path="/60DF196E/60FB376C" Ref="TP?"  Part="1"
 AR Path="/60EE89A9/60FB376C" Ref="TP?"  Part="1"
-AR Path="/60F18EC1/60FB376C" Ref="TP?"  Part="1"
-F 0 "TP?" H 7808 4368 50  0000 L CNN
+AR Path="/60F18EC1/60FB376C" Ref="TP26"  Part="1"
+F 0 "TP26" H 7808 4368 50  0000 L CNN
 F 1 "TestPoint" H 7808 4277 50  0001 L CNN
 F 2 "" H 7950 4250 50  0001 C CNN
@@
 AR Path="/60DF196E/60FB4B71" Ref="TP?"  Part="1"
 AR Path="/60EE89A9/60FB4B71" Ref="TP?"  Part="1"
-AR Path="/60F18EC1/60FB4B71" Ref="TP?"  Part="1"
-F 0 "TP?" H 7808 5368 50  0000 L CNN
+AR Path="/60F18EC1/60FB4B71" Ref="TP27"  Part="1"
+F 0 "TP27" H 7808 5368 50  0000 L CNN
 F 1 "TestPoint" H 7808 5277 50  0001 L CNN
 F 2 "" H 7950 5250 50  0001 C CNN
@@
 AR Path="/60DF196E/60FB684B" Ref="TP?"  Part="1"
 AR Path="/60EE89A9/60FB684B" Ref="TP?"  Part="1"
-AR Path="/60F18EC1/60FB684B" Ref="TP?"  Part="1"
-F 0 "TP?" H 9058 4868 50  0000 L CNN
+AR Path="/60F18EC1/60FB684B" Ref="TP29"  Part="1"
+F 0 "TP29" H 9058 4868 50  0000 L CNN
 F 1 "TestPoint" H 9058 4777 50  0001 L CNN
 F 2 "" H 9200 4750 50  0001 C CNN
@@
 AR Path="/60DF196E/60FB7BCC" Ref="TP?"  Part="1"
 AR Path="/60EE89A9/60FB7BCC" Ref="TP?"  Part="1"
-AR Path="/60F18EC1/60FB7BCC" Ref="TP?"  Part="1"
-F 0 "TP?" H 9058 2868 50  0000 L CNN
+AR Path="/60F18EC1/60FB7BCC" Ref="TP28"  Part="1"
+F 0 "TP28" H 9058 2868 50  0000 L CNN
 F 1 "TestPoint" H 9058 2777 50  0001 L CNN
 F 2 "" H 9200 2750 50  0001 C CNN

Commit message: Add files via upload
Parts:
- Q4, Q6: symbol Transistor_FET:IRLML6402 -> rata-rescue:IRLML6402-Transistor_FET
- Q5, Q7: symbol Transistor_FET:IRLML2060 -> rata-rescue:IRLML2060-Transistor_FET
- R84, R85, R86, R87: symbol Device:R -> rata-rescue:R-Device
- TP24, TP25, TP26, TP27, TP28, TP29: symbol Connector:TestPoint -> rata-rescue:TestPoint-Connector
Changed lines of the file:
@@
 OUT0
 $Comp
-L Transistor_FET:IRLML6402 Q4
+L rata-rescue:IRLML6402-Transistor_FET Q4
 U 1 1 60A19F59
 P 5400 2250
@@
 $EndComp
 $Comp
-L Transistor_FET:IRLML2060 Q5
+L rata-rescue:IRLML2060-Transistor_FET Q5
 U 1 1 60A1C2D8
 P 5400 3250
@@
 $EndComp
 $Comp
-L Device:R R?
+L rata-rescue:R-Device R?
 U 1 1 60B13DFF
 P 5000 3500
@@
 $EndComp
 $Comp
-L Device:R R?
+L rata-rescue:R-Device R?
 U 1 1 60B1B4E2
 P 5000 2000
@@
 $EndSheet
 $Comp
-L Transistor_FET:IRLML6402 Q6
+L rata-rescue:IRLML6402-Transistor_FET Q6
 U 1 1 60F84C82
 P 8400 4250
@@
 $EndComp
 $Comp
-L Transistor_FET:IRLML2060 Q7
+L rata-rescue:IRLML2060-Transistor_FET Q7
 U 1 1 60F84C88
 P 8400 5250
@@
 $EndComp
 $Comp
-L Device:R R?
+L rata-rescue:R-Device R?
 U 1 1 60F84C8E
 P 8000 5500
@@
 $EndComp
 $Comp
-L Device:R R?
+L rata-rescue:R-Device R?
 U 1 1 60F84C94
 P 8000 4000
@@
 	3000 3400 3000 6000
 $Comp
-L Connector:TestPoint TP?
+L rata-rescue:TestPoint-Connector TP?
 U 1 1 60FB0EC1
 P 4750 2250
@@
 $EndComp
 $Comp
-L Connector:TestPoint TP?
+L rata-rescue:TestPoint-Connector TP?
 U 1 1 60FB22C8
 P 4750 3250
@@
 $EndComp
 $Comp
-L Connector:TestPoint TP?
+L rata-rescue:TestPoint-Connector TP?
 U 1 1 60FB376C
 P 7750 4250
@@
 $EndComp
 $Comp
-L Connector:TestPoint TP?
+L rata-rescue:TestPoint-Connector TP?
 U 1 1 60FB4B71
 P 7750 5250
@@
 $EndComp
 $Comp
-L Connector:TestPoint TP?
+L rata-rescue:TestPoint-Connector TP?
 U 1 1 60FB684B
 P 9000 4750
@@
 $EndComp
 $Comp
-L Connector:TestPoint TP?
+L rata-rescue:TestPoint-Connector TP?
 U 1 1 60FB7BCC
 P 9000 2750

Commit message: Add files via upload
Parts:
- TP24, TP25, TP26, TP27, TP28, TP29: footprint (none) -> rata:TP
- renumbered R84 to R55, R85 to R56, R86 to R57, R87 to R58
Changed lines of the file:
@@
 $Descr A4 11693 8268
 encoding utf-8
-Sheet 18 23
-Title ""
-Date ""
-Rev ""
-Comp ""
+Sheet 17 23
+Title "rata"
+Date "2021-09-25"
+Rev "1.0"
+Comp "Yuriy Volkov"
 Comment1 ""
 Comment2 ""
@@
 AR Path="/60B39FE1/60B13DFF" Ref="R?"  Part="1"
 AR Path="/609FED99/60B13DFF" Ref="R?"  Part="1"
-AR Path="/60F18EC1/60B13DFF" Ref="R85"  Part="1"
-F 0 "R85" H 5070 3546 50  0000 L CNN
+AR Path="/60F18EC1/60B13DFF" Ref="R56"  Part="1"
+F 0 "R56" H 5070 3546 50  0000 L CNN
 F 1 "56k" H 5070 3455 50  0000 L CNN
 F 2 "Resistor_SMD:R_0603_1608Metric_Pad0.98x0.95mm_HandSolder" V 4930 3500 50  0001 C CNN
@@
 AR Path="/60B39FE1/60B1B4E2" Ref="R?"  Part="1"
 AR Path="/609FED99/60B1B4E2" Ref="R?"  Part="1"
-AR Path="/60F18EC1/60B1B4E2" Ref="R84"  Part="1"
-F 0 "R84" H 5070 2046 50  0000 L CNN
+AR Path="/60F18EC1/60B1B4E2" Ref="R55"  Part="1"
+F 0 "R55" H 5070 2046 50  0000 L CNN
 F 1 "56k" H 5070 1955 50  0000 L CNN
 F 2 "Resistor_SMD:R_0603_1608Metric_Pad0.98x0.95mm_HandSolder" V 4930 2000 50  0001 C CNN
@@
 AR Path="/60B39FE1/60F84C8E" Ref="R?"  Part="1"
 AR Path="/609FED99/60F84C8E" Ref="R?"  Part="1"
-AR Path="/60F18EC1/60F84C8E" Ref="R87"  Part="1"
-F 0 "R87" H 8070 5546 50  0000 L CNN
+AR Path="/60F18EC1/60F84C8E" Ref="R58"  Part="1"
+F 0 "R58" H 8070 5546 50  0000 L CNN
 F 1 "56k" H 8070 5455 50  0000 L CNN
 F 2 "Resistor_SMD:R_0603_1608Metric_Pad0.98x0.95mm_HandSolder" V 7930 5500 50  0001 C CNN
@@
 AR Path="/60B39FE1/60F84C94" Ref="R?"  Part="1"
 AR Path="/609FED99/60F84C94" Ref="R?"  Part="1"
-AR Path="/60F18EC1/60F84C94" Ref="R86"  Part="1"
-F 0 "R86" H 8070 4046 50  0000 L CNN
+AR Path="/60F18EC1/60F84C94" Ref="R57"  Part="1"
+F 0 "R57" H 8070 4046 50  0000 L CNN
 F 1 "56k" H 8070 3955 50  0000 L CNN
 F 2 "Resistor_SMD:R_0603_1608Metric_Pad0.98x0.95mm_HandSolder" V 7930 4000 50  0001 C CNN
@@
 F 0 "TP24" H 4808 2368 50  0000 L CNN
 F 1 "TestPoint" H 4808 2277 50  0001 L CNN
-F 2 "" H 4950 2250 50  0001 C CNN
+F 2 "rata:TP" H 4950 2250 50  0001 C CNN
 F 3 "~" H 4950 2250 50  0001 C CNN
 	1    4750 2250
@@
 F 0 "TP25" H 4808 3368 50  0000 L CNN
 F 1 "TestPoint" H 4808 3277 50  0001 L CNN
-F 2 "" H 4950 3250 50  0001 C CNN
+F 2 "rata:TP" H 4950 3250 50  0001 C CNN
 F 3 "~" H 4950 3250 50  0001 C CNN
 	1    4750 3250
@@
 F 0 "TP26" H 7808 4368 50  0000 L CNN
 F 1 "TestPoint" H 7808 4277 50  0001 L CNN
-F 2 "" H 7950 4250 50  0001 C CNN
+F 2 "rata:TP" H 7950 4250 50  0001 C CNN
 F 3 "~" H 7950 4250 50  0001 C CNN
 	1    7750 4250
@@
 F 0 "TP27" H 7808 5368 50  0000 L CNN
 F 1 "TestPoint" H 7808 5277 50  0001 L CNN
-F 2 "" H 7950 5250 50  0001 C CNN
+F 2 "rata:TP" H 7950 5250 50  0001 C CNN
 F 3 "~" H 7950 5250 50  0001 C CNN
 	1    7750 5250
@@
 F 0 "TP29" H 9058 4868 50  0000 L CNN
 F 1 "TestPoint" H 9058 4777 50  0001 L CNN
-F 2 "" H 9200 4750 50  0001 C CNN
+F 2 "rata:TP" H 9200 4750 50  0001 C CNN
 F 3 "~" H 9200 4750 50  0001 C CNN
 	1    9000 4750
@@
 F 0 "TP28" H 9058 2868 50  0000 L CNN
 F 1 "TestPoint" H 9058 2777 50  0001 L CNN
-F 2 "" H 9200 2750 50  0001 C CNN
+F 2 "rata:TP" H 9200 2750 50  0001 C CNN
 F 3 "~" H 9200 2750 50  0001 C CNN
 	1    9000 2750
